File: Battman/KiCad/Battman/AuxSupply_USB.kicad_sch (KiCad schematic)
At the start: 24 parts, among them IC400 LM1117MPX-3.3_NOPB, IC401 LT3990IMSE-5#PBF, IC402 TPS2116DRLR

Commit message: Uopdated Schematics fixed
Parts:
- removed C400, C401, C405, C406, C407: 0603YG104ZAT2A, C__Users_otto_Documents_AltiumLL_SamacSys.PcbLib:CAPC1608X90N, symbol Battman-altium-import:AuxSupply/USB_1_0603YG104ZAT2A_SamacSys.SchLib
- removed C403: 1206YD226KAT2A, FP-1206-L_3_2_0_2-W_1_6_0-IPC_C, symbol Battman-altium-import:AuxSupply/USB_0_mirrored_02cd4be3c70576c341d710602a673aa_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
- removed C404: C3216X7S2A225K160AB, FP-C3216-160-0_2-IPC_B, symbol Battman-altium-import:AuxSupply/USB_0_11868f565c42a9108669ba33697ecf6_Altium Co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
- removed D400: SMF5.0CA, C__Users_otto_Documents_AltiumLL_SamacSys.PcbLib:SODFL3618X108N, symbol Battman-altium-import:AuxSupply/USB_3_SMF5.0CA_*
- removed IC400: LM1117MPX-3.3_NOPB, C__Users_otto_Documents_AltiumLL_SamacSys.PcbLib:SOT230P700X180-4N, symbol Battman-altium-import:AuxSupply/USB_0_LM1117MPX-3.3_NOPB_SamacSys.SchLib
- removed L400: 7447714330, WE-PD_1050P, symbol Battman-altium-import:AuxSupply/USB_0_Inductor - 2_Altium Content Vault
- removed TP401: Test Pad 1mm, Test Pad 1mm-Footprint-1, symbol Battman-altium-import:AuxSupply/USB_3_Test Pad 1mm-Symbol-1_EPFL Racing Team
- added C400, C401, C405, C406, C407, C408: 100 nF, 100V, X7R, C__Users_otto_Documents_AltiumLL_SamacSys.PcbLib:MAJx16, symbol Battman-altium-import:AuxSupply/USB_1_MAJCH168BB7104KTEA01_SamacSys.SchLib
- added C403: 33uF 25V X5R, C__Users_otto_Documents_AltiumLL_SamacSys.PcbLib:CAPC3216X180N, symbol Battman-altium-import:AuxSupply/USB_1_C3216X5R1E336M160AC_SamacSys.SchLib
- added C404: 2.2 uF, 100V, X7R, C__Users_otto_Documents_AltiumLL_SamacSys.PcbLib:CAPC2012X145N, symbol Battman-altium-import:AuxSupply/USB_1_C2012X7R2A225K125AC_SamacSys.SchLib
- added IC400: TLV1117LV33DCYR, C__Users_otto_Documents_AltiumLL_SamacSys.PcbLib:SOT230P700X180-4N, symbol Battman-altium-import:AuxSupply/USB_0_TLV1117LV33DCYR_SamacSys.SchLib
- added L400: 47uH, C__Users_otto_Documents_AltiumLL_SamacSys.PcbLib:CLF6045_*, symbol Battman-altium-import:AuxSupply/USB_0_CLF6045NIT-470M-D_SamacSys.SchLib
- added R406: 270k, 1%, C__Users_otto_Documents_AltiumLL_SamacSys.PcbLib:RESC1608X55N, symbol Battman-altium-import:AuxSupply/USB_1_CRG0603F270K_SamacSys.SchLib
- added R407: 150k 0.5%, C__Users_otto_Documents_AltiumLL_SamacSys.PcbLib:ERA3AEB101V, symbol Battman-altium-import:AuxSupply/USB_1_ERA-3AED154V_SamacSys.SchLib
- added TP401: Test Pad 1mm, Test Pad 1mm-Footprint-1, symbol Battman-altium-import:AuxSupply/USB_1_Test Pad 1mm-Symbol-1_EPFL Racing Team
- added TP404, TP?: Test Pad 1mm, Test Pad 1mm-Footprint-1, symbol Battman-altium-import:AuxSupply/USB_0_Test Pad 1mm-Symbol-1_EPFL Racing Team
- C402: value GRM31C5C1H224JE02L -> 220nF 50V C0G; ALTIUM_VALUE 220nF 100V -> 220nF 50V
- R400, R401: value 27R -> 27R 5%; SUPPLIER 1 (none) -> Mouser; SUPPLIER PART NUMBER 1 (none) -> 660-RK73B1JTTD270J
- R402: value 1.3M -> 1.3M 1%; SUPPLIER 1 (none) -> Mouser; SUPPLIER PART NUMBER 1 (none) -> 594-MCT0603MD1304BP5
- R403: ALTIUM_VALUE 374k -> 374k 1%; SUPPLIER 1 (none) -> Avnet; SUPPLIER PART NUMBER 1 (none) -> RMCF0603FT374K
- R404: value 100R -> 100R, 1%; SUPPLIER 1 (none) -> Mouser; SUPPLIER PART NUMBER 1 (none) -> 71-CRCW0603-100-E3
- R405: value 100k -> 100k 1%; SUPPLIER 1 (none) -> Mouser; SUPPLIER PART NUMBER 1 (none) -> 71-CRCW0603100KFKEAC
Connections:
- net 3V3: now also C401.2, IC400.2 (OUT), TP401.1 (TP)
- net 5V: now also C400.2, C405.2, IC400.3 (IN)
- net 5V_Reg: now also C403.2, C406.2, L400.2, R406.2; no longer IC402.4 (PR1)
- net 5V_USB: now also C407.2, C408.2
- net Bat_GND_Fused: now also C400.1, C401.1, C403.1, C404.1, C405.1, C406.1, C407.1, C408.1, IC400.1 (GND), R407.1
- net at C402.2, IC401.9 (SW): now also L400.1
- net at IC401.14 (PG): now also TP?.1 (TP)
- net at IC401.6 (VIN), R404.1: now also C404.2
- net at IC402.8 (ST): now also TP404.1 (TP)
- new net 5V_Sel: IC402.4 (PR1), R406.1, R407.2
- no-connect marks 8 -> 6
Other:
- note added: "A1"
- note removed: "A0"

Commit message: Begin of kicad conversion
Parts:
- removed C400, C401, C405, C406, C407, C408: 100 nF, 100V, X7R, C__Users_otto_Documents_AltiumLL_SamacSys.PcbLib:MAJx16, symbol Battman-altium-import:AuxSupply/USB_1_MAJCH168BB7104KTEA01_SamacSys.SchLib
- removed C402: 220nF 50V C0G, C__Users_otto_Documents_AltiumLL_SamacSys.PcbLib:CAPC3216X180N, symbol Battman-altium-import:AuxSupply/USB_0_GRM31C5C1H224JE02L_SamacSys.SchLib
- removed C403: 33uF 25V X5R, C__Users_otto_Documents_AltiumLL_SamacSys.PcbLib:CAPC3216X180N, symbol Battman-altium-import:AuxSupply/USB_1_C3216X5R1E336M160AC_SamacSys.SchLib
- removed C404: 2.2 uF, 100V, X7R, C__Users_otto_Documents_AltiumLL_SamacSys.PcbLib:CAPC2012X145N, symbol Battman-altium-import:AuxSupply/USB_1_C2012X7R2A225K125AC_SamacSys.SchLib
- removed D401: PRTR5V0U2X,215, C__Users_otto_Documents_AltiumLL_SamacSys.PcbLib:PRTR5V0U2X, symbol Battman-altium-import:AuxSupply/USB_0_PRTR5V0U2X,215_SamacSys.SchLib
- removed IC400: TLV1117LV33DCYR, C__Users_otto_Documents_AltiumLL_SamacSys.PcbLib:SOT230P700X180-4N, symbol Battman-altium-import:AuxSupply/USB_0_TLV1117LV33DCYR_SamacSys.SchLib
- removed IC401: LT3990IMSE-5#PBF, C__Users_otto_Documents_AltiumLL_SamacSys.PcbLib:SOP50P490X110-17N, symbol Battman-altium-import:AuxSupply/USB_0_LT3990IMSE-5#PBF_SamacSys.SchLib
- removed IC402: TPS2116DRLR, C__Users_otto_Documents_AltiumLL_SamacSys.PcbLib:SOTFL50P160X60-8N, symbol Battman-altium-import:AuxSupply/USB_0_TPS2116DRLR_SamacSys.SchLib
- removed L400: 47uH, C__Users_otto_Documents_AltiumLL_SamacSys.PcbLib:CLF6045_*, symbol Battman-altium-import:AuxSupply/USB_0_CLF6045NIT-470M-D_SamacSys.SchLib
- removed R400, R401: 27R 5%, C__Users_otto_Documents_AltiumLL_SamacSys.PcbLib:RESC1608X55N, symbol Battman-altium-import:AuxSupply/USB_0_RK73B1JTTD270J_SamacSys.SchLib
- removed R402: 1.3M 1%, C__Users_otto_Documents_AltiumLL_SamacSys.PcbLib:RESC1608X55N, symbol Battman-altium-import:AuxSupply/USB_1_MCT0603MD1304BP500_SamacSys.SchLib
- removed R403: RMCF0603FT374K, C__Users_otto_Documents_AltiumLL_SamacSys.PcbLib:RESC1608X55N, symbol Battman-altium-import:AuxSupply/USB_2_RMCF0603FT374K_SamacSys.SchLib
- removed R404: 100R, 1%, C__Users_otto_Documents_AltiumLL_SamacSys.PcbLib:RESC1608X50N, symbol Battman-altium-import:AuxSupply/USB_1_CRCW0603100RFKEA_SamacSys.SchLib
- removed R405: 100k 1%, C__Users_otto_Documents_AltiumLL_SamacSys.PcbLib:RESC1608X55N, symbol Battman-altium-import:AuxSupply/USB_1_CRCW0603100KFKEAC_SamacSys.SchLib
- removed R406: 270k, 1%, C__Users_otto_Documents_AltiumLL_SamacSys.PcbLib:RESC1608X55N, symbol Battman-altium-import:AuxSupply/USB_1_CRG0603F270K_SamacSys.SchLib
- removed R407: 150k 0.5%, C__Users_otto_Documents_AltiumLL_SamacSys.PcbLib:ERA3AEB101V, symbol Battman-altium-import:AuxSupply/USB_1_ERA-3AED154V_SamacSys.SchLib
- removed TP400, TP402, TP403, TP404, TP?: Test Pad 1mm, Test Pad 1mm-Footprint-1, symbol Battman-altium-import:AuxSupply/USB_0_Test Pad 1mm-Symbol-1_EPFL Racing Team
- removed TP401: Test Pad 1mm, Test Pad 1mm-Footprint-1, symbol Battman-altium-import:AuxSupply/USB_1_Test Pad 1mm-Symbol-1_EPFL Racing Team
- added C400, C415: 10uF 10V X7R, C__Users_otto_Documents_AltiumLL_SamacSys.PcbLib:GRM18x, symbol Battman-altium-import:AuxSupply/USB_1_GRM188Z71A106MA73D_*
- added C401, C413, C416, C420: 100 nF, 100V, X7R, C__Users_otto_Documents_AltiumLL_SamacSys.PcbLib:MAJx16, symbol Battman-altium-import:AuxSupply/USB_3_MAJCH168BB7104KTEA01_SamacSys.SchLib
- added C402: 220nF 50V X7R, C__Users_otto_Documents_AltiumLL_SamacSys.PcbLib:GRM18x, symbol Battman-altium-import:AuxSupply/USB_0_GRM188R71H224KAC4J_*
- added C403: 33uF 25V X5R, C__Users_otto_Documents_AltiumLL_SamacSys.PcbLib:CAPC3216X180N, symbol Battman-altium-import:AuxSupply/USB_1_C3216X5R1E336M160AC_SamacSys.SchLib
- added C404: 2.2 uF, 100V, X7R, C__Users_otto_Documents_AltiumLL_SamacSys.PcbLib:CAPC2012X145N, symbol Battman-altium-import:AuxSupply/USB_1_C2012X7R2A225K125AC_SamacSys.SchLib
- added C405, C406, C407, C408: 100 nF, 100V, X7R, C__Users_otto_Documents_AltiumLL_SamacSys.PcbLib:MAJx16, symbol Battman-altium-import:AuxSupply/USB_1_MAJCH168BB7104KTEA01_SamacSys.SchLib
- added C409, C410: 100 nF, 100V, X7R, C__Users_otto_Documents_AltiumLL_SamacSys.PcbLib:MAJx16, symbol Battman-altium-import:AuxSupply/USB_2_MAJCH168BB7104KTEA01_SamacSys.SchLib
- added C411, C419: 1uF 50V X7R, C__Users_otto_Documents_AltiumLL_SamacSys.PcbLib:CAPC1608X90N, symbol Battman-altium-import:AuxSupply/USB_1_06035C105MAT2A_SamacSys.SchLib
- added C412: 1uF 50V X7R, C__Users_otto_Documents_AltiumLL_SamacSys.PcbLib:CAPC1608X90N, symbol Battman-altium-import:AuxSupply/USB_3_06035C105MAT2A_SamacSys.SchLib
- added C414, C418, C421: 22uF 10V X5R, C__Users_otto_Documents_AltiumLL_SamacSys.PcbLib:CAPC1608X105N, symbol Battman-altium-import:AuxSupply/USB_1_CL10A226MP8NUNE_*
- added D401: PRTR5V0U2X,215, C__Users_otto_Documents_AltiumLL_SamacSys.PcbLib:PRTR5V0U2X, symbol Battman-altium-import:AuxSupply/USB_0_PRTR5V0U2X,215_SamacSys.SchLib
- added IC400: MAX77827BEFD+T, C__Users_otto_Documents_AltiumLL_SamacSys.PcbLib:MAX77827BEFDT, symbol Battman-altium-import:AuxSupply/USB_3_MAX77827BEFD+T_*
- added IC401: LT3990IMSE-3.3#PBF, C__Users_otto_Documents_AltiumLL_SamacSys.PcbLib:SOP50P490X110-17N, symbol Battman-altium-import:AuxSupply/USB_0_LT3990IMSE-3.3#PBF_*
- added IC402: TPS2116DRLR, C__Users_otto_Documents_AltiumLL_SamacSys.PcbLib:SOTFL50P160X60-8N, symbol Battman-altium-import:AuxSupply/USB_0_TPS2116DRLR_SamacSys.SchLib
- added IC403: ISOUSB111DWXR, C__Users_otto_Documents_AltiumLL_SamacSys.PcbLib:SOP65P1030X260-16N, symbol Battman-altium-import:AuxSupply/USB_0_ISOUSB111DWXR_*
- added L400: VLS5045EX-220M, C__Users_otto_Documents_AltiumLL_SamacSys.PcbLib:VLS5045EX330M, symbol Battman-altium-import:AuxSupply/USB_0_VLS5045EX-220M_*
- added L401: DFE18SBN1R0ME0L, C__Users_otto_Documents_AltiumLL_SamacSys.PcbLib:DFE18SAN1R0ME0L, symbol Battman-altium-import:AuxSupply/USB_0_DFE18SBN1R0ME0L_*
- added PS400, PS401: R05C1TF05S-R, CONV_R05C1TF05S-R, symbol Battman-altium-import:AuxSupply/USB_0_R05C1TF05S-R_R05C1TF05S-R.SchLib
- added R400: 4.99k 1%, C__Users_otto_Documents_AltiumLL_SamacSys.PcbLib:RESC0603X26N, symbol Battman-altium-import:AuxSupply/USB_0_CR0201-FW-4991GLF_*
- added R402: 1.3M 1%, C__Users_otto_Documents_AltiumLL_SamacSys.PcbLib:RESC1608X55N, symbol Battman-altium-import:AuxSupply/USB_1_MCT0603MD1304BP500_SamacSys.SchLib
- added R403: 232k 1%, C__Users_otto_Documents_AltiumLL_SamacSys.PcbLib:RESC1608X50N, symbol Battman-altium-import:AuxSupply/USB_0_CRCW0603232KFKEA_*
- added R404: 100R, 1%, C__Users_otto_Documents_AltiumLL_SamacSys.PcbLib:RESC1608X50N, symbol Battman-altium-import:AuxSupply/USB_1_CRCW0603100RFKEA_SamacSys.SchLib
- added R405: 100k 1%, C__Users_otto_Documents_AltiumLL_SamacSys.PcbLib:RESC1608X55N, symbol Battman-altium-import:AuxSupply/USB_1_CRCW0603100KFKEAC_SamacSys.SchLib
- added R406, R407: 150k 0.5%, C__Users_otto_Documents_AltiumLL_SamacSys.PcbLib:ERA3AEB101V, symbol Battman-altium-import:AuxSupply/USB_1_ERA-3AED154V_SamacSys.SchLib
- added TP400, TP401, TP403, TP407: Testpoint, Testpoint, symbol Battman-altium-import:AuxSupply/USB_1_Testpoint_SamacSys.SchLib
- added TP402, TP404, TP405, TP406: Testpoint, Testpoint, symbol Battman-altium-import:AuxSupply/USB_0_Testpoint_SamacSys.SchLib
- added TP408: Testpoint, Testpoint, symbol Battman-altium-import:AuxSupply/USB_3_Testpoint_SamacSys.SchLib
Connections:
- no-connect marks 6 -> 15
Other:
- removed sheet USB
- note added: "3.3VDC From VBatt"
- note added: "3V3 Selector"
- note added: "A2"
- note added: "Isolated CAN Supply"
- note added: "USB INPUT Protection and Isolation"
- note added: "USB Supply isolation"
- note removed: "3,3V LDO"
- note removed: "5V Selector"
- note removed: "5VDC From VBatt"
- note removed: "A1"
- note removed: "USB INPUT Protection"
