File: Battman/KiCad/Battman/ConfigMultiplexer.kicad_sch (KiCad schematic)
At the start: 5 parts, among them IC500 ADG704BRMZ

Commit message: Uopdated Schematics fixed
Parts:
- removed C500: 0603YG104ZAT2A, C__Users_otto_Documents_AltiumLL_SamacSys.PcbLib:CAPC1608X90N, symbol Battman-altium-import:Repeat(Multiplexer,1,8)_1_0603YG104ZAT2A_SamacSys.SchLib
- added C500: 100 nF, 100V, X7R, C__Users_otto_Documents_AltiumLL_SamacSys.PcbLib:MAJx16, symbol Battman-altium-import:Repeat(Multiplexer,1,8)_1_MAJCH168BB7104KTEA01_SamacSys.S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
Connections:
- net GND_LTC_H: now also C500.1
- net Vreg: now also C500.2
Other:
- note added: "A1"
- note removed: "A0"

Commit message: Begin of kicad conversion
Parts:
- removed C500: 100 nF, 100V, X7R, C__Users_otto_Documents_AltiumLL_SamacSys.PcbLib:MAJx16, symbol Battman-altium-import:Repeat(Multiplexer,1,8)_1_MAJCH168BB7104KTEA01_SamacSys.S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
- removed IC500: ADG704BRMZ, C__Users_otto_Documents_AltiumLL_SamacSys.PcbLib:SOP50P490X110-10N, symbol Battman-altium-import:Repeat(Multiplexer,1,8)_0_ADG704BRMZ_SamacSys.SchLib
- removed JS500, JS501, JS502: SolderJumper, SolderJumper, symbol Battman-altium-import:Repeat(Multiplexer,1,8)_1_SolderJumper_SamacSys.SchLib
- added C500: 100 nF, 100V, X7R, C__Users_otto_Documents_AltiumLL_SamacSys.PcbLib:MAJx16, symbol Battman-altium-import:Repeat(Multiplexer,1,8)_1_MAJCH168BB7104KTEA01_SamacSys.S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
- added IC500: ADG704BRMZ, C__Users_otto_Documents_AltiumLL_SamacSys.PcbLib:SOP50P490X110-10N, symbol Battman-altium-import:Repeat(Multiplexer,1,8)_0_ADG704BRMZ_SamacSys.SchLib
- added JS500, JS501, JS502: SolderJumper, SolderJumper, symbol Battman-altium-import:Repeat(Multiplexer,1,8)_1_SolderJumper_SamacSys.SchLib

Commit message: kicad release
Parts:
- removed C500: 100 nF, 100V, X7R, C__Users_otto_Documents_AltiumLL_SamacSys.PcbLib:MAJx16, symbol Battman-altium-import:Repeat(Multiplexer,1,8)_1_MAJCH168BB7104KTEA01_SamacSys.S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
- removed IC500: ADG704BRMZ, C__Users_otto_Documents_AltiumLL_SamacSys.PcbLib:SOP50P490X110-10N, symbol Battman-altium-import:Repeat(Multiplexer,1,8)_0_ADG704BRMZ_SamacSys.SchLib
- removed JS500, JS501, JS502: SolderJumper, SolderJumper, symbol Battman-altium-import:Repeat(Multiplexer,1,8)_1_SolderJumper_SamacSys.SchLib
- added C500B: 100 nF, 100V, X7R, C__Users_otto_Documents_AltiumLL_SamacSys.PcbLib:MAJx16, symbol Battman-altium-import:Repeat(Multiplexer,1,8)_1_MAJCH168BB7104KTEA01_SamacSys.S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
- added IC500B: ADG704BRMZ, C__Users_otto_Documents_AltiumLL_SamacSys.PcbLib:SOP50P490X110-10N, symbol Battman-altium-import:Repeat(Multiplexer,1,8)_0_ADG704BRMZ_SamacSys.SchLib
- added JS500B (x3): SolderJumper, SolderJumper, symbol Battman-altium-import:Repeat(Multiplexer,1,8)_1_SolderJumper_SamacSys.SchLib
