File: Battman/KiCad/Battman/MCU.kicad_sch (KiCad schematic)
At the start: 52 parts, among them IC700 STM32L552RET6, IC701 TCAN1051HGVDRBRQ1, IC702 ESDA6V1-5SC6, J700 FTSH-105-01-F-D-RA-K, U700 1061TR, Y700 FC-135_32.7680KA-AG0

Commit message: Uopdated Schematics fixed
Parts:
- removed C701: 06031C103K4Z2A, C__Users_otto_Documents_AltiumLL_SamacSys.PcbLib:CAPC1608X90N, symbol Battman-altium-import:MCU_1_06031C103K4Z2A_SamacSys.SchLib
- removed C702, C706, C709, C711: CL10B475KQ8NQNC, C__Users_otto_Documents_AltiumLL_SamacSys.PcbLib:CAPC1608X95N, symbol Battman-altium-import:MCU_1_CL10B475KQ8NQNC_SamacSys.SchLib
- removed C703, C704, C705, C707, C710, C712: 0603YG104ZAT2A, C__Users_otto_Documents_AltiumLL_SamacSys.PcbLib:CAPC1608X90N, symbol Battman-altium-import:MCU_1_0603YG104ZAT2A_SamacSys.SchLib
- removed C708: 0603YG104ZAT2A, C__Users_otto_Documents_AltiumLL_SamacSys.PcbLib:CAPC1608X90N, symbol Battman-altium-import:MCU_0_0603YG104ZAT2A_SamacSys.SchLib
- removed J700: FTSH-105-01-F-D-RA-K, C__Users_otto_Documents_AltiumLL_SamacSys.PcbLib:FTSH-105-XX-YYY-D-RA-K, symbol Battman-altium-import:MCU_0_FTSH-105-01-F-D-RA-K_SamacSys.SchLib
- removed LED700: 150060GS75000, C__Users_otto_Documents_AltiumLL_SamacSys.PcbLib:LEDC1608X80N, symbol Battman-altium-import:MCU_1_150060GS75000_SamacSys.SchLib
- removed R700, R701, R702, R703: ${ALTIUM_VALUE}, C__Users_otto_Documents_AltiumLL_SamacSys.PcbLib:RESC1608X55N, symbol Battman-altium-import:MCU_1_CPF0603F60R4C1_SamacSys.SchLib
- added C701, C703, C704, C705, C707: 100 nF, 100V, X7R, C__Users_otto_Documents_AltiumLL_SamacSys.PcbLib:MAJx16, symbol Battman-altium-import:MCU_1_MAJCH168BB7104KTEA01_SamacSys.SchLib
- added C702, C706, C709, C711: 4.7uF, 10V, X7R, C__Users_otto_Documents_AltiumLL_SamacSys.PcbLib:GRM18x, symbol Battman-altium-import:MCU_1_GRM188Z71A475KE15J_SamacSys.SchLib
- added C708: 100 nF, 100V, X7R, C__Users_otto_Documents_AltiumLL_SamacSys.PcbLib:MAJx16, symbol Battman-altium-import:MCU_2_MAJCH168BB7104KTEA01_SamacSys.SchLib
- added C710, C712: 100nF 100V X5R, C__Users_otto_Documents_AltiumLL_SamacSys.PcbLib:CAPC1608X90N, symbol Battman-altium-import:MCU_1_HMK107BJ104KA-T_SamacSys.SchLib
- added J700: FTSH-105-01-F-D-K, C__Users_otto_Documents_AltiumLL_SamacSys.PcbLib:FTSH-105-XX-YYY-D-K, symbol Battman-altium-import:MCU_0_FTSH-105-01-F-D-K_SamacSys.SchLib
- added LED700: 150060VS75000, C__Users_otto_Documents_AltiumLL_SamacSys.PcbLib:LEDC1608X80N, symbol Battman-altium-import:MCU_1_150060VS75000_SamacSys.SchLib
- added R700, R701, R702, R703: 270R 1%, C__Users_otto_Documents_AltiumLL_SamacSys.PcbLib:RESC1608X55N, symbol Battman-altium-import:MCU_1_ERJ-3EKF2700V_SamacSys.SchLib
- C700: value 06035C105MAT2A -> 1uF 50V X7R
- C713: value 4.7nF 100V -> 4.7nF 100V X7R
- C714, C715: value 10pF -> 10pF 50V C0G
- R704, R705, R706, R712, R713, R714, R715, R716: value 22Ohm -> 22Ohm 1%; SUPPLIER 1 (none) -> Future Electronics; SUPPLIER PART NUMBER 1 (none) -> 8636706
- R707: value 22Ohm -> 22Ohm 1%; ALTIUM_VALUE 22Ohm -> 22Ohm 1%; SUPPLIER 1 (none) -> Future Electronics; SUPPLIER PART NUMBER 1 (none) -> 8636706
- R708, R709: value ${ALTIUM_VALUE} -> 60.4R, 1%; SUPPLIER 1 (none) -> Mouser; SUPPLIER PART NUMBER 1 (none) -> 279-CPF0603F60R4C1
- R710: SUPPLIER 1 (none) -> Mouser; SUPPLIER PART NUMBER 1 (none) -> 71-CRCW060310K0FKEI
- R711: value 5.1k -> 5.1k, 1%; SUPPLIER 1 (none) -> Mouser; SUPPLIER PART NUMBER 1 (none) -> 71-CRCW06035K10FKEBC
Connections:
- net 3V3_Stm: now also C701.2, C702.2, C703.2, C704.2, C705.2, C706.2, C707.2, C711.2, C712.2, J700.1
- net 5V_Stm: now also C709.2, C710.2
- net LED_A: now also R702.2
- net LED_G: now also R700.2
- net LED_R: now also R703.2
- net LED_Y: now also R701.2
- net RST: now also C708.1, J700.10
- net STM_GND: now also C701.1, C702.1, C703.1, C704.1, C705.1, C706.1, C707.1, C708.2, C709.1, C710.1, C711.1, C712.1, J700.3, J700.5, LED700.1 (K)
- net at R712.1: now also J700.2
- net at R713.1: now also J700.4
- net at R714.1: now also J700.6
- net at R715.1: now also J700.8
- net at LED701.2 (A): now also R701.1
- net at LED703.2 (A): now also R703.1
- net at LED702.2 (A): now also R702.1
- new net: LED700.2 (A), R700.1
Other:
- note added: "A2"
- note removed: "A1"

Commit message: Begin of kicad conversion
Parts:
- removed C700: 1uF 50V X7R, C__Users_otto_Documents_AltiumLL_SamacSys.PcbLib:CAPC1608X90N, symbol Battman-altium-import:MCU_1_06035C105MAT2A_SamacSys.SchLib
- removed C701, C703, C704, C705, C707: 100 nF, 100V, X7R, C__Users_otto_Documents_AltiumLL_SamacSys.PcbLib:MAJx16, symbol Battman-altium-import:MCU_1_MAJCH168BB7104KTEA01_SamacSys.SchLib
- removed C702, C706, C709, C711: 4.7uF, 10V, X7R, C__Users_otto_Documents_AltiumLL_SamacSys.PcbLib:GRM18x, symbol Battman-altium-import:MCU_1_GRM188Z71A475KE15J_SamacSys.SchLib
- removed C708: 100 nF, 100V, X7R, C__Users_otto_Documents_AltiumLL_SamacSys.PcbLib:MAJx16, symbol Battman-altium-import:MCU_2_MAJCH168BB7104KTEA01_SamacSys.SchLib
- removed C710, C712: 100nF 100V X5R, C__Users_otto_Documents_AltiumLL_SamacSys.PcbLib:CAPC1608X90N, symbol Battman-altium-import:MCU_1_HMK107BJ104KA-T_SamacSys.SchLib
- removed C713: 4.7nF 100V X7R, C__Users_otto_Documents_AltiumLL_SamacSys.PcbLib:CAPC1608X80N, symbol Battman-altium-import:MCU_0_C1608X7R2A472K080AA_SamacSys.SchLib
- removed C714, C715: 10pF 50V C0G, C__Users_otto_Documents_AltiumLL_SamacSys.PcbLib:CAPC1608X90N, symbol Battman-altium-import:MCU_2_06035A100BAT2A_SamacSys.SchLib
- removed D700: PESD2CANFD27V-TR, C__Users_otto_Documents_AltiumLL_SamacSys.PcbLib:SOT95P230X110-3N, symbol Battman-altium-import:MCU_3_PESD2CANFD27V-TR_SamacSys.SchLib
- removed FL700: ACE1V2012-121-R, C__Users_otto_Documents_AltiumLL_SamacSys.PcbLib:ACE1V2012121R, symbol Battman-altium-import:MCU_0_ACE1V2012-121-R_SamacSys.SchLib
- removed IC701: TCAN1051HGVDRBRQ1, C__Users_otto_Documents_AltiumLL_SamacSys.PcbLib:SON65P300X300X100-9N-D, symbol Battman-altium-import:MCU_0_TCAN1051HGVDRBRQ1_SamacSys.SchLib
- removed IC702: ESDA6V1-5SC6, C__Users_otto_Documents_AltiumLL_SamacSys.PcbLib:SOT95P280X145-6N, symbol Battman-altium-import:MCU_0_ESDA6V1-5SC6_SamacSys.SchLib
- removed J700: FTSH-105-01-F-D-K, C__Users_otto_Documents_AltiumLL_SamacSys.PcbLib:FTSH-105-XX-YYY-D-K, symbol Battman-altium-import:MCU_0_FTSH-105-01-F-D-K_SamacSys.SchLib
- removed JS700: SolderJumper, SolderJumper, symbol Battman-altium-import:MCU_0_SolderJumper_SamacSys.SchLib
- removed LED700: 150060VS75000, C__Users_otto_Documents_AltiumLL_SamacSys.PcbLib:LEDC1608X80N, symbol Battman-altium-import:MCU_1_150060VS75000_SamacSys.SchLib
- removed LED701: 150060YS75000, C__Users_otto_Documents_AltiumLL_SamacSys.PcbLib:LEDC1608X80N, symbol Battman-altium-import:MCU_1_150060YS75000_SamacSys.SchLib
- removed LED702: 150060AS75000, C__Users_otto_Documents_AltiumLL_SamacSys.PcbLib:LEDC1608X80N, symbol Battman-altium-import:MCU_1_150060AS75000_SamacSys.SchLib
- removed LED703: 150060RS75000, C__Users_otto_Documents_AltiumLL_SamacSys.PcbLib:LEDC1608X80N, symbol Battman-altium-import:MCU_1_150060RS75000_SamacSys.SchLib
- removed LS700: CPT-1625-80-SMT-TR, C__Users_otto_Documents_AltiumLL_SamacSys.PcbLib:CPT162580SMTTR, symbol Battman-altium-import:MCU_0_CPT-1625-80-SMT-TR_*
- removed R700, R701, R702, R703: 270R 1%, C__Users_otto_Documents_AltiumLL_SamacSys.PcbLib:RESC1608X55N, symbol Battman-altium-import:MCU_1_ERJ-3EKF2700V_SamacSys.SchLib
- removed R704, R705, R706, R707: 22Ohm 1%, C__Users_otto_Documents_AltiumLL_SamacSys.PcbLib:RESC1608X55N, symbol Battman-altium-import:MCU_0_mirrored_RC0603FR-0722RL_SamacSys.SchLib
- removed R708: 60.4R, 1%, C__Users_otto_Documents_AltiumLL_SamacSys.PcbLib:RESC1608X55N, symbol Battman-altium-import:MCU_0_CPF0603F60R4C1_SamacSys.SchLib
- removed R709: 60.4R, 1%, C__Users_otto_Documents_AltiumLL_SamacSys.PcbLib:RESC1608X55N, symbol Battman-altium-import:MCU_2_CPF0603F60R4C1_SamacSys.SchLib
- removed R710: CRCW060310K0FKEI, C__Users_otto_Documents_AltiumLL_SamacSys.PcbLib:RESC1608X50N, symbol Battman-altium-import:MCU_2_CRCW060310K0FKEI_SamacSys.SchLib
- removed R711: 5.1k, 1%, C__Users_otto_Documents_AltiumLL_SamacSys.PcbLib:RESC1608X55N, symbol Battman-altium-import:MCU_0_CRCW06035K10FKEBC_SamacSys.SchLib
- removed R712, R713, R714, R715, R716: 22Ohm 1%, C__Users_otto_Documents_AltiumLL_SamacSys.PcbLib:RESC1608X55N, symbol Battman-altium-import:MCU_0_RC0603FR-0722RL_SamacSys.SchLib
- removed S700: MJTP1140A, C__Users_otto_Documents_AltiumLL_SamacSys.PcbLib:MJTP1140A, symbol Battman-altium-import:MCU_0_MJTP1140A_SamacSys.SchLib
- removed S701: 218-4LPSTJ, C__Users_otto_Documents_AltiumLL_SamacSys.PcbLib:2184LPSTJ, symbol Battman-altium-import:MCU_0_mirrored_218-4LPSTJ_SamacSys.SchLib
- removed S702: CAS-120TA, C__Users_otto_Documents_AltiumLL_SamacSys.PcbLib:CAS120TA, symbol Battman-altium-import:MCU_0_CAS-120TA_SamacSys.SchLib
- removed S703: CAS-220TA, C__Users_otto_Documents_AltiumLL_SamacSys.PcbLib:CAS220TA, symbol Battman-altium-import:MCU_2_CAS-220TA_SamacSys.SchLib
- removed TP700: Test Pad 1mm, Test Pad 1mm-Footprint-1, symbol Battman-altium-import:MCU_3_Test Pad 1mm-Symbol-1_EPFL Racing Team
- removed U700: 1061TR, C__Users_otto_Documents_AltiumLL_SamacSys.PcbLib:1061TR, symbol Battman-altium-import:MCU_2_1061TR_SamacSys.SchLib
- removed Y700: FC-135_32.7680KA-AG0, C__Users_otto_Documents_AltiumLL_SamacSys.PcbLib:FC135327680KAAG0, symbol Battman-altium-import:MCU_1_FC-135_32.7680KA-AG0_SamacSys.SchLib
- added BT700: 3000TR, C__Users_otto_Documents_AltiumLL_SamacSys.PcbLib:3000TR, symbol Battman-altium-import:MCU_0_mirrored_3000TR_SamacSys.SchLib
- added C700: 1uF 50V X7R, C__Users_otto_Documents_AltiumLL_SamacSys.PcbLib:CAPC1608X90N, symbol Battman-altium-import:MCU_1_06035C105MAT2A_SamacSys.SchLib
- added C701, C703, C704, C705, C707: 100 nF, 100V, X7R, C__Users_otto_Documents_AltiumLL_SamacSys.PcbLib:MAJx16, symbol Battman-altium-import:MCU_1_MAJCH168BB7104KTEA01_SamacSys.SchLib
- added C702, C706: 4.7uF, 10V, X7R, C__Users_otto_Documents_AltiumLL_SamacSys.PcbLib:GRM18x, symbol Battman-altium-import:MCU_1_GRM188Z71A475KE15J_SamacSys.SchLib
- added C708: 100 nF, 100V, X7R, C__Users_otto_Documents_AltiumLL_SamacSys.PcbLib:MAJx16, symbol Battman-altium-import:MCU_2_MAJCH168BB7104KTEA01_SamacSys.SchLib
- added C709: 4.7uF, 10V, X7R, C__Users_otto_Documents_AltiumLL_SamacSys.PcbLib:GRM18x, symbol Battman-altium-import:MCU_1_mirrored_GRM188Z71A475KE15J_SamacSys.SchLib
- added C710: 100nF 100V X5R, C__Users_otto_Documents_AltiumLL_SamacSys.PcbLib:CAPC1608X90N, symbol Battman-altium-import:MCU_1_mirrored_HMK107BJ104KA-T_SamacSys.SchLib
- added C712: 100nF 100V X5R, C__Users_otto_Documents_AltiumLL_SamacSys.PcbLib:CAPC1608X90N, symbol Battman-altium-import:MCU_1_HMK107BJ104KA-T_SamacSys.SchLib
- added C713: 4.7nF 100V X7R, C__Users_otto_Documents_AltiumLL_SamacSys.PcbLib:CAPC1608X80N, symbol Battman-altium-import:MCU_0_C1608X7R2A472K080AA_SamacSys.SchLib
- added C714, C715: 10pF 50V C0G, C__Users_otto_Documents_AltiumLL_SamacSys.PcbLib:CAPC1608X90N, symbol Battman-altium-import:MCU_2_06035A100BAT2A_SamacSys.SchLib
- added D700: PESD2CANFD27V-TR, C__Users_otto_Documents_AltiumLL_SamacSys.PcbLib:SOT95P230X110-3N, symbol Battman-altium-import:MCU_3_PESD2CANFD27V-TR_SamacSys.SchLib
- added FB700: 742792097, FP-742792097-MFG, symbol Battman-altium-import:MCU_1_5f30dd21d616792df468990f7003faa_Altium Content Vault
- added FL700: ACE1V2012-121-R, C__Users_otto_Documents_AltiumLL_SamacSys.PcbLib:ACE1V2012121R, symbol Battman-altium-import:MCU_0_ACE1V2012-121-R_SamacSys.SchLib
- added unit 3 of IC700
- added IC701: ISO1044BDR, C__Users_otto_Documents_AltiumLL_SamacSys.PcbLib:SOIC127P600X175-8N, symbol Battman-altium-import:MCU_0_ISO1044BDR_SamacSys.SchLib
- added IC702: ESDA6V1-5SC6, C__Users_otto_Documents_AltiumLL_SamacSys.PcbLib:SOT95P280X145-6N, symbol Battman-altium-import:MCU_0_mirrored_ESDA6V1-5SC6_SamacSys.SchLib
- added J700: FTSH-105-01-L-DV-K, C__Users_otto_Documents_AltiumLL_SamacSys.PcbLib:FTSH10501LDVK, symbol Battman-altium-import:MCU_0_FTSH-105-01-L-DV-K_SamacSys.SchLib
- added JS700: SolderJumper, SolderJumper, symbol Battman-altium-import:MCU_0_SolderJumper_SamacSys.SchLib
- added LED700: 150060VS75000, C__Users_otto_Documents_AltiumLL_SamacSys.PcbLib:LEDC1608X80N, symbol Battman-altium-import:MCU_1_150060VS75000_SamacSys.SchLib
- added LED701: 150060YS75000, C__Users_otto_Documents_AltiumLL_SamacSys.PcbLib:LEDC1608X80N, symbol Battman-altium-import:MCU_1_150060YS75000_SamacSys.SchLib
- added LED702: 150060AS75000, C__Users_otto_Documents_AltiumLL_SamacSys.PcbLib:LEDC1608X80N, symbol Battman-altium-import:MCU_1_150060AS75000_SamacSys.SchLib
- added LED703: 150060RS75000, C__Users_otto_Documents_AltiumLL_SamacSys.PcbLib:LEDC1608X80N, symbol Battman-altium-import:MCU_1_150060RS75000_SamacSys.SchLib
- added LS700: CPT-1625-80-SMT-TR, C__Users_otto_Documents_AltiumLL_SamacSys.PcbLib:CPT162580SMTTR, symbol Battman-altium-import:MCU_0_CPT-1625-80-SMT-TR_*
- added R700, R701, R702, R703: 270R 1%, C__Users_otto_Documents_AltiumLL_SamacSys.PcbLib:RESC1608X55N, symbol Battman-altium-import:MCU_1_ERJ-3EKF2700V_SamacSys.SchLib
- added R704, R705, R706, R707: 22Ohm 1%, C__Users_otto_Documents_AltiumLL_SamacSys.PcbLib:RESC1608X55N, symbol Battman-altium-import:MCU_1_RC0603FR-0722RL_SamacSys.SchLib
- added R708: 60.4R, 1%, C__Users_otto_Documents_AltiumLL_SamacSys.PcbLib:RESC1608X55N, symbol Battman-altium-import:MCU_0_CPF0603F60R4C1_SamacSys.SchLib
- added R709: 60.4R, 1%, C__Users_otto_Documents_AltiumLL_SamacSys.PcbLib:RESC1608X55N, symbol Battman-altium-import:MCU_2_CPF0603F60R4C1_SamacSys.SchLib
- added R711: 5.1k, 1%, C__Users_otto_Documents_AltiumLL_SamacSys.PcbLib:RESC1608X55N, symbol Battman-altium-import:MCU_0_CRCW06035K10FKEBC_SamacSys.SchLib
- added R712, R713, R714, R715, R716: 22Ohm 1%, C__Users_otto_Documents_AltiumLL_SamacSys.PcbLib:RESC1608X55N, symbol Battman-altium-import:MCU_0_RC0603FR-0722RL_SamacSys.SchLib
- added S700: MJTP1140A, C__Users_otto_Documents_AltiumLL_SamacSys.PcbLib:MJTP1140A, symbol Battman-altium-import:MCU_0_MJTP1140A_SamacSys.SchLib
- added S701: 218-4LPSTJ, C__Users_otto_Documents_AltiumLL_SamacSys.PcbLib:2184LPSTJ, symbol Battman-altium-import:MCU_1_218-4LPSTJ_SamacSys.SchLib
- added S702: CAS-120TA, C__Users_otto_Documents_AltiumLL_SamacSys.PcbLib:CAS120TA, symbol Battman-altium-import:MCU_0_CAS-120TA_SamacSys.SchLib
- added S703: CAS-220TA, C__Users_otto_Documents_AltiumLL_SamacSys.PcbLib:CAS220TA, symbol Battman-altium-import:MCU_2_CAS-220TA_SamacSys.SchLib
- added TP700, TP706: Testpoint, Testpoint, symbol Battman-altium-import:MCU_3_Testpoint_SamacSys.SchLib
- added TP705: Testpoint, Testpoint, symbol Battman-altium-import:MCU_1_Testpoint_SamacSys.SchLib
- added Y700: FC-135_32.7680KA-AG0, C__Users_otto_Documents_AltiumLL_SamacSys.PcbLib:FC135327680KAAG0, symbol Battman-altium-import:MCU_1_FC-135_32.7680KA-AG0_SamacSys.SchLib
Connections:
- net Currents/DischgCurrent is gone; now on net WDT_STM: IC700.8 (PC0)
- net Currents/DischgRef is gone; now on net ~{HardwareFault}: IC700.9 (PC1)
- net LTC_H_Config/A1_2 is gone; now on net LED_G: IC700.34 (PB13)
- net LTC_H_Config/A1_3 is gone; now on net LED_Y: IC700.33 (PB12)
- net LTC_H_Config/A1_4 is gone; now on net LED_R: IC700.30 (PB11)
- net LTC_H_Config/A1_5 is gone; now on net LED_A: IC700.29 (PB10)
- net LTC_H_Config/A1_6 is gone; now on net ~{ErrorReset}: IC700.27 (PB1)
- net LTC_H_Config/A1_7 is gone; now on net DischgEn: IC700.26 (PB0)
- net LTC_H_Config/A1_8 is gone; now on net OutputEnable: IC700.25 (PC5)
- net 3V3_Stm: no longer IC700.13 (VDDA/VREF+)
- net CAN_N: now also S703.2 (COM_1)
- net CAN_P: now also S703.5 (COM_2)
- net ChargeEn: now also IC700.24 (PC4); no longer IC700.14 (PA0)
- net DischgEn: no longer IC700.15 (PA1)
- net LED_A: no longer IC700.57 (PB5)
- net LED_G: no longer IC700.59 (PB7)
- net LED_R: no longer IC700.56 (PB4)
- net LED_Y: no longer IC700.58 (PB6)
- net LTC_Selftest: now also IC700.15 (PA1); no longer IC700.16 (PA2)
- net LTC_SelftestOK: now also IC700.14 (PA0); no longer IC700.17 (PA3)
- net OutputEnable: no longer IC700.6 (PH1-OSC_OUT)
- net WDT_STM: no longer IC700.2 (PC13)
- net ~{ErrorReset}: no longer IC700.5 (PH0-OSC_IN)
- net ~{HardwareFault}: no longer IC700.24 (PC4)
- net Currents/ChgCurrent: no longer names the net of IC700.10 (PC2)
- net Currents/ChgRef: no longer names the net of IC700.11 (PC3)
- removed net LTC_H_Config/A0_1: IC700.43 (PA10)
- removed net LTC_H_Config/A0_2: IC700.42 (PA9)
- removed net LTC_H_Config/A0_3: IC700.41 (PA8)
- removed net LTC_H_Config/A0_4: IC700.40 (PC9)
- removed net LTC_H_Config/A0_5: IC700.39 (PC8)
- net LTC_H_Config/A0_6: no longer names the net of IC700.38 (PC7)
- net LTC_H_Config/A0_7: no longer names the net of IC700.37 (PC6)
- net LTC_H_Config/A0_8: no longer names the net of IC700.36 (PB15)
- net LTC_H_Config/A1_1: no longer names the net of IC700.35 (PB14)
- net SPI_LTC/CS: no longer names the net of IC700.20 (PA4)
- net SPI_LTC/MISO: no longer names the net of IC700.22 (PA6)
- net SPI_LTC/MOSI: no longer names the net of IC700.23 (PA7)
- net SPI_LTC/SCK: no longer names the net of IC700.21 (PA5)
- new net 3V3A_Stm: IC700.13 (VDDA/VREF+)
- no-connect marks 4 -> 5
Other:
- removed sheet Currents
- removed sheet LTC_H_Config
- removed sheet SPI_LTC
- note added: "A3"
- note added: "CR1225(3V)"
- note removed: "A2"
- note removed: "CR2032(3V)"

Commit message: kicad release
Parts:
- removed C710: 100nF 100V X5R, C__Users_otto_Documents_AltiumLL_SamacSys.PcbLib:CAPC1608X90N, symbol Battman-altium-import:MCU_1_mirrored_HMK107BJ104KA-T_SamacSys.SchLib
- removed C712: 100nF 100V X5R, C__Users_otto_Documents_AltiumLL_SamacSys.PcbLib:CAPC1608X90N, symbol Battman-altium-import:MCU_1_HMK107BJ104KA-T_SamacSys.SchLib
- added C710, C712: 100 nF, 100V, X7R, C__Users_otto_Documents_AltiumLL_SamacSys.PcbLib:MAJx16, symbol Battman-altium-import:MCU_1_MAJCH168BB7104KTEA01_SamacSys.SchLib
- R707: ALTIUM_VALUE 22Ohm 1% -> 22Ohm
Connections:
- net Current1: now reaches IC700.10 (PC2)
- net CurrRef1: now reaches IC700.11 (PC3)
- net Current2: now reaches IC700.16 (PA2)
- net CurrRef2: now reaches IC700.17 (PA3)
- net CS: now reaches IC700.20 (PA4)
- net SCK: now reaches IC700.21 (PA5)
- net MISO: now reaches IC700.22 (PA6)
- net MOSI: now reaches IC700.23 (PA7)
