File: Battman/KiCad/Battman/PowerPath.kicad_sch (KiCad schematic)
At the start: 4 parts, among them IC900 CD4044BDR

Commit message: Uopdated Schematics fixed
Parts:
- removed C900: 0603YG104ZAT2A, C__Users_otto_Documents_AltiumLL_SamacSys.PcbLib:CAPC1608X90N, symbol Battman-altium-import:PowerPath_0_0603YG104ZAT2A_SamacSys.SchLib
- added C900: 100 nF, 100V, X7R, C__Users_otto_Documents_AltiumLL_SamacSys.PcbLib:MAJx16, symbol Battman-altium-import:PowerPath_0_MAJCH168BB7104KTEA01_SamacSys.SchLib
- R900: ALTIUM_VALUE 10k -> 10k, 1%; SUPPLIER 1 (none) -> Mouser; SUPPLIER PART NUMBER 1 (none) -> 71-CRCW060310K0FKEI
Connections:
- net 3.3V: now also C900.1
- net GND: now also C900.2
Other:
- note added: "A1"
- note removed: "A0"

Commit message: Begin of kicad conversion
Parts:
- removed C900: 100 nF, 100V, X7R, C__Users_otto_Documents_AltiumLL_SamacSys.PcbLib:MAJx16, symbol Battman-altium-import:PowerPath_0_MAJCH168BB7104KTEA01_SamacSys.SchLib
- removed IC900: CD4044BDR, C__Users_otto_Documents_AltiumLL_SamacSys.PcbLib:SOIC127P600X175-16N, symbol Battman-altium-import:PowerPath_0_CD4044BDR_SamacSys.SchLib
- removed R900: CRCW060310K0FKEI, C__Users_otto_Documents_AltiumLL_SamacSys.PcbLib:RESC1608X50N, symbol Battman-altium-import:PowerPath_0_CRCW060310K0FKEI_SamacSys.SchLib
- removed TP900: Test Pad 1mm, Test Pad 1mm-Footprint-1, symbol Battman-altium-import:PowerPath_3_Test Pad 1mm-Symbol-1_EPFL Racing Team
- added C900: 100 nF, 100V, X7R, C__Users_otto_Documents_AltiumLL_SamacSys.PcbLib:MAJx16, symbol Battman-altium-import:PowerPath_0_MAJCH168BB7104KTEA01_SamacSys.SchLib
- added IC900: SN74LVC2G74DCUTE4, C__Users_otto_Documents_AltiumLL_SamacSys.PcbLib:SOP50P310X90-8N, symbol Battman-altium-import:PowerPath_0_SN74LVC2G74DCUTE4_SamacSys.SchLib
- added R900: CRCW060310K0FKEI, C__Users_otto_Documents_AltiumLL_SamacSys.PcbLib:RESC1608X50N, symbol Battman-altium-import:PowerPath_0_CRCW060310K0FKEI_SamacSys.SchLib
- added TP900: Testpoint, Testpoint, symbol Battman-altium-import:PowerPath_3_Testpoint_SamacSys.SchLib
Connections:
- no-connect marks 4 -> 1
Other:
- removed sheet Currents
- note added: "A2"
- note removed: "A1"

Commit message: kicad release
Other:
- removed sheet Repeat(SinglePath,1,2)
- added sheet SinglePath1 (Singlepath.kicad_sch)
- added sheet SinglePath2 (Singlepath.kicad_sch)
