File: Battman/KiCad/Battman/Singlepath.kicad_sch (KiCad schematic)
At the start: 17 parts, among them IC800 ACS37002KMABTR-050B3, IC801 LTC7000EMSE#PBF, Q800 SQJQ160E-T1_GE3, Q801 QJQ160E-T1_GE3

Commit message: Uopdated Schematics fixed
Parts:
- removed C800: 220nF 100V, C__Users_otto_Documents_AltiumLL_SamacSys.PcbLib:CAPC3216X180N, symbol Battman-altium-import:Repeat(SinglePath,1,2)_2_GRM31C5C1H224JE02L_SamacSys.SchL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
- removed C802: 0603YG104ZAT2A, C__Users_otto_Documents_AltiumLL_SamacSys.PcbLib:CAPC1608X90N, symbol Battman-altium-import:Repeat(SinglePath,1,2)_2_0603YG104ZAT2A_SamacSys.SchLib
- removed C803: 100nF 100V, C__Users_otto_Documents_AltiumLL_SamacSys.PcbLib:CAPC1608X90N, symbol Battman-altium-import:Repeat(SinglePath,1,2)_1_HMK107BJ104KA-T_SamacSys.SchLib
- removed F800: 3555, C__Users_otto_Documents_AltiumLL_SamacSys.PcbLib:3555, symbol Battman-altium-import:Repeat(SinglePath,1,2)_0_3555_SamacSys.SchLib
- removed LED800: 150060GS75000, C__Users_otto_Documents_AltiumLL_SamacSys.PcbLib:LEDC1608X80N, symbol Battman-altium-import:Repeat(SinglePath,1,2)_2_150060GS75000_SamacSys.SchLib
- added C800, C803: 100 nF, 100V, X7R, C__Users_otto_Documents_AltiumLL_SamacSys.PcbLib:MAJx16, symbol Battman-altium-import:Repeat(SinglePath,1,2)_1_MAJCH168BB7104KTEA01_SamacSys.Sc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
- added C802: 680nF, 35V, X7R, C__Users_otto_Documents_AltiumLL_SamacSys.PcbLib:CAPC1608X90N, symbol Battman-altium-import:Repeat(SinglePath,1,2)_0_CGA3E1X7R1V684K080AC_SamacSys.Sc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
- added C804: 1uF 50V X7R, C__Users_otto_Documents_AltiumLL_SamacSys.PcbLib:CAPC1608X90N, symbol Battman-altium-import:Repeat(SinglePath,1,2)_1_06035C105MAT2A_SamacSys.SchLib
- added LED800: 150060VS75000, C__Users_otto_Documents_AltiumLL_SamacSys.PcbLib:LEDC1608X80N, symbol Battman-altium-import:Repeat(SinglePath,1,2)_2_150060VS75000_SamacSys.SchLib
- C801: value 06035C105MAT2A -> 1uF 50V X7R
- R800: value 3k3 -> 3k3 1%; SUPPLIER 1 (none) -> Avnet; SUPPLIER PART NUMBER 1 (none) -> 46AK9312
Connections:
- net 3.3V: now also C800.2, C804.2
- net Battery: now also IC800.5 (IP-_1), IC800.6 (IP-_2), IC800.7 (IP-_3), IC800.8 (IP-_4)
- net BatteryFused: now also C803.2
- net GND: now also C800.1, C803.1, C804.1, LED800.1 (K)
- net TS: now also C802.2
- net at R800.2: now also LED800.2 (A)
- net at IC801.14 (BST): now also C802.1
Other:
- note added: "A2"
- note removed: "A1"

Commit message: Begin of kicad conversion
Parts:
- removed C800, C803: 100 nF, 100V, X7R, C__Users_otto_Documents_AltiumLL_SamacSys.PcbLib:MAJx16, symbol Battman-altium-import:Repeat(SinglePath,1,2)_1_MAJCH168BB7104KTEA01_SamacSys.Sc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
- removed C801, C804: 1uF 50V X7R, C__Users_otto_Documents_AltiumLL_SamacSys.PcbLib:CAPC1608X90N, symbol Battman-altium-import:Repeat(SinglePath,1,2)_1_06035C105MAT2A_SamacSys.SchLib
- removed C802: 680nF, 35V, X7R, C__Users_otto_Documents_AltiumLL_SamacSys.PcbLib:CAPC1608X90N, symbol Battman-altium-import:Repeat(SinglePath,1,2)_0_CGA3E1X7R1V684K080AC_SamacSys.Sc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
- removed IC800: ACS37002KMABTR-050B3, C__Users_otto_Documents_AltiumLL_SamacSys.PcbLib:SOIC127P1030X265-16N, symbol Battman-altium-import:Repeat(SinglePath,1,2)_3_ACS37002KMABTR-050B3_SamacSys.Sc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
- removed IC801: LTC7000EMSE#PBF, C__Users_otto_Documents_AltiumLL_SamacSys.PcbLib:SOP50P490X110-17N, symbol Battman-altium-import:Repeat(SinglePath,1,2)_0_LTC7000EMSE#PBF_SamacSys.SchLib
- removed LED800: 150060VS75000, C__Users_otto_Documents_AltiumLL_SamacSys.PcbLib:LEDC1608X80N, symbol Battman-altium-import:Repeat(SinglePath,1,2)_2_150060VS75000_SamacSys.SchLib
- removed Q800: SQJQ160E-T1_GE3, C__Users_otto_Documents_AltiumLL_SamacSys.PcbLib:SQJQ160ET1_GE3, symbol Battman-altium-import:Repeat(SinglePath,1,2)_1_SQJQ160E-T1_GE3_SamacSys.SchLib
- removed Q801: QJQ160E-T1_GE3, C__Users_otto_Documents_AltiumLL_SamacSys.PcbLib:SQJQ160ET1_GE3, symbol Battman-altium-import:Repeat(SinglePath,1,2)_1_mirrored_SQJQ160E-T1_GE3_SamacSy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
- removed R800: 3k3 1%, C__Users_otto_Documents_AltiumLL_SamacSys.PcbLib:RESC1608X55N, symbol Battman-altium-import:Repeat(SinglePath,1,2)_0_CRGH0603F3K3_SamacSys.SchLib
- removed R801, R802: 0Ohm, C__Users_otto_Documents_AltiumLL_SamacSys.PcbLib:RESC1608X50N, symbol Battman-altium-import:Repeat(SinglePath,1,2)_1_CRCW06030000Z0EC_SamacSys.SchLib
- removed R803, R804: 0Ohm, C__Users_otto_Documents_AltiumLL_SamacSys.PcbLib:RESC1608X50N, symbol Battman-altium-import:Repeat(SinglePath,1,2)_0_CRCW06030000Z0EC_SamacSys.SchLib
- removed TP800: Test Pad 1mm, Test Pad 1mm-Footprint-1, symbol Battman-altium-import:Repeat(SinglePath,1,2)_2_Test Pad 1mm-Symbol-1_EPFL Racin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
- removed TP801: Test Pad 1mm, Test Pad 1mm-Footprint-1, symbol Battman-altium-import:Repeat(SinglePath,1,2)_0_Test Pad 1mm-Symbol-1_EPFL Racin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
- added C800, C803, C805: 100 nF, 100V, X7R, C__Users_otto_Documents_AltiumLL_SamacSys.PcbLib:MAJx16, symbol Battman-altium-import:Repeat(SinglePath,1,2)_1_MAJCH168BB7104KTEA01_SamacSys.Sc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
- added C801, C804: 1uF 50V X7R, C__Users_otto_Documents_AltiumLL_SamacSys.PcbLib:CAPC1608X90N, symbol Battman-altium-import:Repeat(SinglePath,1,2)_1_06035C105MAT2A_SamacSys.SchLib
- added C802: 680nF, 35V, X7R, C__Users_otto_Documents_AltiumLL_SamacSys.PcbLib:CAPC1608X90N, symbol Battman-altium-import:Repeat(SinglePath,1,2)_0_CGA3E1X7R1V684K080AC_SamacSys.Sc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
- added D800: SMBJ43A, C__Users_otto_Documents_AltiumLL_SamacSys.PcbLib:DIOM5436X244N, symbol Battman-altium-import:Repeat(SinglePath,1,2)_3_SMBJ43A_*
- added IC800: ACS37002KMABTR-050B3, C__Users_otto_Documents_AltiumLL_SamacSys.PcbLib:SOIC127P1030X265-16N, symbol Battman-altium-import:Repeat(SinglePath,1,2)_1_ACS37002KMABTR-050B3_SamacSys.Sc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
- added IC801: LTC7000EMSE#PBF, C__Users_otto_Documents_AltiumLL_SamacSys.PcbLib:SOP50P490X110-17N, symbol Battman-altium-import:Repeat(SinglePath,1,2)_0_LTC7000EMSE#PBF_SamacSys.SchLib
- added LED800: 150060VS75000, C__Users_otto_Documents_AltiumLL_SamacSys.PcbLib:LEDC1608X80N, symbol Battman-altium-import:Repeat(SinglePath,1,2)_2_150060VS75000_SamacSys.SchLib
- added Q800: SQJQ160E-T1_GE3, C__Users_otto_Documents_AltiumLL_SamacSys.PcbLib:SQJQ160ET1_GE3, symbol Battman-altium-import:Repeat(SinglePath,1,2)_1_SQJQ160E-T1_GE3_SamacSys.SchLib
- added Q801: SQJQ160E-T1_GE3, C__Users_otto_Documents_AltiumLL_SamacSys.PcbLib:SQJQ160ET1_GE3, symbol Battman-altium-import:Repeat(SinglePath,1,2)_1_mirrored_SQJQ160E-T1_GE3_SamacSy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
- added R800: 3.3k 0.5% 0.5W, C__Users_otto_Documents_AltiumLL_SamacSys.PcbLib:ERJP06D1000V, symbol Battman-altium-import:Repeat(SinglePath,1,2)_0_ERJ-P06J332V_*
- added R801, R802: 0Ohm, C__Users_otto_Documents_AltiumLL_SamacSys.PcbLib:RESC1608X50N, symbol Battman-altium-import:Repeat(SinglePath,1,2)_1_CRCW06030000Z0EC_SamacSys.SchLib
- added R803, R804: 0Ohm, C__Users_otto_Documents_AltiumLL_SamacSys.PcbLib:RESC1608X50N, symbol Battman-altium-import:Repeat(SinglePath,1,2)_0_CRCW06030000Z0EC_SamacSys.SchLib
- added R805: 200uOhm 3W 1%, C__Users_otto_Documents_AltiumLL_SamacSys.PcbLib:RESC10052X63N, symbol Battman-altium-import:Repeat(SinglePath,1,2)_0_PU3921FKN130U2L_*
- added R806: 100R, 1%, C__Users_otto_Documents_AltiumLL_SamacSys.PcbLib:RESC1608X50N, symbol Battman-altium-import:Repeat(SinglePath,1,2)_0_CRCW0603100RFKEA_SamacSys.SchLib
- added R807: 40k 0.1%, C__Users_otto_Documents_AltiumLL_SamacSys.PcbLib:RESC1608X55N, symbol Battman-altium-import:Repeat(SinglePath,1,2)_1_AT0603BRD0740KL_*
- added TP800, TP801: Testpoint, Testpoint, symbol Battman-altium-import:Repeat(SinglePath,1,2)_2_Testpoint_SamacSys.SchLib
- added TP802: Testpoint, Testpoint, symbol Battman-altium-import:Repeat(SinglePath,1,2)_0_Testpoint_SamacSys.SchLib
Connections:
- no-connect marks 5 -> 1
Other:
- note added: "A3"
- note removed: "A2"

Commit message: kicad release
Parts:
- removed C800, C803, C805: 100 nF, 100V, X7R, C__Users_otto_Documents_AltiumLL_SamacSys.PcbLib:MAJx16, symbol Battman-altium-import:Repeat(SinglePath,1,2)_1_MAJCH168BB7104KTEA01_SamacSys.Sc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
- removed C801, C804: 1uF 50V X7R, C__Users_otto_Documents_AltiumLL_SamacSys.PcbLib:CAPC1608X90N, symbol Battman-altium-import:Repeat(SinglePath,1,2)_1_06035C105MAT2A_SamacSys.SchLib
- removed C802: 680nF, 35V, X7R, C__Users_otto_Documents_AltiumLL_SamacSys.PcbLib:CAPC1608X90N, symbol Battman-altium-import:Repeat(SinglePath,1,2)_0_CGA3E1X7R1V684K080AC_SamacSys.Sc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
- removed D800: SMBJ43A, C__Users_otto_Documents_AltiumLL_SamacSys.PcbLib:DIOM5436X244N, symbol Battman-altium-import:Repeat(SinglePath,1,2)_3_SMBJ43A_*
- removed IC800: ACS37002KMABTR-050B3, C__Users_otto_Documents_AltiumLL_SamacSys.PcbLib:SOIC127P1030X265-16N, symbol Battman-altium-import:Repeat(SinglePath,1,2)_1_ACS37002KMABTR-050B3_SamacSys.Sc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
- removed IC801: LTC7000EMSE#PBF, C__Users_otto_Documents_AltiumLL_SamacSys.PcbLib:SOP50P490X110-17N, symbol Battman-altium-import:Repeat(SinglePath,1,2)_0_LTC7000EMSE#PBF_SamacSys.SchLib
- removed LED800: 150060VS75000, C__Users_otto_Documents_AltiumLL_SamacSys.PcbLib:LEDC1608X80N, symbol Battman-altium-import:Repeat(SinglePath,1,2)_2_150060VS75000_SamacSys.SchLib
- removed Q800: SQJQ160E-T1_GE3, C__Users_otto_Documents_AltiumLL_SamacSys.PcbLib:SQJQ160ET1_GE3, symbol Battman-altium-import:Repeat(SinglePath,1,2)_1_SQJQ160E-T1_GE3_SamacSys.SchLib
- removed Q801: SQJQ160E-T1_GE3, C__Users_otto_Documents_AltiumLL_SamacSys.PcbLib:SQJQ160ET1_GE3, symbol Battman-altium-import:Repeat(SinglePath,1,2)_1_mirrored_SQJQ160E-T1_GE3_SamacSy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
- removed R800: 3.3k 0.5% 0.5W, C__Users_otto_Documents_AltiumLL_SamacSys.PcbLib:ERJP06D1000V, symbol Battman-altium-import:Repeat(SinglePath,1,2)_0_ERJ-P06J332V_*
- removed R801, R802: 0Ohm, C__Users_otto_Documents_AltiumLL_SamacSys.PcbLib:RESC1608X50N, symbol Battman-altium-import:Repeat(SinglePath,1,2)_1_CRCW06030000Z0EC_SamacSys.SchLib
- removed R803, R804: 0Ohm, C__Users_otto_Documents_AltiumLL_SamacSys.PcbLib:RESC1608X50N, symbol Battman-altium-import:Repeat(SinglePath,1,2)_0_CRCW06030000Z0EC_SamacSys.SchLib
- removed R805: 200uOhm 3W 1%, C__Users_otto_Documents_AltiumLL_SamacSys.PcbLib:RESC10052X63N, symbol Battman-altium-import:Repeat(SinglePath,1,2)_0_PU3921FKN130U2L_*
- removed R806: 100R, 1%, C__Users_otto_Documents_AltiumLL_SamacSys.PcbLib:RESC1608X50N, symbol Battman-altium-import:Repeat(SinglePath,1,2)_0_CRCW0603100RFKEA_SamacSys.SchLib
- removed R807: 40k 0.1%, C__Users_otto_Documents_AltiumLL_SamacSys.PcbLib:RESC1608X55N, symbol Battman-altium-import:Repeat(SinglePath,1,2)_1_AT0603BRD0740KL_*
- removed TP800, TP801: Testpoint, Testpoint, symbol Battman-altium-import:Repeat(SinglePath,1,2)_2_Testpoint_SamacSys.SchLib
- removed TP802: Testpoint, Testpoint, symbol Battman-altium-import:Repeat(SinglePath,1,2)_0_Testpoint_SamacSys.SchLib
- added C800A, C803A, C805A: 100 nF, 100V, X7R, C__Users_otto_Documents_AltiumLL_SamacSys.PcbLib:MAJx16, symbol Battman-altium-import:Repeat(SinglePath,1,2)_1_MAJCH168BB7104KTEA01_SamacSys.Sc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
- added C801A, C804A: 1uF 50V X7R, C__Users_otto_Documents_AltiumLL_SamacSys.PcbLib:CAPC1608X90N, symbol Battman-altium-import:Repeat(SinglePath,1,2)_1_06035C105MAT2A_SamacSys.SchLib
- added C802A: 680nF, 35V, X7R, C__Users_otto_Documents_AltiumLL_SamacSys.PcbLib:CAPC1608X90N, symbol Battman-altium-import:Repeat(SinglePath,1,2)_0_CGA3E1X7R1V684K080AC_SamacSys.Sc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
- added D800A: SMBJ43A, C__Users_otto_Documents_AltiumLL_SamacSys.PcbLib:DIOM5436X244N, symbol Battman-altium-import:Repeat(SinglePath,1,2)_3_SMBJ43A_*
- added IC800A: ACS37002KMABTR-050B3, C__Users_otto_Documents_AltiumLL_SamacSys.PcbLib:SOIC127P1030X265-16N, symbol Battman-altium-import:Repeat(SinglePath,1,2)_1_ACS37002KMABTR-050B3_SamacSys.Sc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
- added IC801A: LTC7000EMSE#PBF, C__Users_otto_Documents_AltiumLL_SamacSys.PcbLib:SOP50P490X110-17N, symbol Battman-altium-import:Repeat(SinglePath,1,2)_0_LTC7000EMSE#PBF_SamacSys.SchLib
- added LED800A: 150060VS75000, C__Users_otto_Documents_AltiumLL_SamacSys.PcbLib:LEDC1608X80N, symbol Battman-altium-import:Repeat(SinglePath,1,2)_2_150060VS75000_SamacSys.SchLib
- added Q800A: SQJQ160E-T1_GE3, C__Users_otto_Documents_AltiumLL_SamacSys.PcbLib:SQJQ160ET1_GE3, symbol Battman-altium-import:Repeat(SinglePath,1,2)_1_SQJQ160E-T1_GE3_SamacSys.SchLib
- added Q801A: SQJQ160E-T1_GE3, C__Users_otto_Documents_AltiumLL_SamacSys.PcbLib:SQJQ160ET1_GE3, symbol Battman-altium-import:Repeat(SinglePath,1,2)_1_mirrored_SQJQ160E-T1_GE3_SamacSy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
- added R800A: 3.3k 0.5% 0.5W, C__Users_otto_Documents_AltiumLL_SamacSys.PcbLib:ERJP06D1000V, symbol Battman-altium-import:Repeat(SinglePath,1,2)_0_ERJ-P06J332V_*
- added R801A, R802A: 0Ohm, C__Users_otto_Documents_AltiumLL_SamacSys.PcbLib:RESC1608X50N, symbol Battman-altium-import:Repeat(SinglePath,1,2)_1_CRCW06030000Z0EC_SamacSys.SchLib
- added R803A, R804A: 0Ohm, C__Users_otto_Documents_AltiumLL_SamacSys.PcbLib:RESC1608X50N, symbol Battman-altium-import:Repeat(SinglePath,1,2)_0_CRCW06030000Z0EC_SamacSys.SchLib
- added R805A: 200uOhm 3W 1%, C__Users_otto_Documents_AltiumLL_SamacSys.PcbLib:RESC10052X63N, symbol Battman-altium-import:Repeat(SinglePath,1,2)_0_PU3921FKN130U2L_*
- added R806A: 100R, 1%, C__Users_otto_Documents_AltiumLL_SamacSys.PcbLib:RESC1608X50N, symbol Battman-altium-import:Repeat(SinglePath,1,2)_0_CRCW0603100RFKEA_SamacSys.SchLib
- added R807A: 40k 0.1%, C__Users_otto_Documents_AltiumLL_SamacSys.PcbLib:RESC1608X55N, symbol Battman-altium-import:Repeat(SinglePath,1,2)_1_AT0603BRD0740KL_*
- added TP800A, TP801A: Testpoint, Testpoint, symbol Battman-altium-import:Repeat(SinglePath,1,2)_2_Testpoint_SamacSys.SchLib
- added TP802A: Testpoint, Testpoint, symbol Battman-altium-import:Repeat(SinglePath,1,2)_0_Testpoint_SamacSys.SchLib
