File: Battman/KiCad/Battman/cell_inputfilter.kicad_sch (KiCad schematic)
At the start: 1 part

Commit message: Begin of kicad conversion
Parts:
- removed F100: 0466.250NR, C__Users_otto_Documents_AltiumLL_SamacSys.PcbLib:FUSC3215X66N, symbol Battman-altium-import:CellFilter_0_0466.250NR_SamacSys.SchLib
- added F100: 0466.250NR, C__Users_otto_Documents_AltiumLL_SamacSys.PcbLib:FUSC3215X66N, symbol Battman-altium-import:CellFilter_0_0466.250NR_SamacSys.SchLib
Connections:
- no-connect marks 0 -> 1
Other:
- removed sheet 
- removed sheet CellTaps
- removed sheet Software Protection Taps
- sheet CellFilter1 ports: added Cell+_Fused; removed none
- sheet CellFilter10 ports: added Cell+_Fused; removed none
- sheet CellFilter2 ports: added Cell+_Fused; removed none
- sheet CellFilter3 ports: added Cell+_Fused; removed none
- sheet CellFilter4 ports: added Cell+_Fused; removed none
- sheet CellFilter5 ports: added Cell+_Fused; removed none
- sheet CellFilter6 ports: added Cell+_Fused; removed none
- sheet CellFilter7 ports: added Cell+_Fused; removed none
- sheet CellFilter8 ports: added Cell+_Fused; removed none
- sheet CellFilter9 ports: added Cell+_Fused; removed none
- note added: "A1"
- note removed: "A0"
