File: Battman/KiCad/Battman/singlefilter.kicad_sch (KiCad schematic)
At the start: 11 parts, among them Q200 NX2301P,215

Commit message: Uopdated Schematics fixed
Parts:
- removed R203, R204: AC2010FK-0768RL, C__Users_otto_Documents_AltiumLL_SamacSys.PcbLib:RESC5025X65N, symbol Battman-altium-import:CellFilter10_1_AC2010FK-0768RL_SamacSys.SchLib
- added R203: 33R, 2W, 5%, C__Users_otto_Documents_AltiumLL_SamacSys.PcbLib:RESC6331X80N, symbol Battman-altium-import:CellFilter10_1_CRM2512-JW-330ELF_SamacSys.SchLib
- C200, C201: value 06031C103K4Z2A -> 10nF 100V X7R
- R200: ALTIUM_VALUE 1k -> 1k, 1%; SUPPLIER 1 (none) -> Avnet; SUPPLIER PART NUMBER 1 (none) -> AF0603FR-071KL
- R201: SUPPLIER 1 (none) -> Mouser; SUPPLIER PART NUMBER 1 (none) -> 71-CRCW0603-100-E3
- R202: value 3k3 -> 3k3 1%; SUPPLIER 1 (none) -> Avnet; SUPPLIER PART NUMBER 1 (none) -> 46AK9312
Connections:
- net Cell-: now also R203.1
- net at Q200.3 (D): now also R203.2
Other:
- note added: "A1"
- note removed: "A0"

Commit message: Begin of kicad conversion
Parts:
- removed C200, C201: 10nF 100V X7R, C__Users_otto_Documents_AltiumLL_SamacSys.PcbLib:CAPC1608X90N, symbol Battman-altium-import:CellFilter10_1_06031C103K4Z2A_SamacSys.SchLib
- removed F200: 0466.250NR, C__Users_otto_Documents_AltiumLL_SamacSys.PcbLib:FUSC3215X66N, symbol Battman-altium-import:CellFilter10_0_0466.250NR_SamacSys.SchLib
- removed Q200: NX2301P,215, C__Users_otto_Documents_AltiumLL_SamacSys.PcbLib:SOT95P230X110-3N, symbol Battman-altium-import:CellFilter10_2_NX2301P,215_SamacSys.SchLib
- removed R200: AF0603FR-071KL, C__Users_otto_Documents_AltiumLL_SamacSys.PcbLib:RESC1608X55N, symbol Battman-altium-import:CellFilter10_0_AF0603FR-071KL_SamacSys.SchLib
- removed R201: CRCW0603100RFKEA, C__Users_otto_Documents_AltiumLL_SamacSys.PcbLib:RESC1608X50N, symbol Battman-altium-import:CellFilter10_0_CRCW0603100RFKEA_SamacSys.SchLib
- removed R202: 3k3 1%, C__Users_otto_Documents_AltiumLL_SamacSys.PcbLib:RESC1608X55N, symbol Battman-altium-import:CellFilter10_0_CRGH0603F3K3_SamacSys.SchLib
- removed R203: 33R, 2W, 5%, C__Users_otto_Documents_AltiumLL_SamacSys.PcbLib:RESC6331X80N, symbol Battman-altium-import:CellFilter10_1_CRM2512-JW-330ELF_SamacSys.SchLib
- removed Z200, Z201: MMSZ4692T1G, C__Users_otto_Documents_AltiumLL_SamacSys.PcbLib:SOD3716X135N, symbol Battman-altium-import:CellFilter10_3_MMSZ4692T1G_SamacSys.SchLib
- added C200, C201: 10nF 100V X7R, C__Users_otto_Documents_AltiumLL_SamacSys.PcbLib:CAPC1608X90N, symbol Battman-altium-import:CellFilter6_1_06031C103K4Z2A_SamacSys.SchLib
- added F200: 0466.250NR, C__Users_otto_Documents_AltiumLL_SamacSys.PcbLib:FUSC3215X66N, symbol Battman-altium-import:CellFilter6_0_0466.250NR_SamacSys.SchLib
- added Q200: NX2301P,215, C__Users_otto_Documents_AltiumLL_SamacSys.PcbLib:SOT95P230X110-3N, symbol Battman-altium-import:CellFilter6_2_NX2301P,215_SamacSys.SchLib
- added R200: AF0603FR-071KL, C__Users_otto_Documents_AltiumLL_SamacSys.PcbLib:RESC1608X55N, symbol Battman-altium-import:CellFilter6_0_AF0603FR-071KL_SamacSys.SchLib
- added R201: CRCW0603100RFKEA, C__Users_otto_Documents_AltiumLL_SamacSys.PcbLib:RESC1608X50N, symbol Battman-altium-import:CellFilter6_0_CRCW0603100RFKEA_SamacSys.SchLib
- added R202: 3k3 1%, C__Users_otto_Documents_AltiumLL_SamacSys.PcbLib:RESC1608X55N, symbol Battman-altium-import:CellFilter6_0_CRGH0603F3K3_SamacSys.SchLib
- added R203: 33R, 2W, 5%, C__Users_otto_Documents_AltiumLL_SamacSys.PcbLib:RESC6331X80N, symbol Battman-altium-import:CellFilter6_1_CRM2512-JW-330ELF_SamacSys.SchLib
- added Z200, Z201: MMSZ4692T1G, C__Users_otto_Documents_AltiumLL_SamacSys.PcbLib:SOD3716X135N, symbol Battman-altium-import:CellFilter6_3_MMSZ4692T1G_SamacSys.SchLib
Other:
- note added: "A3"
- note removed: "A1"

Commit message: kicad release
Parts:
- removed C200, C201: 10nF 100V X7R, C__Users_otto_Documents_AltiumLL_SamacSys.PcbLib:CAPC1608X90N, symbol Battman-altium-import:CellFilter6_1_06031C103K4Z2A_SamacSys.SchLib
- removed F200: 0466.250NR, C__Users_otto_Documents_AltiumLL_SamacSys.PcbLib:FUSC3215X66N, symbol Battman-altium-import:CellFilter6_0_0466.250NR_SamacSys.SchLib
- removed Q200: NX2301P,215, C__Users_otto_Documents_AltiumLL_SamacSys.PcbLib:SOT95P230X110-3N, symbol Battman-altium-import:CellFilter6_2_NX2301P,215_SamacSys.SchLib
- removed R200: AF0603FR-071KL, C__Users_otto_Documents_AltiumLL_SamacSys.PcbLib:RESC1608X55N, symbol Battman-altium-import:CellFilter6_0_AF0603FR-071KL_SamacSys.SchLib
- removed R201: CRCW0603100RFKEA, C__Users_otto_Documents_AltiumLL_SamacSys.PcbLib:RESC1608X50N, symbol Battman-altium-import:CellFilter6_0_CRCW0603100RFKEA_SamacSys.SchLib
- removed R202: 3k3 1%, C__Users_otto_Documents_AltiumLL_SamacSys.PcbLib:RESC1608X55N, symbol Battman-altium-import:CellFilter6_0_CRGH0603F3K3_SamacSys.SchLib
- removed R203: 33R, 2W, 5%, C__Users_otto_Documents_AltiumLL_SamacSys.PcbLib:RESC6331X80N, symbol Battman-altium-import:CellFilter6_1_CRM2512-JW-330ELF_SamacSys.SchLib
- removed Z200, Z201: MMSZ4692T1G, C__Users_otto_Documents_AltiumLL_SamacSys.PcbLib:SOD3716X135N, symbol Battman-altium-import:CellFilter6_3_MMSZ4692T1G_SamacSys.SchLib
- added C200J, C201J: 10nF 100V X7R, C__Users_otto_Documents_AltiumLL_SamacSys.PcbLib:CAPC1608X90N, symbol Battman-altium-import:CellFilter6_1_06031C103K4Z2A_SamacSys.SchLib
- added F200J: 0466.250NR, C__Users_otto_Documents_AltiumLL_SamacSys.PcbLib:FUSC3215X66N, symbol Battman-altium-import:CellFilter6_0_0466.250NR_SamacSys.SchLib
- added Q200J: NX2301P,215, C__Users_otto_Documents_AltiumLL_SamacSys.PcbLib:SOT95P230X110-3N, symbol Battman-altium-import:CellFilter6_2_NX2301P,215_SamacSys.SchLib
- added R200J: AF0603FR-071KL, C__Users_otto_Documents_AltiumLL_SamacSys.PcbLib:RESC1608X55N, symbol Battman-altium-import:CellFilter6_0_AF0603FR-071KL_SamacSys.SchLib
- added R201J: 100R, 1%, C__Users_otto_Documents_AltiumLL_SamacSys.PcbLib:RESC1608X50N, symbol Battman-altium-import:CellFilter6_0_CRCW0603100RFKEA_SamacSys.SchLib
- added R202J: 3k3 1%, C__Users_otto_Documents_AltiumLL_SamacSys.PcbLib:RESC1608X55N, symbol Battman-altium-import:CellFilter6_0_CRGH0603F3K3_SamacSys.SchLib
- added R203J: 33R, 2W, 5%, C__Users_otto_Documents_AltiumLL_SamacSys.PcbLib:RESC6331X80N, symbol Battman-altium-import:CellFilter6_1_CRM2512-JW-330ELF_SamacSys.SchLib
- added Z200J, Z201J: MMSZ4692T1G, C__Users_otto_Documents_AltiumLL_SamacSys.PcbLib:SOD3716X135N, symbol Battman-altium-import:CellFilter6_3_MMSZ4692T1G_SamacSys.SchLib
Connections:
- net Cell+: now also F200J.1
- net Cell+_Fused: now also F200J.2, Q200J.2 (S), R200J.1, R201J.1
- net Cell-: now also R203J.1
- net Cell_GND: now also C200J.1, C201J.1
- net LTC_H_C+: now also C200J.2, R200J.2
- net LTC_H_C-: now also Z200J.2 (A)
- net LTC_S_C+: now also C201J.2, R201J.2
- net LTC_S_C-: now also Z201J.2 (A)
- net LTC_S_S: now also R202J.2
- new net: Q200J.1 (G), R202J.1
- new net: Q200J.3 (D), R203J.2
