File: ElonMux/Interface - Connectors.kicad_sch (KiCad schematic)
At the start: 20 parts, among them J1001 Conn_01x04, J1002 Conn_01x04, J1003 Conn_01x04, J1004 USB4105-GF-A, J1005 S2B-PH-SM4-TB, J1006 S2B-PH-SM4-TB

Commit message: Finished V1.1, maybe extra cleaning needed of some details in the doc
Other:
- note added: "2x"
- note added: "Removed JTAG in V1.1"
- note removed: "Removed JTAG"

Commit message: Small adjustments
Parts:
- J1001: Manufacturer (none) -> JST Commercial; Manufacturer Part Number (none) -> S4B-PH-SM4-TB(LF)(SN); Supplier (none) -> Mouser Electronics; Supplier Part Number (none) -> 306-S4BPHSM4TBLFSN
- J1003: now left out of the parts list
- J1005, J1006: Manufacturer Part Number S2B-PH-SM4-TB -> S2B-PH-SM4-TB(LF)(SN); Supplier Digikey -> Mouser Electronics; Supplier Part Number 455-S2B-PH-SM4-TBCT-ND -> 306-S2BPHSM4TBLFSN
