File: ElonMux/MCU - Unit.kicad_sch (KiCad schematic)
At the start: 53 parts, among them U401 ESP32-S3FN8, Y401 ECS-400-10-33B-CKM-TR

Commit message: Done with changes of v1.1, need to final check and order
Parts:
- removed JP402: Solder Jumper, Jumper:SolderJumper-2_P1.3mm_Open_RoundedPad1.0x1.5mm, symbol Jumper:Jumper_2_Small_Open
- removed R407: 10k 1%, Resistor_SMD:R_0402_1005Metric, symbol Device:R
- removed TP401: MTCK, Charge_Manager_FP:TestPoint_Pad_D0.5mm_Front, symbol Connector:TestPoint
- removed TP402: MTDO, Charge_Manager_FP:TestPoint_Pad_D0.5mm_Front, symbol Connector:TestPoint
- removed TP403: MTDI, Charge_Manager_FP:TestPoint_Pad_D0.5mm_Front, symbol Connector:TestPoint
- removed TP404: MTMS, Charge_Manager_FP:TestPoint_Pad_D0.5mm_Front, symbol Connector:TestPoint
- removed TP405: SPI_NCS, Charge_Manager_FP:TestPoint_Pad_D0.5mm_Front, symbol Connector:TestPoint
- removed TP406: SPI_MOSI, Charge_Manager_FP:TestPoint_Pad_D0.5mm_Front, symbol Connector:TestPoint
- removed TP407: SPI_MISO, Charge_Manager_FP:TestPoint_Pad_D0.5mm_Front, symbol Connector:TestPoint
- removed TP408: SPI_CLK, Charge_Manager_FP:TestPoint_Pad_D0.5mm_Front, symbol Connector:TestPoint
- R403, R404, R405, R406: value 10k 1% -> 100k 1%; Manufacturer KOA Speer -> Panasonic; Manufacturer Part Number SG73P1EWTTP1002F -> ERJ-2RKF1003X; Supplier Part Number 660-SG73P1EWTTP1002F -> 667-ERJ-2RKF1003X
- renumbered R408 to R407, R409 to R408, TP409 to TP401, TP410 to TP402, TP411 to TP403, TP412 to TP404, TP413 to TP405, TP414 to TP406, TP415 to TP407, TP416 to TP408, TP417 to TP409, TP418 to TP410, TP419 to TP411, TP420 to TP412, TP421 to TP413, TP422 to TP414, TP423 to TP415
Connections:
- net FAULT1: now also R404.2; no longer R405.2
- net FAULT2: now also R403.2; no longer R404.2
- net INTn: now also R405.2; no longer R406.2
- net PGn: now also R406.2
- net MTCK: no longer names the net of U401.44 (MTCK)
- net MTDI: no longer names the net of U401.47 (MTDI)
- net MTDO: no longer names the net of U401.45 (MTDO)
- net MTMS: no longer names the net of U401.48 (MTMS)
- net SPI_CLK: no longer names the net of U401.14 (GPIO9)
- net SPI_MISO: no longer names the net of U401.13 (GPIO8)
- net SPI_MOSI: no longer names the net of U401.12 (GPIO7)
- net SPI_NCS: no longer names the net of U401.11 (GPIO6)
- net SPI_NCS: no longer R403.2
- no-connect marks 16 -> 24
Other:
- moved on the sheet: JP401

Commit message: Finished V1.1, maybe extra cleaning needed of some details in the doc
Other:
- note added: "Removed JTAG in V1.1"
Changed lines of the file:
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@@
 	(title_block
 		(title "MCU - Unit")
-		(date "2025-06-17")
+		(date "2025-07-24")
 		(rev "${REVISION}")
 		(company "${COMPANY}")
@@
 		)
 	)
+	(text "Removed JTAG in V1.1"
+		(exclude_from_sim no)
+		(at 61.976 197.612 0)
+		(effects
+			(font
+				(size 3.81 3.81)
+			)
+		)
+	)
 	(text "Espressif Datasheet p.30 (GPIO0 boot)"
 		(exclude_from_sim no)
@@
 			"AAAAAAAAAAAAAAAAAAAAAAAAAAAAAAAAAAAAAAAAAAAAAAAAAAAAAAAAAAAAAAAAAAAAAAAAAAAA"
 			"AAAAAAAAAAAAAAAAAAAAAAAAAAAAAAAAAAAAAAAAAAAAAAAAAAAAAAAAAAAAAAAAAAAAAAAAAAAA"
+			"AAAAAAAAAAAAAAAAAAAAAAAAAAAAAAAAAAAAAAAAAAAAAAAAAAAAAAAAAAAAAAAAAAAAAAAAAAAA"
+			"AAAAAAAAAAAAAAAAAAAAAAAAAAAAAAAAAAAAAAAAAAAAAAAAAAAAAAAAAAAAAAAAAAAAAAAAAAAA"
+			"AAAAAAAAAAAAAAAAAAAAAAAAAAAAAAAAAAAAAAAAAAAAAAAAAAAAAAAAAAAAAAAAAAAAAAAAAAAA"
+			"AAAAAAAAAAAAAAAAAAAAAAAAAAAAAAAAAAAAAAAAAAAAAAAAAAAAAAAAAAAAAAAAAAAAAAAAAAAA"
+			"AAAAAAAAAAAAAAAAAAAAAAAAAAAAAAAAAAAAAAAAAAAAAAAAAAAAAAAAAAAAAAAAAAAAAAAAAAAA"
+			"AAAAAAAAAAAAAAAAAAAAAAAAAAAAAAAAAAAAAAAAAAAAAAAAAAAAAAAAAAAAAAAAAAAAAAAAAAAA"
+			"AAAAAAAAAAAAAAAAAAAAAAAAAAAAAAAAAAAAAAAAAAAAAAAAAAAAAAAAAAAAAAAAAAAAAAAAAAAA"
+			"AAAAAAAAAAAAAAAAAAAAAAAAAAAAAAAAAAAAAAAAAAAAAAAAAAAAAAAAAAAAAAAAAAAAAAAAAAAA"
+			"AAAAAAAAAAAAAAAAAAAAAAAAAAAAAAAAAAAAAAAAAAAAAAAAAAAAAAAAAAAAAAAAAAAAAAAAAAAA"
+			"AAAAAAAAAAAAAAAAAAAAAAAAAAAAAAAAAAAAAAAAAAAAAAAAAAAAAAAAAAAAAAAAAAAAAAAAAAAA"
+			"AAAAAAAAAAAAAAAAAAAAAAAAAAAAAAAAAAAAAAAAAAAAAAAAAAAAAAAAAAAAAAAAAAAAAAAAAAAA"
+			"AAAAAAAAAAAAAAAAAAAAAAAAAAAAAAAAAAAAAAAAAAAAAAAAAAAAAAAAAAAAAAAAAAAAAAAAAAAA"
+			"AAAAAAAAAAAAAAAAAAAAAAAAAAAAAAAAAAAAAAAAAAAAAAAAAAAAAAAAAAAAAAAAAAAAAAAAAAAA"
+			"AAAAAAAAAAAAAAAAAAAAAAAAAAAAAAAAAAAAAAAAAAAAAAAAAAAAAAAAAAAAAAAAAAAAAAAAAAAA"
+			"AAAAAAAAAAAAAAAAAAAAAAAAAAAAAAAAAAAAAAAAAAAAAAAAAAAAAAAAAAAAAAAAAAAAAAAAAAAA"
+			"AAAAAAAAAAAAAAAAAAAAAAAAAAAAAAAAAAAAAAAAAAAAAAAAAAAAAAAAAAAAAAAAAAAAAAAAAAAA"
+			"AAAAAAAAAAAAAAAAAAAAAAAAAAAAAAAAAAAAAAAAAAAAAAAAAAAAAAAAAAAAAAAAAAAAAAAAAAAA"
+			"AAAAAAAAAAAAAAAAAAAAAAAAAAAAAAAAAAAAAAAAAAAAAAAAAAAAAAAAAAAAAAAAAAAAAAAAAAAA"
 			"AAAAAAAAAAAAAAAAAAAAAAAAAAAAAAAAAAAAAAAAAAAAAAAAAA=="
 		)
@@
 			"AAAATAAAAFkAAABJAAAAaQAAAHcAAABrAAAAKwAAAG8AAABPAAAAVQAAAFQAAABYAAAARwAAAHUA"
 			"AABVAAAAYwAAAGYAAABmAAAAVAAAAFMAAABXAAAAQgAAAFQAAAB4AAAAUAAAAFkAAAA2AAAAawAA"
-			"AEUAAABlAAAAQwAAAA=="
+			"AEUAAABlAAAAQwAAAE4AAABsAAAASQAAAEkAAABGAAAARwAAAEoAAAArAAAAQgAAAFMAAABRAAAA"
+			"QQAAAHIAAABSAAAAUAAAAGMAAABiAAAAUAAAAHIAAABBAAAARwAAAEMAAAB1AAAAZgAAAGIAAAB0"
+			"AAAAMgAAADIAAABzAAAAUAAAAE4AAAA3AAAAMQAAAHAAAAAwAAAAbQAAAFoAAABrAAAAcwAAAE0A"
+			"AABPAAAAMwAAAGwAAAB3AAAAVgAAAGwAAABYAAAAagAAAGQAAABEAAAAYgAAAEQAAABvAAAANwAA"
+			"AHUAAABMAAAAWgAAAC8AAABXAAAASAAAADUAAABaAAAAZgAAADMAAABYAAAAdAAAAHYAAAB2AAAA"
+			"cgAAAHEAAABxAAAAdwAAAFUAAAArAAAAdwAAAE0AAABnAAAAYQAAAGQAAABFAAAAdgAAADEAAABy"
+			"AAAATAAAADcAAAA2AAAANgAAAG0AAABMAAAATQAAAG0AAABEAAAASAAAAEsAAABiAAAATAAAAFAA"
+			"AABXAAAAeAAAAFkAAABmAAAAKwAAAG8AAAAyAAAAeAAAAFEAAABnAAAAWgAAAEYAAABaAAAAMgAA"
+			"AGUAAABtAAAAcQAAAGkAAABBAAAAYwAAAG4AAABlAAAATgAAAEMAAABGAAAATwAAAGIAAABRAAAA"
+			"YwAAADgAAABFAAAASAAAAGIAAABlAAAAZQAAAGUAAABkAAAAVgAAAHgAAABOAAAAZAAAADEAAABM"
+			"AAAAMQAAAHEAAABUAAAAYQAAAEYAAABOAAAARwAAADcAAABiAAAAYgAAAEgAAABlAAAAYQAAAGYA"
+			"AABwAAAAZgAAACsAAABHAAAAeAAAADEAAABiAAAAdAAAAHIAAAAyAAAANAAAAE8AAAA3AAAATwAA"
+			"AHUAAABIAAAAdAAAAFUAAABYAAAAMQAAAHQAAABhAAAAbwAAADkAAABGAAAAMwAAAEUAAABsAAAA"
+			"SQAAAEMAAAAzAAAAaQAAAEcAAAB1AAAAagAAAHEAAABQAAAATgAAAGEAAABkAAAAaQAAADcAAAA3"
+			"AAAATgAAAGcAAABWAAAARAAAAFAAAABzAAAAcQAAADkAAABqAAAATwAAAGgAAABzAAAAVQAAAFkA"
+			"AABYAAAAKwAAAGQAAABuAAAAWQAAAHEAAABJAAAAMQAAADcAAABXAAAAYgAAAGMAAAA2AAAAQQAA"
+			"AGkAAAA2AAAATwAAAGMAAAByAAAAZwAAACsAAABkAAAAeAAAAG4AAABKAAAAKwAAAHUAAABQAAAA"
+			"OAAAAE4AAABoAAAAUQAAAHQAAABJAAAAegAAADMAAABlAAAAKwAAACsAAAArAAAAMAAAADUAAAA4"
+			"AAAAKwAAAHUAAABtAA=="
 		)
 	)
@@
 			"MQAAAGgAAABMAAAAdwAAAFEAAABnAAAAQQAAAEEAAABFAAAASQAAAFEAAABBAAAAQQAAAEMAAABF"
 			"AAAASQAAAEEAAABBAAAAQgAAAEYAAABJAAAAbQAAAGcAAABHAAAAQQAAAHAAAABaAAAAYQAAAEEA"
-			"AABrAA=="
+			"AABrAAAAAAAAAAAAAAAAAAAAAAAAAAAAAAAAAAAAAAAAAAAAAAAAAAAAAAAAAAAAAAAAAAAAAAAA"
+			"AAAAAAAAAAAAAAAAAAAAAAAAAAAAAAAAAAAAAAAAAAAAAAAAAAAAAAAAAAAAAAAAAAAAAAAAAAAA"
+			"AAAAAAAAAAAAAAAAAAAAAAAAAAAAAAAAAAAAAAAAAAAAAAAAAAAAAAAAAAAAAAAAAAAAAAAAAAAA"
+			"AAAAAAAAAAAAAAAAAAAAAAAAAAAAAAAAAAAAAAAAAAAAAAAAAAAAAAAAAAAAAAAAAAAAAAAAAAAA"
+			"AAAAAAAAAAAAAAAAAAAAAAAAAAAAAAAAAAAAAAAAAAAAAAAAAAAAAAAAAAAAAAAAAAAAAAAAAAAA"
+			"AAAAAAAAAAAAAAAAAAAAAAAAAAAAAAAAAAAAAAAAAAAAAAAAAAAAAAAAAAAAAAAAAAAAAAAAAAAA"
+			"AAAAAAAAAAAAAAAAAAAAAAAAAAAAAAAAAAAAAAAAAAAAAAAAAAAAAAAAAAAAAAAAAAAAAAAAAAAA"
+			"AAAAAAAAAAAAAAAAAAAAAAAAAAAAAAAAAAAAAAAAAAAAAAAAAAAAAAAAAAAAAAAAAAAAAAAAAAAA"
+			"AAAAAAAAAAAAAAAAAAAAAAAAAAAAAAAAAAAAAAAAAAAAAAAAAAAAAAAAAAAAAAAAAAAAAAAAAAAA"
+			"AAAAAAAAAAAAAAAAAAAAAAAAAAAAAAAAAAAAAAAAAAAAAAAAAAAAAAAAAAAAAAAAAAAAAAAAAAAA"
+			"AAAAAAAAAAAAAAAAAAAAAAAAAAAAAAAAAAAAAAAAAAAAAAAAAAAAAAAAAAAAAAAAAAAAAAAAAAAA"
+			"AAAAAAAAAAAAAAAAAAAAAAAAAAAAAAAAAAAAAAAAAAAAAAAAAAAAAAAAAAAAAAAAAAAAAAAAAAAA"
+			"AAAAAAAAAAAAAAAAAAAAAAAAAAAAAAAAAAAAAAAAAAAAAAAAAAAAAAAAAAAAAAAAAAAAAAAAAAAA"
+			"AAAAAAAAAAAAAAAAAAAAAAAAAAAAAAAAAAAAAAAAAAAAAAAAAAAAAAAAAAAAAAAAAAAAAAAAAAAA"
+			"AAAAAAAAAAAAAAAAAAAAAAAAAAAAAAAAAAAAAAAAAAAAAAAAAAAAAAAAAAAAAAAAAAAAAAAAAAAA"
+			"AAAAAAAAAAAAAAAAAAAAAAAAAAAAAAAAAAAAAAAAAAAAAAAAAAAAAAAAAAAAAAAAAAAAAAAAAAAA"
+			"AAAAAAAAAAAAAAAAAAAAAAAAAAAAAAAAAAAAAAAAAAAAAAAAAAAAAAAAAAAAAAAAAAAAAAAAAAAA"
+			"AAAAAAAAAAAAAAAAAAAAAAAAAAAAAAAAAAAAAAAAAAAAAAAAAAAAAAAAAAAAAAAAAAAAAAAAAAAA"
+			"AAAAAA=="
 		)
 	)
@@
 			"AAAAAAAAAAAAAAAAAAAAAAAAAAAAAAAAAAAAAAAAAAAAAAAAAAAAAAAAAAAAAAAAAAAAAAAAAAAA"
 			"AAAAAAAAAAAAAAAAAAAAAAAAAAAAAAAAAAAAAAAAAAAAAAAAAAAAAAAAAAAAAAAAAAAAAAAAAAAA"
+			"AAAAAAAAAAAAAAAAAAAAAAAAAAAAAAAAAAAAAAcAAAAHAAAABwAAAAcAAAAHAAAABwAAAAcAAAAH"
+			"AAAABwAAAAcAAAAHAAAABwAAAAcAAAAHAAAABwAAAAcAAAAHAAAABwAAAAcAAAAHAAAABwAAAAcA"
+			"AAAHAAAABwAAAAcAAAAHAAAABwAAAAcAAAAHAAAABwAAAAcAAAAHAAAABwAAAAcAAAAHAAAABwAA"
+			"AAcAAAAHAAAABwAAAAcAAAAHAAAABwAAAAcAAAAHAAAABwAAAAcAAAAHAAAABwAAAAcAAAAHAAAA"
+			"BwAAAAcAAAAHAAAABwAAAAcAAAAHAAAABwAAAAcAAAAHAAAABwAAAAcAAAAHAAAABwAAAAcAAAAH"
+			"AAAABwAAAAcAAAAHAAAABwAAAAcAAAAHAAAABwAAAAcAAAAHAAAABwAAAAcAAAAHAAAABwAAAAcA"
+			"AAAHAAAABwAAAAcAAAAHAAAABwAAAAcAAAAHAAAABwAAAAcAAAAHAAAABwAAAAcAAAAHAAAABwAA"
+			"AAcAAAAHAAAABwAAAAcAAAAHAAAABwAAAAcAAAAHAAAABwAAAAcAAAAHAAAABwAAAAcAAAAHAAAA"
+			"BwAAAAcAAAAHAAAABwAAAAcAAAAHAAAABwAAAAcAAAAHAAAABwAAAAcAAAAHAAAABwAAAAcAAAAH"
+			"AAAABwAAAAcAAAAHAAAABwAAAAcAAAAHAAAABwAAAAcAAAAHAAAABwAAAAcAAAAHAAAABwAAAAcA"
+			"AAAHAAAABwAAAAcAAAAHAAAABwAAAAcAAAAHAAAABwAAAAcAAAAHAAAABwAAAAcAAAAHAAAABwAA"
+			"AAcAAAAHAAAABwAAAAcAAAAHAAAABwAAAAcAAAAHAAAABwAAAAcAAAAHAAAABwAAAAcAAAAHAAAA"
+			"BwAAAAcAAAAHAAAABwAAAAcAAAAFAAAAAAAAAAAAAAAAAAAAAAAAAAAAAAAAAAAAAAAAAAAAAAAA"
+			"AAAAAAAAAAAAAAAAAAAAAAAAAAAAAAAAAAAAAAAAAAAAAAAAAAAAAAAAAAAAAAAAAAAAAAAAAAAA"
+			"AAAAAAAAAAAAAAAAAAAAAAAAAAAAAAAAAAAAAAAAAAAAAAAAAAAAAAAAAAAAAAAAAAAAAAAAAAAA"
+			"AAAAAAAAAAAAAAAAAAAAAAAAAAAAAAAAAAAAAAAAAAAAAAAAAAAAAAAAAAAAAAAAAAAAAAAAAAAA"
+			"AAAAAAAAAAAAAAAAAAAAAAAAAAAAAAAAAAAAAAAAAAAAAAAAAAAAAAAAAAAAAAAAAAAAAAAAAAAA"
+			"AAAAAAAAAAAAAAAAAAAAAAAAAAAAAAAAAAAAAAAAAAAAAAAAAAAAAAAAAAAAAAAAAAAAAAAAAAAA"
 			"AAAAAAAAAAAAAAAAAAAAAAAAAAAAAAAAAA=="
 		)
@@
 			"AAAAAAAAAAAAAAAAAAAAAAAAAAAAAAAAAAAAAAAAAAAAAAAAAAAAAAAAAAAAAAAAAAAAAAAAAAAA"
 			"AAAAAAAAAAAAAAAAAAAAAAAAAAAAAAAAAAAAAAAAAAAAAAAAAAAAAAAAAAAAAAAAAAAAAAAAAAAA"
+			"AAAAAAAAAAAAAAAAAAAAAAAAAAAAAAAAAAAAAAAAAAAAAAAAAAAAAAAAAAAAAAAAAAAAAAAAAAAA"
+			"AAAAAAAAAAAAAAAAAAAAAAAAAAAAAAAAAAAAAAAAAAAAAAAAAAAAAAAAAAAAAAAAAAAAAAAAAAAA"
+			"AAAAAAAAAAAAAAAAAAAAAAAAAAAAAAAAAAAAAAAAAAAAAAAAAAAAAAAAAAAAAAAAAAAAAAAAAAAA"
+			"AAAAAAAAAAAAAAAAAAAAAAAAAAAAAAAAAAAAAAAAAAAAAAAAAAAAAAAAAAAAAAAAAAAAAAAAAAAA"
+			"AAAAAAAAAAAAAAAAAAAAAAAAAAAAAAAAAAAAAAAAAAAAAAAAAAAAAAAAAAAAAAAAAAAAAAAAAAAA"
+			"AAAAAAAAAAAAAAAAAAAAAAAAAAAAAAAAAAAAAAAAAAAAAAAAAAAAAAAAAAAAAAAAAAAAAAAAAAAA"
+			"AAAAAAAAAAAAAAAAAAAAAAAAAAAAAAAAAAAAAAAAAAAAAAAAAAAAAAAAAAAAAAAAAAAAAAAAAAAA"
+			"AAAAAAAAAAAAAAAAAAAAAAAAAAAAAAAAAAATID86GBoNDxUVFRUVDRAUHSEZAQAAAAAAAAAAAAAA"
+			"AAAAAAAAAAAAAAAAAAAAAAAAAAAAAAAAAAAAAAAAAAAAAAAAAAAAAAAAAAAAAAAAAAAAAAAAAAAA"
+			"AAAAAAAAAAAAAAAAAAAAAAAAAAAAAAAAAAAAAAAAAAAAAAAAAAAAAAAAAAAAAAAAAAAAAAAAAAAA"
+			"AAAAAAAAAAAAAAAAAAAAAAAAAAAAAAAAAAAAAAAAAAAAAAAAAAAAAAAAAAAAAAAAAAAAAAAAAAAA"
+			"AAAAAAAAAAAAAAAAAAAAAAAAAAAAAAAAAAAAAAAAAAAAAAAAAAAAAAAAAAAAAAAAAAAAAAAAAAAA"
+			"AAAAAAAAAAAAAAAAAAAAAAAAAAAAAAAAAAAAAAAAAAAAAAAAAAAAAAAAAAAAAAAAAAAAAAAAAAAA"
+			"AAAAAAAAAAAAAAAAAAAAAAAAAAAAAAAAAAAAAAAAAAAAAAAAAAAAAAAAAAAAAAAAAAAAAAAAAAAA"
+			"AAAAAAAAAAAAAAAAAAAAAAAAAAAAAAAAAAAAAAAAAAAAAAAAAAAAAAAAAAAAAAAAAAAAAAAAAAAA"
+			"AAAAAAAAAAAAAAAAAAAAAAAAAAAAAAAAAAAAAAAAAAAAAAAAAAAAAAAAAAAAAAAAAAAAAAAJARMA"
+			"AAAAAAAAAAAAAAAAAAAAAAAAAAAAAAAAAAAAAAAAAAAAAAAAAAAAAAAAAAAAAAAAAAAAAAAAAAAA"
+			"AAAAAAAAAAAAAAAAAAAAAAAAAAAAAAAAAAAAAAAAAAAAAAAAAAAAAAAAAAAAAAAAAAAAAAAAAAAA"
