File: Bucky/Bucky.kicad_pcb (KiCad board)
At the start: 2 copper layers, 120.5 x 66 mm, 188 parts, among them IC1 INA239AQDGSRQ1, IC1201 MAX25262AFOF_VY+, IC1701 TPA6205A1DGN, IC2 INA239AQDGSRQ1, IC2001 INA239AQDGSRQ1, IC3 INA239AQDGSRQ1, IC4 LTC4372CMS8#TRPBF, IC5 LTC4372CMS8#TRPBF, IC701 LTC4372CMS8#TRPBF, IC702 LTC4372CMS8#TRPBF, IC801 TPS629206QDRLRQ1, J1 XT60PW-M, J11 XT30AW-M, J12 XT30AW-M, J13 XT30AW-M, J14 XT30AW-M, J15 502585-0470, J16 FTSH-105-01-F-D-RA-K, J17 XT30UPB-F, J1701 53048-0450, J1702 505110-3091, J18 XT30UPB-F, J1801 S2B-PH-SM4-TB, J2 XT60PW-F, J202 Conn_Picoblade_JST_DEBUG, J3 XT30PW-M, J4 XT30PW-M, J403 USB4105-GF-A, J5 XT30PW-M, J6 XT30PW-M, J7 XT30UPB-F, J8 XT30UPB-F, Q1 BSC016N06NSATMA1, Q1401 PMV90ENER, Q2 BSC016N06NSATMA1, Q3 BSC016N06NSATMA1, Q4 BSC016N06NSATMA1, Q701 BSC016N06NSATMA1, Q702 BSC016N06NSATMA1, Q703 BSC016N06NSATMA1, Q704 BSC016N06NSATMA1, Q801 PMV90ENER, Q802 PMV90ENER, U1 TPS2116DRLR, U1701 74LVC1G125, U1801 DGD0216WT-7, U401 STM32G483RET6, U802 LMR36506MSC5RPERQ1, Y201 ABM8W-48.0000MHZ-4-D1X-T3

Commit message: removed 12V local generation
Parts:
- removed C1701: 100n X7R 50V, 0_capacitor_smd:C_0402_1005_DensityHigh
- removed C1702, C1703, C1704: 4.7n X7R 50V, 0_capacitor_smd:C_0603_1608_DensityHigh
- removed C1705, C1706: 470n X5R 16V, 0_capacitor_smd:C_0603_1608_DensityHigh
- removed C1707: 220n X7R 10V, 0_capacitor_smd:C_0603_1608_DensityHigh
- removed C1708: 1u X7R 16V, 0_capacitor_smd:C_0603_1608_DensityHigh
- removed the C1801 at (234.4, 132.2)
- removed the C1801 at (242.1, 84.5)
- removed the C1802 at (234.8, 130.1)
- removed the C1802 at (238.3, 84.2)
- removed D2: SMAJ24A, Diode_SMD:D_SMA
- removed IC1701: TPA6205A1DGN, 0_connectors:SOP65P490X110-9N
- removed J1701: 53048-0450, 0_connectors:SHDRRA4W35P0X125_1X4_675X550X350P
- removed the J1801 at (210.0, 157.5)
- removed the J1801 at (266.1, 156.6)
- removed the Q1401 at (235.3, 126.8)
- removed the Q1401 at (238.8, 80.8)
- removed Q701, Q702, Q703, Q704: BSC016N06NSATMA1, 0_transistor_fet:PG-TDSON-8_INF
- removed R1701, R1702: 33 1% 1/10W, 0_resistor_smd:R_0603_1608_DensityHigh
- removed R1703, R1704, R1706: 1k 1% 1/10W, 0_resistor_smd:R_0603_1608_DensityHigh
- removed R1705: 47k 1% 1/10W, 0_resistor_smd:R_0603_1608_DensityHigh
- removed R1707, R1708: 10k 1% 1/10W, 0_resistor_smd:R_0603_1608_DensityHigh
- removed R1709, R1710: 20k 1% 1/10W, 0_resistor_smd:R_0603_1608_DensityHigh
- removed R404: 10k 1% 1/16W, 0_resistor_smd:R_0402_1005_DensityHigh
- removed U1701: 74LVC1G125, 0_package_SON:SOT95P280X145-5N
- removed the U1801 at (239.5, 98.4)
- removed the U1801 at (239.1, 76.2)
- added C10: 1u X7R 10V, 0_capacitor_smd:C_0402_1005_DensityHigh, F.Cu at (86.2, 122.4)
- added C11: 1u X7R 10V, 0_capacitor_smd:C_0402_1005_DensityHigh, F.Cu at (86.2, 124.2)
- added C12: 1u X7R 10V, 0_capacitor_smd:C_0402_1005_DensityHigh, F.Cu at (86.2, 126.0)
- added C1801: 100n X7R 50V, 0_capacitor_smd:C_0402_1005_DensityHigh, B.Cu at (267.3, 60.2)
- added C1802: 4.7u X7R 16V, 0_capacitor_smd:C_0603_1608_DensityHigh, B.Cu at (269.6, 75.1)
- added C8: 100n X7R 50V, 0_capacitor_smd:C_0402_1005_DensityHigh, F.Cu at (135.2, 120.4)
- added C9: 1u X7R 10V, 0_capacitor_smd:C_0402_1005_DensityHigh, F.Cu at (86.2, 120.6)
- added H1: M2 (3.2mm), MountingHole:MountingHole_2.2mm_M2_Pad_Via, F.Cu at (258.4, 54.0)
- added H2: M2 (3.2mm), MountingHole:MountingHole_2.2mm_M2_Pad_Via, F.Cu at (260.0, 105.0)
- added H3: M2 (3.2mm), MountingHole:MountingHole_2.2mm_M2_Pad_Via, F.Cu at (170.0, 56.6)
- added H501: M2 (3.2mm), MountingHole:MountingHole_2.2mm_M2_Pad_Via, F.Cu at (173.3, 105.0)
- added IC6: INA239AQDGSRQ1, 0_diode_smd:SOP50P490X110-10N, F.Cu at (137.6, 107.1)
- added J1801: S2B-PH-SM4-TB, 0_connectors:JST_PH_S2B-PH-SM4-TB_1x02-1MP_P2.00mm_Horizontal, F.Cu at (270.0, 90.0)
- added NT7: NetTieShuntH, 0_net_tie:NetTie-2_SMD_Pad0.2mm, F.Cu at (138.9, 116.4)
- added NT8: NetTieShuntL, 0_net_tie:NetTie-2_SMD_Pad0.2mm, F.Cu at (138.9, 117.9)
- added Q1401: PMV90ENER, 0_package_SOT_TO_SMD:SOT-23-3, B.Cu at (270.1, 85.3)
- added Q5: ISC016N04NM7V, 0_transistor_fet:IFX-PG-TDSON-8-36-V, B.Cu at (199.4, 54.9)
- added Q6: ISC016N04NM7V, 0_transistor_fet:IFX-PG-TDSON-8-36-V, B.Cu at (191.6, 54.9)
- added Q7: ISC016N04NM7V, 0_transistor_fet:IFX-PG-TDSON-8-36-V, B.Cu at (210.0, 55.0)
- added Q8: ISC016N04NM7V, 0_transistor_fet:IFX-PG-TDSON-8-36-V, B.Cu at (212.1, 45.0)
- added R8: 0.3m, 0_resistor_smd:RES_WSLP3921_.003OHM_VIS, F.Cu at (127.8, 116.2)
- added U1801: DGD0216WT-7, Package_TO_SOT_SMD:TSOT-23-5, B.Cu at (270.5, 70.8)
- C1201, C1202, C1203, C1204, C1205, C1206, C1207, C1709, C203, C207, C403, C404, C405, C406, C407, C408, C409, C410, C411, C412, C413, C414, C415, C416, C417, C701, C703, C801, C802, C803, C804, C805, C806, C807, C808, C809, C810, C811, C812, C813, C814, C815, C816, C817, C818, C820, D203, D402, D702, D8, D9, FB1201, FB801, IC1201, IC2001, IC4, IC5, IC701, IC702, IC801, L801, L802, L803, NT1601, NT1602, Q801, Q802, R4, R401, R402, R403, R405, R406, R407, R408, R5, R701, R702, R703, R801, R802, R803, R804, R805, R806, R807, R808, U1, U401, U802, Y201: moved to B.Cu
- F1: footprint SamacSys_Parts:FUSC6127X294N -> 0_diode_smd:FUSC6127X294N; moved to B.Cu
- F2, F3, F4: footprint SamacSys_Parts:FUSC6127X294N -> 0_diode_smd:FUSC6127X294N
- J1, J11, J12, J13, J14, J15, J16, J17, J1702, J18, J2, J403, J7, J8: moved to F.Cu
- J3, J4, J5, J6: value XT30PW-M -> XT30PW-F; footprint SamacSys_Parts:XT30PWM -> SamacSys_Parts:XT30PWF; moved to F.Cu
- Q1, Q2, Q3, Q4: value BSC016N06NSATMA1 -> ISC016N04NM7V; footprint 0_transistor_fet:PG-TDSON-8_INF -> 0_transistor_fet:IFX-PG-TDSON-8-36-V; moved to B.Cu
- moved F4 206.0 mm to (245.0, 80.0), turned to 0 degrees
- moved C1206 190.0 mm to (246.5, 107.5), turned to -90 degrees
- moved F3 181.7 mm to (225.0, 80.0), turned to 0 degrees
- moved C804 176.4 mm to (237.8, 107.6), turned to -90 degrees
- moved C805 176.4 mm to (240.5, 107.6), turned to -90 degrees
- moved R807 176.4 mm to (233.6, 88.7), turned to 180 degrees
- moved L801 176.1 mm to (232.5, 107.8), turned to -90 degrees
- moved R808 174.6 mm to (233.6, 90.5), turned to 180 degrees
- moved C803 173.5 mm to (243.6, 107.4), turned to -90 degrees
- moved C807 172.6 mm to (239.5, 102.0), turned to 180 degrees
- moved C1207 171.6 mm to (249.5, 107.6), turned to -90 degrees
- moved Q801 169.8 mm to (237.5, 94.0), turned to 180 degrees
- moved R806 168.7 mm to (223.5, 103.5), turned to 180 degrees
- moved IC801 167.9 mm to (230.6, 100.8), turned to 180 degrees
- moved C820 167.7 mm to (222.8, 101.5), turned to -90 degrees
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Connections:
- C1201 pad 1: /PConnectors/VBuck_in -> /PConnectors/VBatt
- C810 pad 1: /PConnectors/VBuck_in -> /PConnectors/VBatt
- F1 pad 1: /PConnectors/Vout_5V -> /PConnectors/Vin_5V
- F2 pad 1: /PConnectors/Vout_12V -> /PConnectors/Vin_12V
- F3 pad 1: /PConnectors/Vout_15V -> /PConnectors/Vin_15V
- F4 pad 1: /PConnectors/Vout_24V -> /PConnectors/Vin_24V
- F6 pad 1: /PConnectors/VBuck_in -> /PConnectors/VBatt
- FB1201 pad 1: /PConnectors/VBuck_in -> /PConnectors/VBatt
- FB801 pad 1: /PConnectors/VBuck_in -> /PConnectors/VBatt
- IC1 pad 1: /Sensor/SPI1_NSS -> /Sensor/SPI1_NSS1
- IC1 pad 10: /Sensor/shunt+ -> /Sensor/shunt12+
- IC1 pad 8: /Sensor/shunt- -> /Sensor/shunt12-
- IC1 pad 9: /Sensor/shunt- -> /Sensor/shunt12-
- IC2 pad 1: /Sensor/SPI1_NSS -> /Sensor/SPI1_NSS2
- IC2 pad 10: /Sensor/shunt+ -> /Sensor/shunt15+
- IC2 pad 8: /Sensor/shunt- -> /Sensor/shunt15-
- IC2 pad 9: /Sensor/shunt- -> /Sensor/shunt15-
- IC2001 pad 1: /Sensor/SPI1_NSS -> /Sensor/SPI1_NSS0
- IC2001 pad 10: /Sensor/shunt+ -> /Sensor/shunt5+
- IC2001 pad 8: /Sensor/shunt- -> /Sensor/shunt5-
- IC2001 pad 9: /Sensor/shunt- -> /Sensor/shunt5-
- IC3 pad 1: /Sensor/SPI1_NSS -> /Sensor/SPI1_NSS3
- IC3 pad 10: /Sensor/shunt+ -> /Sensor/shunt24+
- IC3 pad 8: /Sensor/shunt- -> /Sensor/shunt24-
- IC3 pad 9: /Sensor/shunt- -> /Sensor/shunt24-
- J11 pad 1: /PConnectors/Vin_5V -> Net-(F1-Pad2)
- J12 pad 1: /PConnectors/Vin_12V -> Net-(F2-Pad2)
- J13 pad 1: /PConnectors/Vin_15V -> Net-(F3-Pad2)
- J14 pad 1: /PConnectors/Vin_24V -> Net-(F4-Pad2)
- J1702 pad 10: /DisplayInterface/APWM -> /MCU/APWM
- J1702 pad 12: /DisplayInterface/nSHDN -> /MCU/nSHDN
- J1702 pad 2: /DisplayInterface/NRST -> /MCU/NRST
- J1702 pad 3: /DisplayInterface/INT -> /MCU/INT
- J1702 pad 4: /DisplayInterface/SPI2_NSS -> /MCU/SPI2_NSS
- J1702 pad 6: /DisplayInterface/SPI2_MOSI -> /MCU/SPI2_MOSI
- J1702 pad 7: /DisplayInterface/SPI2_MISO -> /MCU/SPI2_MISO
- J1702 pad 8: /DisplayInterface/SPI2_SCK -> /MCU/SPI2_SCK
- J2 pad 1: GND -> /PConnectors/VBuck_in
- J2 pad 2: /PConnectors/VBuck_in -> GND
- J3 pad 1: /PConnectors/Vout_5V -> GND
- J3 pad 2: GND -> /PConnectors/Vout_5V
- J4 pad 1: /PConnectors/Vout_12V -> GND
- J4 pad 2: GND -> /PConnectors/Vout_12V
- J5 pad 1: /PConnectors/Vout_15V -> GND
- J5 pad 2: GND -> /PConnectors/Vout_15V
- J6 pad 1: /PConnectors/Vout_24V -> GND
- J6 pad 2: GND -> /PConnectors/Vout_24V
- NT1 pad 1: /Sensor/shunt+ -> /Sensor/shunt12+
- NT1601 pad 1: /Sensor/shunt+ -> /Sensor/shunt5+
- NT1602 pad 1: /Sensor/shunt- -> /Sensor/shunt5-
- NT2 pad 1: /Sensor/shunt- -> /Sensor/shunt12-
- NT3 pad 1: /Sensor/shunt+ -> /Sensor/shunt15+
- NT4 pad 1: /Sensor/shunt- -> /Sensor/shunt15-
- NT5 pad 1: /Sensor/shunt+ -> /Sensor/shunt24+
- NT6 pad 1: /Sensor/shunt- -> /Sensor/shunt24-
- Q1 pad 1: /PConnectors/Vout15V -> Net-(IC4-SOURCE)
- Q1 pad 2: Net-(Q1-G) -> Net-(IC4-SOURCE)
- Q2 pad 1: /PConnectors/Vout24V -> Net-(IC5-SOURCE)
- Q2 pad 2: Net-(Q2-G) -> Net-(IC5-SOURCE)
- Q3 pad 1: /PConnectors/Vout_15V -> Net-(IC4-SOURCE)
- Q3 pad 2: Net-(IC4-GATE) -> Net-(IC4-SOURCE)
- Q4 pad 1: /PConnectors/Vout_24V -> Net-(IC5-SOURCE)
- Q4 pad 2: Net-(IC5-GATE) -> Net-(IC5-SOURCE)
- R4 pad 1: Net-(Q1-G) -> Net-(Q1-GATE)
- R5 pad 1: Net-(Q2-G) -> Net-(Q2-GATE)
- U401 pad 18: /MCU/SPI1_NSS -> unconnected-(U401A-PA4-Pad18)
- U401 pad 25: /DisplayInterface/FAN -> /MCU/FAN_CTRL
- U401 pad 40: unconnected-(U401A-PC8-Pad40) -> /MCU/SPI1_NSS0
- U401 pad 41: unconnected-(U401A-PC9-Pad41) -> /MCU/SPI1_NSS1
- U401 pad 42: /MCU/I2C2_SDA -> unconnected-(U401A-PA8-Pad42)
- U401 pad 43: /MCU/I2C2_SCL -> unconnected-(U401A-PA9-Pad43)
- U401 pad 52: unconnected-(U401A-PC10-Pad52) -> /MCU/SPI1_NSS2
- U401 pad 53: unconnected-(U401A-PC11-Pad53) -> /MCU/SPI1_NSS3
- U401 pad 54: unconnected-(U401A-PC12-Pad54) -> /MCU/SPI1_NSS4
Routing:
- net /PConnectors/Vout5V: track 0.00 -> 20.5 mm, vias 0 -> 3
- net /PConnectors/Vout_5V: track 0.00 -> 19.2 mm
- net /PConnectors/Vin_5V: track 0.00 -> 12.0 mm, vias 0 -> 5
- net Net-(IC701-GATE): track 0.00 -> 9.79 mm
- net Net-(Q5-GATE): track 0.00 -> 7.13 mm, vias 0 -> 2
- net Net-(F1-Pad2): track 0.00 -> 4.41 mm
- net GND: track 0.00 -> 3.78 mm
- net /Sensor/shunt5-: track 0.00 -> 3.44 mm
- net Net-(IC701-SOURCE): track 0.00 -> 2.07 mm
- net /Sensor/shunt5+: track 0.00 -> 1.91 mm
- net Net-(IC701-INTVCC): track 0.00 -> 1.75 mm
- net Net-(C701-Pad2): track 0.00 -> 1.64 mm
Other:
- board size 120.5 x 66 mm -> 110 x 60 mm
