File: GEODE/rev1/SMPS_Motherboard/power_precharge.kicad_sch (KiCad schematic)
At the start: 20 parts, among them IC5 TPS2490DGSRG4, Q1101 SOT233 ZXMP10A13F, Q1102 SOT233 BSS123N

Commit message: ERC passed
Parts:
- C1501: renamed from C49; value 10uF X7R 100V -> 10uF X7R 100V
- renumbered C54 to C1103, C50 to C1502, C54 to C1504, IC5 to IC1501, NT301 to NT1101, NT301 to NT1103, R1705 to R1103, R33 to R1104, R33 to R1105, R33 to R1501, R34 to R1502, R37 to R1503, R38 to R1504, R39 to R1505, R40 to R1507
