File: Icky/PRECHARGE_MOS.kicad_sch (KiCad schematic)
At the start: 15 parts, among them U13 SQJQ112E-T1_GE3, U14 SQJQ112E-T1_GE3, U15 SQJQ112E-T1_GE3, U16 SQJQ112E-T1_GE3, U3 SQJQ112E-T1_GE3, U4 SQJQ112E-T1_GE3

Commit message: ERC passed v2
Parts:
- removed C30: 6.8 nF X7R 50V, symbol Device:C_Small
- removed R57, R59: 10 1% 1/16W, symbol Device:R_Small
- removed U13, U16: SQJQ112E-T1_GE3, DPAK_2E-T1_GE3_VIS, symbol SQJQ112E-T1_GE3:SQJQ112E-T1_GE3
- renumbered C5 to C20, C1 to C6, R15 to R44, R16 to R45, R13 to R51, R14 to R53, U14 to U13, U15 to U16, U3 to U7, U4 to U8
Other:
- moved on the sheet: C20, R45, R53, U16, U8
