File: Icky/15V_Interface.kicad_sch (KiCad schematic)
At the start: 21 parts, among them IC2 INA239AQDGSRQ1, IC8 LTC4368IMS-2#PBF, Q2 SOT233 BSS123N, U10 SQJQ112E-T1_GE3, U9 SQJQ112E-T1_GE3

Commit message: ERC passed
Connections:
- net SPI1_NSS2 renamed SPI1_NSS1
Changed lines of the file:
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@@
 	)
 	(rectangle
-		(start 19.05 39.37)
+		(start 17.78 39.37)
 		(end 156.21 127)
 		(stroke
@@
 	)
 	(bus_entry
-		(at 33.02 91.44)
+		(at 178.435 60.96)
 		(size 2.54 2.54)
 		(stroke
@@
 	)
 	(bus_entry
-		(at 178.435 60.96)
+		(at 178.435 58.42)
 		(size 2.54 2.54)
 		(stroke
@@
 	)
 	(bus_entry
-		(at 178.435 58.42)
+		(at 178.435 66.04)
 		(size 2.54 2.54)
 		(stroke
@@
 	)
 	(bus_entry
-		(at 178.435 66.04)
+		(at 33.02 88.9)
 		(size 2.54 2.54)
 		(stroke
@@
 	)
 	(bus_entry
-		(at 33.02 93.98)
+		(at 178.435 63.5)
 		(size 2.54 2.54)
 		(stroke
@@
 	)
 	(bus_entry
-		(at 178.435 63.5)
+		(at 33.02 93.98)
 		(size 2.54 2.54)
 		(stroke
@@
 	)
 	(bus_entry
-		(at 33.02 88.9)
+		(at 33.02 91.44)
 		(size 2.54 2.54)
 		(stroke
@@
 		)
 	)
-	(bus
-		(pts
-			(xy 33.02 88.9) (xy 31.75 87.63)
-		)
-		(stroke
-			(width 0)
-			(type default)
-		)
-	)
-	(wire
-		(pts
-			(xy 35.56 93.98) (xy 44.45 93.98)
-		)
-		(stroke
-			(width 0)
-			(type default)
-		)
-	)
 	(wire
 		(pts
@@
 	(bus
 		(pts
-			(xy 33.02 88.9) (xy 33.02 91.44)
-		)
-		(stroke
-			(width 0)
-			(type default)
-		)
-	)
-	(bus
-		(pts
 			(xy 178.435 63.5) (xy 178.435 66.04)
 		)
@@
 		)
 	)
-	(wire
+	(bus
 		(pts
-			(xy 225.425 63.5) (xy 225.425 66.04)
+			(xy 33.02 91.44) (xy 33.02 93.98)
 		)
 		(stroke
@@
 	(wire
 		(pts
-			(xy 71.12 78.74) (xy 71.12 80.01)
+			(xy 225.425 63.5) (xy 225.425 66.04)
 		)
 		(stroke
@@
 	(wire
 		(pts
-			(xy 223.52 63.5) (xy 225.425 63.5)
+			(xy 71.12 78.74) (xy 71.12 80.01)
 		)
 		(stroke
@@
 	(wire
 		(pts
-			(xy 35.56 96.52) (xy 45.72 96.52)
+			(xy 223.52 63.5) (xy 225.425 63.5)
 		)
 		(stroke
@@
 	(wire
 		(pts
-			(xy 35.56 91.44) (xy 48.26 91.44)
-		)
-		(stroke
-			(width 0)
-			(type default)
-		)
-	)
-	(wire
-		(pts
 			(xy 111.76 62.23) (xy 113.03 62.23)
 		)
@@
 	(wire
 		(pts
+			(xy 35.56 96.52) (xy 45.72 96.52)
+		)
+		(stroke
+			(width 0)
+			(type default)
+		)
+	)
+	(wire
+		(pts
+			(xy 35.56 93.98) (xy 45.72 93.98)
+		)
+		(stroke
+			(width 0)
+			(type default)
+		)
+	)
+	(wire
+		(pts
 			(xy 67.31 91.44) (xy 67.31 90.17)
 		)
@@
 		)
 	)
+	(bus
+		(pts
+			(xy 33.02 88.9) (xy 31.75 87.63)
+		)
+		(stroke
+			(width 0)
+			(type default)
+		)
+	)
 	(wire
 		(pts
@@
 		)
 	)
-	(bus
+	(wire
 		(pts
-			(xy 33.02 91.44) (xy 33.02 93.98)
+			(xy 35.56 91.44) (xy 48.26 91.44)
 		)
 		(stroke
@@
 		)
 	)
+	(bus
+		(pts
+			(xy 33.02 88.9) (xy 33.02 91.44)
+		)
+		(stroke
+			(width 0)
+			(type default)
+		)
+	)
 	(wire
 		(pts
@@
 		)
 	)
+	(label "15V_ALERT"
+		(at 45.72 96.52 180)
+		(effects
+			(font
+				(size 1.27 1.27)
+			)
+			(justify right bottom)
+		)
+	)
 	(label "15V_OUT"
 		(at 123.19 62.23 0)
@@
 	)
 	(label "15V_ALERT"
-		(at 45.72 96.52 180)
-		(effects
-			(font
-				(size 1.27 1.27)
-			)
-			(justify right bottom)
-		)
-	)
-	(label "15V_ALERT"
 		(at 181.61 71.12 0)
 		(effects
@@
 		)
 	)
-	(label "SPI1_NSS2"
-		(at 180.975 60.96 0)
+	(label "15V_SHDN"
+		(at 45.72 91.44 180)
 		(effects
 			(font
 				(size 1.27 1.27)
 			)
-			(justify left bottom)
+			(justify right bottom)
 		)
 	)
-	(label "shunt15+"
-		(at 226.695 60.96 0)
+	(label "15V_FLT"
+		(at 45.72 93.98 180)
 		(effects
 			(font
 				(size 1.27 1.27)
 			)
-			(justify left bottom)
+			(justify right bottom)
 		)
 	)
-	(label "shunt15-"
-		(at 226.695 63.5 0)
+	(label "SPI1_NSS1"
+		(at 180.975 60.96 0)
 		(effects
 			(font
@@
 		)
 	)
-	(label "15V_SHDN"
-		(at 35.56 91.44 0)
+	(label "shunt15+"
+		(at 226.695 60.96 0)
 		(effects
 			(font
@@
 		)
 	)
-	(label "15V_FLT"
-		(at 44.45 93.98 180)
+	(label "shunt15-"
+		(at 226.695 63.5 0)
 		(effects
 			(font
 				(size 1.27 1.27)
 			)
-			(justify right bottom)
+			(justify left bottom)
 		)
 	)
@@
 		)
 	)
-	(hierarchical_label "{SPI_BAT}"
+	(hierarchical_label "{15V_PROT}"
 		(shape bidirectional)
-		(at 175.26 57.15 180)
+		(at 31.75 87.63 180)
 		(effects
 			(font
@@
 		)
 	)
-	(hierarchical_label "15V_IN"
-		(shape input)
-		(at 34.29 62.23 180)
+	(hierarchical_label "{SPI_BAT}"
+		(shape bidirectional)
+		(at 175.26 57.15 180)
 		(effects
 			(font
@@
 		)
 	)
-	(hierarchical_label "{15V_PROT}"
-		(shape bidirectional)
-		(at 31.75 87.63 180)
+	(hierarchical_label "15V_IN"
+		(shape input)
+		(at 34.29 62.23 180)
 		(effects
 			(font

Commit message: ERC passed v2
Changed lines of the file:
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@@
 		)
 	)
-	(hierarchical_label "{SPI_BAT}"
+	(hierarchical_label "{SPI_SENSORS}"
 		(shape bidirectional)
 		(at 175.26 57.15 180)

Commit message: routing
Parts:
- removed NT3: NetTieShuntH, 0_net_tie:NetTie-2_SMD_Pad0.2mm, symbol Device:NetTie_2
- removed NT4: NetTieShuntL, 0_net_tie:NetTie-2_SMD_Pad0.2mm, symbol Device:NetTie_2
- C2: footprint 0_capacitor_smd:C_0402_1005_DensityHigh -> Capacitor_SMD:C_0603_1608Metric
- C23, C24, C34: footprint (none) -> Capacitor_SMD:C_0603_1608Metric
- IC2: footprint 0_diode_smd:SOP50P490X110-10N -> SamacSys_Parts:SOP50P490X110-10N
- IC8: footprint SOP50P490X110-10N -> SamacSys_Parts:SOP50P490X110-10N
- Q2: footprint 0_package_SOT_TO_SMD:SOT-23-3 -> SamacSys_Parts:BSS123N
- R22, R23, R24, R25, R26, R27, R28, R29, R46: footprint (none) -> Resistor_SMD:R_0603_1608Metric
- R30: footprint (none) -> Resistor_SMD:R_2010_5025Metric; Mfr (none) -> HoLLR2010-1.5W-4mR-1%
- U10, U9: footprint DPAK_2E-T1_GE3_VIS -> SamacSys_Parts:DPAK_2E-T1_GE3_VIS
Connections:
- net shunt15+ is gone; now on net 15V_D: IC2.10 (IN+)
- net shunt15- is gone; now on net 15V_OUT: IC2.8 (VBUS), IC2.9 (IN-)
Other:
- moved on the sheet: C2, IC2
