File: Icky/24V_Interface.kicad_sch (KiCad schematic)
At the start: 21 parts, among them IC3 INA239AQDGSRQ1, IC9 LTC4368IMS-2#PBF, Q3 SOT233 BSS123N, U11 SQJQ112E-T1_GE3, U12 SQJQ112E-T1_GE3

Commit message: ERC passed
Connections:
- net SPI1_NSS3 renamed SPI1_NSS2
Changed lines of the file:
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@@
 	)
 	(rectangle
-		(start 20.32 38.1)
+		(start 19.05 38.1)
 		(end 157.48 125.73)
 		(stroke
@@
 	(text_box "DESIGN NOTE - TO COMPLETE"
 		(exclude_from_sim no)
-		(at 20.32 158.75 0)
+		(at 19.05 158.75 0)
 		(size 30.48 5.08)
 		(margins 1.3525 1.3525 1.3525 1.3525)
@@
 	(text_box "DESIGN NOTE - Loss / temperature\nPair hot resistance estimate about 16.5mOhm (worst case VGS and derated with the graph) Use Rds(on) vs Tj graph as reference\nPpair = I^2 x R = 10^2 x 0.0165 = 1.65W\nR_jtoamb = 40°C/W => 1.65W * 40°C/W = 66°C + 55° (Poland, summer, hot metal box) = 121 °C < 175 °C \n\n\n"
 		(exclude_from_sim no)
-		(at 20.32 128.27 0)
+		(at 19.05 128.27 0)
 		(size 90.17 15.24)
 		(margins 1.3525 1.3525 1.3525 1.3525)
@@
 	(text_box "DESIGN NOTE - Rating\nIn order to maintain the rating the PCB needs to be routed to ensure that 10 to 15A with some margin can pass"
 		(exclude_from_sim no)
-		(at 20.32 144.78 0)
+		(at 19.05 144.78 0)
 		(size 64.77 11.43)
 		(margins 1.3525 1.3525 1.3525 1.3525)
@@
 	)
 	(junction
-		(at 57.15 60.96)
+		(at 49.53 90.17)
 		(diameter 0)
 		(color 0 0 0 0)
 	)
 	(junction
-		(at 68.58 99.06)
+		(at 57.15 60.96)
 		(diameter 0)
 		(color 0 0 0 0)
 	)
 	(junction
-		(at 91.44 77.47)
+		(at 68.58 99.06)
 		(diameter 0)
 		(color 0 0 0 0)
 	)
 	(junction
-		(at 137.16 109.22)
+		(at 91.44 77.47)
 		(diameter 0)
 		(color 0 0 0 0)
 	)
 	(junction
-		(at 49.53 90.17)
+		(at 137.16 109.22)
 		(diameter 0)
 		(color 0 0 0 0)
@@
 	)
 	(bus_entry
-		(at 34.29 87.63)
+		(at 33.02 92.71)
 		(size 2.54 2.54)
 		(stroke
@@
 	)
 	(bus_entry
-		(at 34.29 92.71)
+		(at 33.02 90.17)
 		(size 2.54 2.54)
 		(stroke
@@
 	)
 	(bus_entry
-		(at 180.34 62.23)
+		(at 33.02 87.63)
 		(size 2.54 2.54)
 		(stroke
@@
 	)
 	(bus_entry
-		(at 34.29 90.17)
+		(at 180.34 62.23)
 		(size 2.54 2.54)
 		(stroke
@@
 		)
 	)
-	(bus
-		(pts
-			(xy 34.29 90.17) (xy 34.29 92.71)
-		)
-		(stroke
-			(width 0)
-			(type default)
-		)
-	)
 	(wire
 		(pts
@@
 		)
 	)
-	(bus
-		(pts
-			(xy 34.29 87.63) (xy 34.29 90.17)
-		)
-		(stroke
-			(width 0)
-			(type default)
-		)
-	)
 	(wire
 		(pts
@@
 		)
 	)
-	(wire
+	(bus
 		(pts
-			(xy 36.83 92.71) (xy 45.72 92.71)
+			(xy 33.02 87.63) (xy 33.02 90.17)
 		)
 		(stroke
@@
 	(wire
 		(pts
-			(xy 36.83 95.25) (xy 46.99 95.25)
+			(xy 68.58 110.49) (xy 68.58 109.22)
 		)
 		(stroke
@@
 	(wire
 		(pts
-			(xy 68.58 110.49) (xy 68.58 109.22)
+			(xy 68.58 119.38) (xy 57.15 119.38)
 		)
 		(stroke
@@
 	(wire
 		(pts
-			(xy 68.58 119.38) (xy 57.15 119.38)
+			(xy 224.79 74.93) (xy 227.33 74.93)
 		)
 		(stroke
@@
 	(wire
 		(pts
-			(xy 224.79 74.93) (xy 227.33 74.93)
+			(xy 68.58 90.17) (xy 68.58 88.9)
 		)
 		(stroke
@@
 		)
 	)
-	(wire
+	(bus
 		(pts
-			(xy 68.58 90.17) (xy 68.58 88.9)
+			(xy 33.02 87.63) (xy 31.75 86.36)
 		)
 		(stroke
@@
 	(wire
 		(pts
+			(xy 35.56 92.71) (xy 45.72 92.71)
+		)
+		(stroke
+			(width 0)
+			(type default)
+		)
+	)
+	(wire
+		(pts
 			(xy 224.79 64.77) (xy 241.3 64.77)
 		)
@@
 		)
 	)
+	(bus
+		(pts
+			(xy 33.02 90.17) (xy 33.02 92.71)
+		)
+		(stroke
+			(width 0)
+			(type default)
+		)
+	)
 	(wire
 		(pts
@@
 	(wire
 		(pts
+			(xy 35.56 95.25) (xy 45.72 95.25)
+		)
+		(stroke
+			(width 0)
+			(type default)
+		)
+	)
+	(wire
+		(pts
 			(xy 102.87 67.31) (xy 102.87 71.12)
 		)
@@
 	(wire
 		(pts
+			(xy 35.56 90.17) (xy 49.53 90.17)
+		)
+		(stroke
+			(width 0)
+			(type default)
+		)
+	)
+	(wire
+		(pts
 			(xy 95.25 60.96) (xy 95.25 69.85)
 		)
@@
 	(wire
 		(pts
-			(xy 36.83 90.17) (xy 49.53 90.17)
-		)
-		(stroke
-			(width 0)
-			(type default)
-		)
-	)
-	(wire
-		(pts
 			(xy 57.15 85.09) (xy 62.23 85.09)
 		)
@@
 		)
 	)
-	(bus
-		(pts
-			(xy 34.29 87.63) (xy 33.02 86.36)
-		)
-		(stroke
-			(width 0)
-			(type default)
-		)
-	)
 	(wire
 		(pts
@@
 		)
 	)
-	(label "24V_ALERT"
-		(at 46.99 95.25 180)
+	(label "24V_SHDN_PIN"
+		(at 149.86 88.9 180)
 		(effects
 			(font
@@
 		)
 	)
-	(label "24V_SHDN_PIN"
-		(at 149.86 88.9 180)
+	(label "SPI1_MOSI"
+		(at 182.88 67.31 0)
 		(effects
 			(font
 				(size 1.27 1.27)
 			)
-			(justify right bottom)
+			(justify left bottom)
 		)
 	)
-	(label "SPI1_MOSI"
-		(at 182.88 67.31 0)
+	(label "24V_ALERT"
+		(at 45.72 95.25 180)
 		(effects
 			(font
 				(size 1.27 1.27)
 			)
-			(justify left bottom)
+			(justify right bottom)
 		)
 	)
@@
 		)
 	)
+	(label "24V_SHDN"
+		(at 45.72 90.17 180)
+		(effects
+			(font
+				(size 1.27 1.27)
+			)
+			(justify right bottom)
+		)
+	)
 	(label "SPI1_MISO"
 		(at 182.88 69.85 0)
@@
 		)
 	)
-	(label "24V_SHDN"
-		(at 36.83 90.17 0)
-		(effects
-			(font
-				(size 1.27 1.27)
-			)
-			(justify left bottom)
-		)
-	)
 	(label "24V_OUT"
 		(at 124.46 60.96 0)
@@
 		)
 	)
-	(label "SPI1_NSS3"
+	(label "SPI1_NSS2"
 		(at 182.88 64.77 0)
 		(effects
@@
 		)
 	)
+	(hierarchical_label "{24V_PROT}"
+		(shape bidirectional)
+		(at 31.75 86.36 180)
+		(effects
+			(font
+				(size 1.27 1.27)
+			)
+			(justify right)
+		)
+	)
 	(hierarchical_label "24V_IN"
 		(shape input)
@@
 		)
 	)
-	(hierarchical_label "{24V_PROT}"
-		(shape bidirectional)
-		(at 33.02 86.36 180)
-		(effects
-			(font
-				(size 1.27 1.27)
-			)
-			(justify right)
-		)
-	)

Commit message: ERC passed v2
Changed lines of the file:
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@@
 		)
 	)
-	(hierarchical_label "{SPI_BAT}"
+	(hierarchical_label "{SPI_SENSORS}"
 		(shape bidirectional)
 		(at 177.165 60.96 180)

Commit message: routing
Parts:
- removed NT5: NetTieShuntH, 0_net_tie:NetTie-2_SMD_Pad0.2mm, symbol Device:NetTie_2
- removed NT6: NetTieShuntL, 0_net_tie:NetTie-2_SMD_Pad0.2mm, symbol Device:NetTie_2
- C25, C26, C35: footprint (none) -> Capacitor_SMD:C_0603_1608Metric
- C3: footprint 0_capacitor_smd:C_0402_1005_DensityHigh -> Capacitor_SMD:C_0603_1608Metric
- IC3: footprint 0_diode_smd:SOP50P490X110-10N -> SamacSys_Parts:SOP50P490X110-10N
- IC9: footprint SOP50P490X110-10N -> SamacSys_Parts:SOP50P490X110-10N
- Q3: footprint 0_package_SOT_TO_SMD:SOT-23-3 -> SamacSys_Parts:BSS123N
- R1, R3, R31, R32, R33, R34, R35, R36, R37: footprint (none) -> Resistor_SMD:R_0603_1608Metric
- R38: footprint (none) -> Resistor_SMD:R_2010_5025Metric; Mfr (none) -> HoLLR2010-1.5W-4mR-1%
- U11, U12: footprint DPAK_2E-T1_GE3_VIS -> SamacSys_Parts:DPAK_2E-T1_GE3_VIS
Connections:
- net shunt24+ is gone; now on net 24V_D: IC3.10 (IN+)
- net shunt24- is gone; now on net 24V_OUT: IC3.8 (VBUS), IC3.9 (IN-)
Other:
- moved on the sheet: C3, IC3
