File: Icky/Icky.kicad_pcb (KiCad board)
At the start: 6 copper layers, 98 x 77 mm, 129 parts, among them IC1 INA239AQDGSRQ1, IC2 INA239AQDGSRQ1, IC2001 INA239AQDGSRQ1, IC3 INA239AQDGSRQ1, IC4 LTC4368IMS-2#PBF, IC6 INA239AQDGSRQ1, IC801 TPS629206QDRLRQ1, J1 XT60PW-M, J10 Conn_SWD_10, J11 XT30AW-M, J12 XT30AW-M, J13 XT30AW-M, J14 XT30AW-M, J17 XT30UPB-F, J18 XT30UPB-F, J2 XT60PW-F, J3 XT30PW-F, J4 XT30PW-F, J403 USB4105-GF-A, J5 XT30PW-F, J6 XT30PW-F, J7 XT30UPB-F, J8 XT30UPB-F, Q3 ISC030N10NM6ATMA1, U1 STM32G483RET6, U2 TPS2116DRLR, U802 LMR36506MSC5RPERQ1, Y201 ABM8W-48.0000MHZ-4-D1X-T3

Commit message: routing
Parts:
- removed C2001: 100n X7R 50V, 0_capacitor_smd:C_0402_1005_DensityHigh
- removed C203: 12p NP0 25V, Capacitor_SMD:C_0402_1005Metric
- removed D13: SMCJ12A, Diode_SMD:D_SMA
- removed D14: SMCJ15A, Diode_SMD:D_SMA
- removed D15, D16: SMCJ24A, Diode_SMD:D_SMA
- removed D7: PTVS1-029C-H, Bucky:PTVS1029CH
- removed D9: SMCJ30A, Diode_SMD:D_SMA
- removed H501: M2 (3.2mm), MountingHole:MountingHole_2.2mm_M2_Pad_Via
- removed IC2001: INA239AQDGSRQ1, 0_diode_smd:SOP50P490X110-10N
- removed J12: XT30AW-M, Bucky:XT30AWM
- removed J18: XT30UPB-F, Bucky:XT30UPBF
- removed L802: 2u2, 0_inductor_smd:L_Coilcraft_LPS3314
- removed NT1, NT1601, NT3, NT5, NT7: NetTieShuntH, 0_net_tie:NetTie-2_SMD_Pad0.2mm
- removed NT1602, NT2, NT4, NT6, NT8: NetTieShuntL, 0_net_tie:NetTie-2_SMD_Pad0.2mm
- removed R1505: 3m, 0_resistor_smd:RES_WSLP3921_.003OHM_VIS
- added C15: 100n X7R 50V, Capacitor_SMD:C_0603_1608Metric, F.Cu at (304.8, 114.0)
- added C18: 17.5 nF X7R 25V, Capacitor_SMD:C_0603_1608Metric, F.Cu at (304.8, 116.5)
- added C19: 22 nF X7R 25V, Capacitor_SMD:C_0603_1608Metric, F.Cu at (304.8, 119.0)
- added C20: 470n X7R 50V, Capacitor_SMD:C_0603_1608Metric, F.Cu at (330.8, 116.5)
- added C22: 100n X7R 50V, Capacitor_SMD:C_0603_1608Metric, F.Cu at (330.8, 119.0)
- added C23: 17.5 nF X7R 25V, Capacitor_SMD:C_0603_1608Metric, F.Cu at (304.8, 99.4)
- added C24: 22 nF X7R 25V, Capacitor_SMD:C_0603_1608Metric, F.Cu at (304.8, 102.0)
- added C25: 17.5 nF X7R 25V, Capacitor_SMD:C_0603_1608Metric, F.Cu at (318.8, 99.4)
- added C26: 22 nF X7R 25V, Capacitor_SMD:C_0603_1608Metric, F.Cu at (318.8, 102.0)
- added C27: 17.5 nF X7R 25V, Capacitor_SMD:C_0603_1608Metric, F.Cu at (318.8, 116.5)
- added C28: 22 nF X7R 25V, Capacitor_SMD:C_0603_1608Metric, F.Cu at (318.8, 119.0)
- added C29: 100n X7R 50V, Capacitor_SMD:C_0603_1608Metric, F.Cu at (330.8, 121.5)
- added C30: 6.8 nF X7R 50V, Capacitor_SMD:C_0603_1608Metric, F.Cu at (324.8, 116.5)
- added C31: 10p NP0 25V, Capacitor_SMD:C_0603_1608Metric, F.Cu at (250.7, 55.0)
- added C32: 6.8 nF X7R 50V, Capacitor_SMD:C_0603_1608Metric, F.Cu at (304.8, 121.5)
- added C34: 6.8 nF X7R 50V, Capacitor_SMD:C_0603_1608Metric, F.Cu at (304.8, 104.5)
- added C35: 6.8 nF X7R 50V, Capacitor_SMD:C_0603_1608Metric, F.Cu at (318.8, 104.5)
- added C4: 100n X7R 50V, Capacitor_SMD:C_0603_1608Metric, F.Cu at (304.8, 128.5)
- added D1: ESDS314DBVR, Bucky:SOT95P280X145-5N, F.Cu at (309.4, 129.6)
- added D17: SMCJ5.0CA, Diode_SMD:D_SMA, F.Cu at (46.1, -50.1)
- added D19: SMCJ15CA, Diode_SMD:D_SMA, F.Cu at (125.4, 117.3)
- added D20: SMCJ24CA, Diode_SMD:D_SMA, F.Cu at (108.8, -41.0)
- added D21: SMCJ30CA, Diode_SMD:D_SMA, F.Cu at (136.0, 49.2)
- added H4: M2 (2.2mm), MountingHole:MountingHole_2.2mm_M2_Pad_Via, F.Cu at (60.0, 122.0)
- added IC10: LTC4368IMS-2#PBF, SamacSys_Parts:SOP50P490X110-10N, F.Cu at (287.4, 123.5)
- added IC5: INA239AQDGSRQ1, SamacSys_Parts:SOP50P490X110-10N, F.Cu at (261.8, 68.2)
- added IC7: INA239AQDGSRQ1, SamacSys_Parts:SOP50P490X110-10N, F.Cu at (61.7, -32.5)
- added IC8: LTC4368IMS-2#PBF, SamacSys_Parts:SOP50P490X110-10N, F.Cu at (131.3, 100.8)
- added IC9: LTC4368IMS-2#PBF, SamacSys_Parts:SOP50P490X110-10N, F.Cu at (266.0, 97.0)
- added L5: 2u2, Inductor_SMD:L_1008_2520Metric, F.Cu at (270.2, 50.6)
- added Q1: SOT233 BSS123N, SamacSys_Parts:BSS123N, F.Cu at (229.5, 130.3)
- added Q2: SOT233 BSS123N, SamacSys_Parts:BSS123N, F.Cu at (229.5, 122.3)
- added Q4: SOT233 BSS123N, SamacSys_Parts:BSS123N, F.Cu at (237.5, 122.3)
- added R10: 100k 1% 1/16W, Resistor_SMD:R_0603_1608Metric, F.Cu at (308.8, 124.0)
- added R11: 100k 1% 1/16W, Resistor_SMD:R_0603_1608Metric, F.Cu at (312.8, 114.0)
- added R12: 100k 1%, Resistor_SMD:R_0603_1608Metric, F.Cu at (304.8, 131.1)
- added R13: 10 1% 1/16W, Resistor_SMD:R_0603_1608Metric, F.Cu at (324.8, 119.0)
- added R14: 10 1% 1/16W, Resistor_SMD:R_0603_1608Metric, F.Cu at (324.8, 121.5)
- added R15: 10 1% 1/16W, Resistor_SMD:R_0603_1608Metric, F.Cu at (324.8, 124.0)
- added R16: 10 1% 1/16W, Resistor_SMD:R_0603_1608Metric, F.Cu at (324.8, 126.5)
- added R17: 120k 1% 1/16W, Resistor_SMD:R_0603_1608Metric, F.Cu at (244.6, 102.4)
- added R18: 10 1% 1/16W, Resistor_SMD:R_0603_1608Metric, F.Cu at (312.8, 116.5)
- added R19: 10 1% 1/16W, Resistor_SMD:R_0603_1608Metric, F.Cu at (312.8, 119.0)
- added R20: 1m 1% 8W, SamacSys_Parts:WSL39211L000JEA, F.Cu at (79.3, 84.5)
- added R21: 100k 1% 1/16W, Resistor_SMD:R_0603_1608Metric, F.Cu at (330.8, 126.5)
- added R22: 100k 1% 1/16W, Resistor_SMD:R_0603_1608Metric, F.Cu at (304.8, 107.0)
- added R23: 100k 1% 1/16W, Resistor_SMD:R_0603_1608Metric, F.Cu at (304.8, 109.5)
- added R24: 6.8M 1% 1/16W, Resistor_SMD:R_0603_1608Metric, F.Cu at (308.8, 99.4)
- added R25: 56k 1% 1/16W, Resistor_SMD:R_0603_1608Metric, F.Cu at (308.8, 102.0)
- added R26: 330k 1% 1/16W, Resistor_SMD:R_0603_1608Metric, F.Cu at (308.8, 104.5)
- added R27: 22k 1% 1/16W, Resistor_SMD:R_0603_1608Metric, F.Cu at (308.8, 107.0)
- added R28: 10 1% 1/16W, Resistor_SMD:R_0603_1608Metric, F.Cu at (308.8, 109.5)
- added R29: 10 1% 1/16W, Resistor_SMD:R_0603_1608Metric, F.Cu at (312.8, 99.4)
- added R30: 4m, Resistor_SMD:R_2010_5025Metric, F.Cu at (126.8, 95.0)
- added R31: 100k 1% 1/16W, Resistor_SMD:R_0603_1608Metric, F.Cu at (318.8, 107.0)
- added R32: 15M 1% 1/16W, Resistor_SMD:R_0603_1608Metric, F.Cu at (318.8, 109.5)
- added R33: 39k 1% 1/16W, Resistor_SMD:R_0603_1608Metric, F.Cu at (318.8, 112.0)
- added R34: 300k 1% 1/16W, Resistor_SMD:R_0603_1608Metric, F.Cu at (322.8, 99.4)
- added R35: 22k 1% 1/16W, Resistor_SMD:R_0603_1608Metric, F.Cu at (322.8, 102.0)
- added R36: 10 1% 1/16W, Resistor_SMD:R_0603_1608Metric, F.Cu at (322.8, 104.5)
- added R37: 10 1% 1/16W, Resistor_SMD:R_0603_1608Metric, F.Cu at (322.8, 107.0)
- added R38: 4m, Resistor_SMD:R_2010_5025Metric, F.Cu at (102.5, -16.5)
- added R39: 10k 1% 1/16W, Resistor_SMD:R_0603_1608Metric, F.Cu at (304.8, 133.6)
- added R4: 470k 1% 1/16W, Resistor_SMD:R_0603_1608Metric, F.Cu at (304.8, 124.0)
- added R40: 100k 1% 1/16W, Resistor_SMD:R_0603_1608Metric, F.Cu at (318.8, 121.5)
- added R41: 20M 1% 1/16W, Resistor_SMD:R_0603_1608Metric, F.Cu at (318.8, 124.0)
- added R42: 120k 1% 1/16W, Resistor_SMD:R_0603_1608Metric, F.Cu at (318.8, 126.5)
- added R43: 330k 1% 1/16W, Resistor_SMD:R_0603_1608Metric, F.Cu at (318.8, 129.1)
- added R44: 10 1% 1/16W, Resistor_SMD:R_0603_1608Metric, F.Cu at (330.8, 129.1)
- added R45: 10 1% 1/16W, Resistor_SMD:R_0603_1608Metric, F.Cu at (330.8, 131.6)
- added R46: 100k 1% 1/16W, Resistor_SMD:R_0603_1608Metric, F.Cu at (312.8, 104.5)
- added R5: 4m, Resistor_SMD:R_2010_5025Metric, F.Cu at (56.2, -25.6)
- added R52: 100k 1% 1/16W, Resistor_SMD:R_0603_1608Metric, F.Cu at (312.8, 121.5)
- added R53: 10k 1% 1/16W, Resistor_SMD:R_0603_1608Metric, F.Cu at (244.6, 104.9)
- added R54: 10k 1% 1/16W, Resistor_SMD:R_0603_1608Metric, F.Cu at (244.6, 107.4)
- added R55: 22k 1% 1/16W, Resistor_SMD:R_0603_1608Metric, F.Cu at (244.6, 109.9)
- added R56: 100k 1% 1/16W, Resistor_SMD:R_0603_1608Metric, F.Cu at (330.8, 134.1)
- added R57: 10 1% 1/16W, Resistor_SMD:R_0603_1608Metric, F.Cu at (324.8, 129.1)
- added R58: 22k 1% 1/16W, Resistor_SMD:R_0603_1608Metric, F.Cu at (318.8, 131.6)
- added R59: 10 1% 1/16W, Resistor_SMD:R_0603_1608Metric, F.Cu at (324.8, 131.6)
- added R6: 150k 1% 1/16W, Resistor_SMD:R_0603_1608Metric, F.Cu at (308.8, 116.5)
- added R62: 100k 1% 1/16W, Resistor_SMD:R_0603_1608Metric, F.Cu at (318.8, 134.1)
- added R7: 4.75M 1% 1/16W, Resistor_SMD:R_0603_1608Metric, F.Cu at (308.8, 119.0)
- added R9: 22k 1% 1/16W, Resistor_SMD:R_0603_1608Metric, F.Cu at (308.8, 121.5)
- added U10: SQJQ112E-T1_GE3, SamacSys_Parts:DPAK_2E-T1_GE3_VIS, F.Cu at (118.5, 101.1)
- added U11: SQJQ112E-T1_GE3, SamacSys_Parts:DPAK_2E-T1_GE3_VIS, F.Cu at (109.0, -33.7)
- added U12: SQJQ112E-T1_GE3, SamacSys_Parts:DPAK_2E-T1_GE3_VIS, F.Cu at (109.0, -20.6)
- added U13: SQJQ112E-T1_GE3, SamacSys_Parts:DPAK_2E-T1_GE3_VIS, F.Cu at (92.3, 48.1)
- added U14: SQJQ112E-T1_GE3, SamacSys_Parts:DPAK_2E-T1_GE3_VIS, F.Cu at (108.3, 48.3)
- added U15: SQJQ112E-T1_GE3, SamacSys_Parts:DPAK_2E-T1_GE3_VIS, F.Cu at (108.0, 59.4)
- added U16: SQJQ112E-T1_GE3, SamacSys_Parts:DPAK_2E-T1_GE3_VIS, F.Cu at (108.2, 71.2)
- added U17: SQJQ112E-T1_GE3, SamacSys_Parts:DPAK_2E-T1_GE3_VIS, F.Cu at (62.0, 96.3)
- added U3: SQJQ112E-T1_GE3, SamacSys_Parts:DPAK_2E-T1_GE3_VIS, F.Cu at (92.7, 71.1)
- added U4: SamacSys_Parts:DPAK_2E-T1_GE3_VIS, Bucky:DPAK_2E-T1_GE3_VIS, F.Cu at (92.5, 59.6)
- added U5: SQJQ112E-T1_GE3, SamacSys_Parts:DPAK_2E-T1_GE3_VIS, F.Cu at (51.0, -43.2)
- added U6: SQJQ112E-T1_GE3, SamacSys_Parts:DPAK_2E-T1_GE3_VIS, F.Cu at (51.0, -33.8)
- added U7: SQJQ112E-T1_GE3, SamacSys_Parts:DPAK_2E-T1_GE3_VIS, F.Cu at (84.1, 96.6)
- added U8: SQJQ112E-T1_GE3, SamacSys_Parts:DPAK_2E-T1_GE3_VIS, F.Cu at (73.2, 96.5)
- added U9: SQJQ112E-T1_GE3, SamacSys_Parts:DPAK_2E-T1_GE3_VIS, F.Cu at (128.0, 110.8)
- C1: value 100n X7R 50V -> 6.8 nF X7R 50V; footprint 0_capacitor_smd:C_0402_1005_DensityHigh -> Capacitor_SMD:C_0603_1608Metric; moved to F.Cu
- C10, C11, C12, C13, C14, C7: footprint Capacitor_SMD:C_1812_4532Metric_Pad1.57x3.40mm_HandSolder -> Capacitor_SMD:C_0603_1608Metric
- C16, C17, C21, C403, C417, C9: footprint 0_capacitor_smd:C_0402_1005_DensityHigh -> Capacitor_SMD:C_0603_1608Metric
- C2, C3, C406, C407, C408, C409, C410, C412, C413, C414, C415, C416, C8, C808, C809, C814, C815, C816, C818, C820: footprint 0_capacitor_smd:C_0402_1005_DensityHigh -> Capacitor_SMD:C_0603_1608Metric; moved to F.Cu
- C207: value 12p NP0 25V -> 10p NP0 25V; footprint Capacitor_SMD:C_0402_1005Metric -> Capacitor_SMD:C_0603_1608Metric; moved to F.Cu
- C411, C813: footprint 0_capacitor_smd:C_0603_1608_DensityHigh -> Capacitor_SMD:C_0603_1608Metric; moved to F.Cu
- C5: value 100u -> 6.8 nF X7R 50V; footprint Capacitor_SMD:C_1812_4532Metric_Pad1.57x3.40mm_HandSolder -> Capacitor_SMD:C_0603_1608Metric
- C6: value 100u -> 100n X7R 50V; footprint Capacitor_SMD:C_1812_4532Metric_Pad1.57x3.40mm_HandSolder -> Capacitor_SMD:C_0603_1608Metric
- C806: footprint 0_capacitor_smd:C_1210_3225_DensityHigh -> Capacitor_SMD:C_0603_1608Metric; moved to F.Cu
- C807, C810, C811: footprint 0_capacitor_smd:C_0805_2012_DensityHigh -> Capacitor_SMD:C_0603_1608Metric; moved to F.Cu
- C812: footprint 0_resistor_smd:R_0805_2012_DensityHigh -> Capacitor_SMD:C_0603_1608Metric; moved to F.Cu
- C817: footprint 0_capacitor_smd:C_0805_2012_DensityHighest -> Capacitor_SMD:C_0603_1608Metric; moved to F.Cu
- D10, D8: value SMCJ30A -> SMCJ30CA
- D11: value SMCJ30A -> SMCJ5.0CA
- D12: value SMCJ5.0A -> 5.0SMDJ30CA; footprint Diode_SMD:D_SMA -> Bucky:DIONM7959X262N
- D3: value SMCJ5.0A -> SMCJ24CA
- D4: value SMCJ15A -> SMCJ15CA
- D5: value PTVS1-029C-H -> 5.0SMDJ30CA; footprint Bucky:PTVS1029CH -> Bucky:DIONM7959X262N
- D6: value SMCJ12A -> 5.0SMDJ30CA; footprint Diode_SMD:D_SMA -> Bucky:DIONM7959X262N
- FB201, U1: moved to F.Cu
- FB801: footprint 0_resistor_smd:R_0805_2012_DensityHigh -> Resistor_SMD:R_0805_2012Metric; moved to F.Cu
- H1, H2, H3: value M2 (3.2mm) -> M2 (2.2mm)
- IC1: value INA239AQDGSRQ1 -> LM5069MM-2_NOPB; footprint 0_diode_smd:SOP50P490X110-10N -> SamacSys_Parts:SOP50P490X110-10N; moved to F.Cu
- IC2, IC3, IC6: footprint 0_diode_smd:SOP50P490X110-10N -> SamacSys_Parts:SOP50P490X110-10N; moved to F.Cu
- IC4: footprint Bucky:SOP50P490X110-10N -> SamacSys_Parts:SOP50P490X110-10N; moved to F.Cu
- IC801, U2: footprint 0_switching_regulator:SOTFL50P160X60-8N -> SamacSys_Parts:SOTFL50P160X60-8N; moved to F.Cu
- J3, J4, J5: value XT30PW-F -> XT30UPB-F; footprint Bucky:XT30PWF -> Bucky:XT30UPBF
- J6: value XT30PW-F -> XT60PW-F; footprint Bucky:XT30PWF -> Bucky:XT60PWF
- L803: footprint 0_inductor_smd:L_Coilcraft_LPS4018 -> Inductor_SMD:L_Coilcraft_LPS4018; moved to F.Cu
- Q3: value ISC030N10NM6ATMA1 -> SOT233 BSS123N; footprint Bucky:ISC030N10NM6ATMA1 -> SamacSys_Parts:BSS123N
- R1, R3: value 3m -> 100k 1% 1/16W; footprint 0_resistor_smd:RES_WSLP3921_.003OHM_VIS -> Resistor_SMD:R_0603_1608Metric; moved to F.Cu
- R2: value 3m -> 400k 1%; footprint 0_resistor_smd:RES_WSLP3921_.003OHM_VIS -> Resistor_SMD:R_0603_1608Metric; moved to F.Cu
- R402, R403, R407, R408: footprint 0_resistor_smd:R_0402_1005_DensityHigh -> Resistor_SMD:R_0603_1608Metric
- R405, R47, R48, R49, R50, R802, R803, R804, R805, R806: footprint 0_resistor_smd:R_0402_1005_DensityHigh -> Resistor_SMD:R_0603_1608Metric; moved to F.Cu
- R51: value 10k 1% 1/16W -> 10 1% 1/16W; footprint 0_resistor_smd:R_0402_1005_DensityHigh -> Resistor_SMD:R_0603_1608Metric; moved to F.Cu
- R8: value WSL39211L000FEA -> 1m 1% 8W; footprint Bucky:WSL39211L000JEA -> SamacSys_Parts:WSL39211L000JEA; moved to F.Cu
- R801: footprint 0_resistor_smd:R_0603_1608_DensityHigh -> Resistor_SMD:R_0603_1608Metric; moved to F.Cu
- U802: value LMR36506MSC5RPERQ1 -> LMR36506MSCQRPERQ1; footprint 0_switching_regulator:LMR36503 -> SamacSys_Parts:LMR36506MSC5RPERQ1; moved to F.Cu
- Y201: value ABM8W-48.0000MHZ-4-D1X-T3 -> ABM8W-48.0000MHZ-7-D1X-T3; footprint 0_diode_smd:ABM8W480000MHZ6D1XT3 -> SamacSys_Parts:ABM8W480000MHZ6D1XT3; moved to F.Cu
- moved D11 194.0 mm to (45.7, -26.8)
- moved C16 156.4 mm to (211.3, 41.9), turned to 0 degrees
- moved D5 151.2 mm to (79.2, 60.4), turned to 90 degrees
- moved C21 140.3 mm to (211.3, 46.9), turned to 0 degrees
- moved J11 139.2 mm to (48.3, -56.0), turned to 180 degrees
- moved C8 137.1 mm to (220.7, 51.4), turned to 0 degrees
- moved C1 133.7 mm to (226.8, 51.4)
- moved U802 130.2 mm to (272.9, 61.4), turned to 0 degrees
- moved L803 130.2 mm to (272.5, 66.9), turned to 0 degrees
- moved J14 130.0 mm to (106.2, -47.4), turned to 0 degrees
- moved D3 127.8 mm to (108.4, -13.1), turned to 180 degrees
- moved FB801 127.4 mm to (270.0, 53.9), turned to 0 degrees
- moved IC801 125.2 mm to (254.5, 55.5), turned to 0 degrees
- moved J8 122.5 mm to (48.9, -20.7)
- moved D12 120.8 mm to (78.3, 72.0), turned to -90 degrees
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Connections:
- net /Project Architecture/MCU & Local Power/5V alert renamed /Project Architecture/MCU & Local Power/5V_ALERT
- net /Project Architecture/MCU & Local Power/input alert renamed /Project Architecture/MCU & Local Power/VIN_ALERT
- C1 pad 1: +3V3 -> Net-(C1-Pad1)
- C1 pad 2: GND -> /Project Architecture/Protection & Monitoring/VIN_MOS/GATE
- C10 pad 1: /Project Architecture/PowerConnectors/15V_safe -> /Project Architecture/PowerConnectors/15V_VSAFE
- C11 pad 1: /Project Architecture/PowerConnectors/24V_safe -> /Project Architecture/PowerConnectors/24V_VSAFE
- C12 pad 1: /Project Architecture/PowerConnectors/5V_safe -> /Project Architecture/PowerConnectors/5V_VSAFE
- C13 pad 1: /Project Architecture/PowerConnectors/5V_safe -> /Project Architecture/PowerConnectors/5V_VSAFE
- C14 pad 1: /Project Architecture/PowerConnectors/24V_safe -> /Project Architecture/PowerConnectors/24V_VSAFE
- C5 pad 1: /Project Architecture/PowerConnectors/12V_safe -> Net-(C5-Pad1)
- C5 pad 2: GND -> /Project Architecture/Protection & Monitoring/VIN_MOS/GATE
- C6 pad 1: /Project Architecture/PowerConnectors/12V_safe -> VBAT
- C7 pad 1: /Project Architecture/PowerConnectors/15V_safe -> /Project Architecture/PowerConnectors/15V_VSAFE
- C810 pad 1: /Project Architecture/PowerConnectors/VBuck_in -> /Project Architecture/Protection & Monitoring/VIN_OUT
- D10 pad 1: /Project Architecture/PowerConnectors/VBuck_in -> GND
- D10 pad 2: GND -> /Project Architecture/Protection & Monitoring/VIN_OUT
- D11 pad 1: /Project Architecture/PowerConnectors/VBuck_in -> GND
- D11 pad 2: GND -> /Project Architecture/PowerConnectors/5V_VSAFE
- D12 pad 1: /Project Architecture/PowerConnectors/5V_safe -> GND
- D12 pad 2: GND -> VBAT
- D3 pad 1: /Project Architecture/PowerConnectors/Vin_5V -> GND
- D3 pad 2: GND -> /Project Architecture/PowerConnectors/24V_VSAFE
- D4 pad 1: /Project Architecture/PowerConnectors/Vin_15V -> /Project Architecture/PowerConnectors/15V_VSAFE
- D5 pad 2: /Project Architecture/PowerConnectors/VBuck_in -> VBAT
- D6 pad 1: /Project Architecture/PowerConnectors/Vin_12V -> GND
- D6 pad 2: GND -> /Project Architecture/PowerConnectors/VMOT_OUT
- D8 pad 1: /Project Architecture/PowerConnectors/VBuck_in -> GND
- D8 pad 2: GND -> /Project Architecture/Protection & Monitoring/VIN_OUT
- FB801 pad 1: /Project Architecture/PowerConnectors/VBuck_in -> /Project Architecture/Protection & Monitoring/VIN_OUT
- IC1 pad 1: /Project Architecture/MCU & Local Power/SPI1_NSS1 -> /Project Architecture/Protection & Monitoring/VMOT/VMOT_SENS-
- IC1 pad 10: /Project Architecture/Sensors/shunt12+ -> Net-(IC1-GATE)
- IC1 pad 2: /Project Architecture/MCU & Local Power/SPI1_MOSI -> VBAT
- IC1 pad 3: /Project Architecture/MCU & Local Power/15V alert -> Net-(IC1-UVLO)
- IC1 pad 4: /Project Architecture/MCU & Local Power/SPI1_MISO -> Net-(IC1-OVLO)
- IC1 pad 5: /Project Architecture/MCU & Local Power/SPI1_SCK -> GND
- IC1 pad 6: +3V3 -> Net-(IC1-TIMER)
- IC1 pad 7: GND -> Net-(IC1-PWR)
- IC1 pad 8: /Project Architecture/Sensors/shunt12- -> /Project Architecture/MCU & Local Power/PG_VMOT
- IC1 pad 9: /Project Architecture/Sensors/shunt12- -> /Project Architecture/PowerConnectors/VMOT_OUT
- IC2 pad 1: /Project Architecture/MCU & Local Power/SPI1_NSS2 -> /Project Architecture/MCU & Local Power/SPI1_NSS1
- IC2 pad 10: /Project Architecture/Sensors/shunt15+ -> /Project Architecture/Protection & Monitoring/15V/15V_D
- IC2 pad 3: /Project Architecture/MCU & Local Power/12V alert -> /Project Architecture/MCU & Local Power/15V_ALERT
- IC2 pad 8: /Project Architecture/Sensors/shunt15- -> /Project Architecture/PowerConnectors/15V_VSAFE
- IC2 pad 9: /Project Architecture/Sensors/shunt15- -> /Project Architecture/PowerConnectors/15V_VSAFE
- IC3 pad 1: /Project Architecture/MCU & Local Power/SPI1_NSS3 -> /Project Architecture/MCU & Local Power/SPI1_NSS2
- IC3 pad 10: /Project Architecture/Sensors/shunt24+ -> /Project Architecture/Protection & Monitoring/24V/24V_D
- IC3 pad 3: /Project Architecture/MCU & Local Power/24V alert -> /Project Architecture/MCU & Local Power/24V_ALERT
- IC3 pad 8: /Project Architecture/Sensors/shunt24- -> /Project Architecture/PowerConnectors/24V_VSAFE
- IC3 pad 9: /Project Architecture/Sensors/shunt24- -> /Project Architecture/PowerConnectors/24V_VSAFE
- IC4 pad 1: unconnected-(IC4-VIN-Pad1) -> /Project Architecture/PowerConnectors/5V_VBUCK
- IC4 pad 10: unconnected-(IC4-GATE-Pad10) -> Net-(IC4-GATE)
- IC4 pad 2: unconnected-(IC4-UV-Pad2) -> Net-(IC4-UV)
- IC4 pad 3: unconnected-(IC4-OV-Pad3) -> Net-(IC4-OV)
- IC4 pad 4: unconnected-(IC4-RETRY-Pad4) -> Net-(IC4-RETRY)
- IC4 pad 5: unconnected-(IC4-GND-Pad5) -> GND
- IC4 pad 6: unconnected-(IC4-~{SHDN}-Pad6) -> /Project Architecture/Protection & Monitoring/5V/5V_SHDN_PIN
- IC4 pad 7: unconnected-(IC4-~{FAULT}-Pad7) -> /Project Architecture/MCU & Local Power/5V_FLT
- IC4 pad 8: unconnected-(IC4-VOUT-Pad8) -> /Project Architecture/PowerConnectors/5V_VSAFE
- IC4 pad 9: unconnected-(IC4-SENSE-Pad9) -> /Project Architecture/Protection & Monitoring/5V/5V_D
- IC6 pad 1: /Project Architecture/MCU & Local Power/SPI1_NSS4 -> /Project Architecture/MCU & Local Power/SPI1_NSS3
- IC6 pad 10: /Project Architecture/Sensors/shuntBatt+ -> /Project Architecture/Protection & Monitoring/VIN_D
- IC6 pad 8: /Project Architecture/Sensors/shuntBatt- -> /Project Architecture/Protection & Monitoring/VIN_OUT
- IC6 pad 9: /Project Architecture/Sensors/shuntBatt- -> /Project Architecture/Protection & Monitoring/VIN_OUT
- J1 pad 2: /Project Architecture/PowerConnectors/VBatt_in -> VBAT
- J11 pad 1: /Project Architecture/PowerConnectors/Vin_5V -> /Project Architecture/PowerConnectors/5V_VBUCK
- J13 pad 1: /Project Architecture/PowerConnectors/Vin_15V -> /Project Architecture/PowerConnectors/15V_VBUCK
- J14 pad 1: /Project Architecture/PowerConnectors/Vin_24V -> /Project Architecture/PowerConnectors/24V_VBUCK
- J17 pad 1: /Project Architecture/PowerConnectors/VBuck_in -> /Project Architecture/Protection & Monitoring/VIN_OUT
- J2 pad 1: /Project Architecture/PowerConnectors/VBuck_in -> VBAT
- J3 pad 1: GND -> /Project Architecture/PowerConnectors/15V_VSAFE
- J3 pad 2: /Project Architecture/PowerConnectors/5V_safe -> GND
- J4 pad 1: GND -> /Project Architecture/PowerConnectors/24V_VSAFE
- J4 pad 2: /Project Architecture/PowerConnectors/12V_safe -> GND
- J5 pad 1: GND -> /Project Architecture/Protection & Monitoring/VIN_OUT
- J5 pad 2: /Project Architecture/PowerConnectors/15V_safe -> GND
- J6 pad 1: GND -> /Project Architecture/PowerConnectors/VMOT_OUT
- J6 pad 2: /Project Architecture/PowerConnectors/24V_safe -> GND
- J7 pad 1: /Project Architecture/PowerConnectors/VBuck_in -> /Project Architecture/Protection & Monitoring/VIN_OUT
- J8 pad 1: /Project Architecture/PowerConnectors/VBuck_in -> /Project Architecture/PowerConnectors/5V_VSAFE
- Q3 pad 1: unconnected-(Q3-S_1-Pad1) -> /Project Architecture/MCU & Local Power/24V_SHDN
- Q3 pad 2: unconnected-(Q3-S_2-Pad2) -> GND
- Q3 pad 3: unconnected-(Q3-S_3-Pad3) -> /Project Architecture/Protection & Monitoring/24V/24V_SHDN_PIN
- R1 pad 1: /Project Architecture/PowerConnectors/Vin_15V -> /Project Architecture/MCU & Local Power/24V_SHDN
- R1 pad 2: /Project Architecture/ProtectionCircuitry/out15V -> GND
- R2 pad 1: /Project Architecture/PowerConnectors/Vin_12V -> Net-(U802-FB)
- R2 pad 2: /Project Architecture/ProtectionCircuitry/out12V -> Net-(U2-MODE)
- R3 pad 1: /Project Architecture/PowerConnectors/Vin_24V -> +3V3
- R3 pad 2: /Project Architecture/ProtectionCircuitry/out24V -> /Project Architecture/MCU & Local Power/24V_FLT
- R48 pad 1: /Project Architecture/MCU & Local Power/24V alert -> /Project Architecture/MCU & Local Power/15V_ALERT
- R50 pad 1: /Project Architecture/MCU & Local Power/15V alert -> /Project Architecture/MCU & Local Power/24V_ALERT
- R51 pad 1: /Project Architecture/MCU & Local Power/12V alert -> Net-(IC1-GATE)
- R51 pad 2: +3V3 -> Net-(U8-G)
- R8 pad 1: /Project Architecture/PowerConnectors/VBatt_in -> /Project Architecture/Protection & Monitoring/VIN_OUT
- R8 pad 2: /Project Architecture/Sensors/outBatt -> /Project Architecture/Protection & Monitoring/VIN_D
- U1 pad 10: /Project Architecture/MCU & Local Power/PG_5V -> unconnected-(U1A-PC2-Pad10)
- U1 pad 11: /Project Architecture/MCU & Local Power/PG_12V -> unconnected-(U1A-PC3-Pad11)
- U1 pad 12: /Project Architecture/MCU & Local Power/24V alert -> /Project Architecture/MCU & Local Power/15V_ALERT
- U1 pad 13: /Project Architecture/MCU & Local Power/15V alert -> /Project Architecture/MCU & Local Power/24V_ALERT
- U1 pad 14: /Project Architecture/MCU & Local Power/12V alert -> unconnected-(U1A-PA2-Pad14)
- U1 pad 17: /Project Architecture/MCU & Local Power/MV5_SHDN -> /Project Architecture/MCU & Local Power/5V_SHDN
- U1 pad 22: /Project Architecture/MCU & Local Power/PG_15V -> /Project Architecture/MCU & Local Power/VMOT_SHDN
- U1 pad 23: /Project Architecture/MCU & Local Power/PG_24V -> /Project Architecture/MCU & Local Power/PG_VMOT
- U1 pad 25: /Project Architecture/MCU & Local Power/fan -> unconnected-(U1A-PB1-Pad25)
- U1 pad 3: unconnected-(U1A-PC14-Pad3) -> /Project Architecture/MCU & Local Power/VIN_FLT
- U1 pad 35: unconnected-(U1A-PB13-Pad35) -> /Project Architecture/MCU & Local Power/5V_FLT
- U1 pad 36: unconnected-(U1A-PB14-Pad36) -> /Project Architecture/MCU & Local Power/15V_FLT
- U1 pad 37: unconnected-(U1A-PB15-Pad37) -> /Project Architecture/MCU & Local Power/24V_FLT
- U1 pad 38: /Project Architecture/MCU & Local Power/PG_Batt -> /Project Architecture/MCU & Local Power/VMOT_ALERT
- U1 pad 39: /Project Architecture/MCU & Local Power/INT -> unconnected-(U1A-PC7-Pad39)
- U1 pad 44: /Project Architecture/MCU & Local Power/MV12_SHDN -> unconnected-(U1A-PA10-Pad44)
- U1 pad 57: /Project Architecture/MCU & Local Power/MV15_SHDN -> /Project Architecture/MCU & Local Power/15V_SHDN
- U1 pad 60: /Project Architecture/MCU & Local Power/MV24_SHDN -> /Project Architecture/MCU & Local Power/24V_SHDN
- U802 pad 8: Net-(U2-MODE) -> Net-(U802-FB)
Routing:
- net +3V3: track 363.2 -> 0.00 mm, vias 19 -> 0
- net (no net): track 361.8 -> 0.00 mm, vias 374 -> 27
- net /Project Architecture/MCU & Local Power/5V_ALERT: track 152.1 -> 0.00 mm, vias 2 -> 0
- net /Project Architecture/MCU & Local Power/SPI1_MISO: track 141.7 -> 0.00 mm, vias 6 -> 0
- net /Project Architecture/MCU & Local Power/SPI1_SCK: track 130.6 -> 0.00 mm, vias 6 -> 0
- net /Project Architecture/MCU & Local Power/SPI1_MOSI: track 122.8 -> 0.00 mm, vias 6 -> 0
- net /Project Architecture/MCU & Local Power/SPI1_NSS4: track 100.0 -> 0.00 mm, vias 2 -> 0
- net /Project Architecture/PowerConnectors/12V_safe: track 96.4 -> 0.00 mm, vias 56 -> 0
- net /Project Architecture/MCU & Local Power/PG_5V: track 92.6 -> 0.00 mm, vias 4 -> 0
- net /Project Architecture/MCU & Local Power/SPI1_NSS0: track 92.1 -> 0.00 mm, vias 4 -> 0
- net +5V: track 89.5 -> 0.00 mm, vias 1 -> 0
- net /Project Architecture/MCU & Local Power/MV5_SHDN: track 84.7 -> 0.00 mm, vias 2 -> 0
- net /Project Architecture/MCU & Local Power/VIN_ALERT: track 82.0 -> 0.00 mm, vias 2 -> 0
- net /Project Architecture/MCU & Local Power/15V alert: track 71.4 -> 0.00 mm, vias 4 -> 0
- net /Project Architecture/MCU & Local Power/MV12_SHDN: track 69.9 -> 0.00 mm, vias 3 -> 0
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- removed copper zone on B.Cu, net (none)
- removed copper zone on F.Cu, net (none)
- removed copper zone on In2.Cu, net (none)
- removed copper zone on B.Cu, net /Project Architecture/PowerConnectors/12V_safe
- removed copper zone on F.Cu, net /Project Architecture/PowerConnectors/12V_safe
- removed copper zone on In2.Cu, net /Project Architecture/PowerConnectors/12V_safe
- removed copper zone on B.Cu, net /Project Architecture/PowerConnectors/15V_safe
- removed copper zone on F.Cu, net /Project Architecture/PowerConnectors/15V_safe
- removed copper zone on In2.Cu, net /Project Architecture/PowerConnectors/15V_safe
- removed copper zone on B.Cu, net /Project Architecture/PowerConnectors/24V_safe
- removed copper zone on F.Cu, net /Project Architecture/PowerConnectors/24V_safe
- removed copper zone on In2.Cu, net /Project Architecture/PowerConnectors/24V_safe
- removed copper zone on B.Cu, net /Project Architecture/PowerConnectors/5V_safe
- removed copper zone on F.Cu, net /Project Architecture/PowerConnectors/5V_safe
- removed copper zone on In2.Cu, net /Project Architecture/PowerConnectors/5V_safe
- removed copper zone on B.Cu, net /Project Architecture/PowerConnectors/VBatt_in
- removed copper zone on F.Cu, net /Project Architecture/PowerConnectors/VBatt_in
- removed copper zone on In2.Cu, net /Project Architecture/PowerConnectors/VBatt_in
- removed copper zone on B.Cu, net /Project Architecture/PowerConnectors/VBuck_in
- removed copper zone on F.Cu, net /Project Architecture/PowerConnectors/VBuck_in
- removed copper zone on In2.Cu, net /Project Architecture/PowerConnectors/VBuck_in
- removed copper zone on B.Cu, net /Project Architecture/PowerConnectors/Vin_12V
- removed copper zone on F.Cu, net /Project Architecture/PowerConnectors/Vin_12V
- removed copper zone on In2.Cu, net /Project Architecture/PowerConnectors/Vin_12V
- removed copper zone on B.Cu, net /Project Architecture/PowerConnectors/Vin_15V
- removed copper zone on F.Cu, net /Project Architecture/PowerConnectors/Vin_15V
- removed copper zone on In2.Cu, net /Project Architecture/PowerConnectors/Vin_15V
- removed copper zone on B.Cu, net /Project Architecture/PowerConnectors/Vin_24V
- removed copper zone on F.Cu, net /Project Architecture/PowerConnectors/Vin_24V
- removed copper zone on In2.Cu, net /Project Architecture/PowerConnectors/Vin_24V
- removed copper zone on B.Cu, net /Project Architecture/PowerConnectors/Vin_5V
- removed copper zone on F.Cu, net /Project Architecture/PowerConnectors/Vin_5V
- removed copper zone on In2.Cu, net /Project Architecture/PowerConnectors/Vin_5V
- removed copper zone on B.Cu, net /Project Architecture/ProtectionCircuitry/out12V
- removed copper zone on F.Cu, net /Project Architecture/ProtectionCircuitry/out12V
- removed copper zone on In2.Cu, net /Project Architecture/ProtectionCircuitry/out12V
- removed copper zone on B.Cu, net /Project Architecture/ProtectionCircuitry/out15V
- removed copper zone on F.Cu, net /Project Architecture/ProtectionCircuitry/out15V
- removed copper zone on In2.Cu, net /Project Architecture/ProtectionCircuitry/out15V
- removed copper zone on B.Cu, net /Project Architecture/ProtectionCircuitry/out24V
- removed copper zone on F.Cu, net /Project Architecture/ProtectionCircuitry/out24V
- removed copper zone on In2.Cu, net /Project Architecture/ProtectionCircuitry/out24V
- removed copper zone on B.Cu, net /Project Architecture/ProtectionCircuitry/out5V
- removed copper zone on F.Cu, net /Project Architecture/ProtectionCircuitry/out5V
- removed copper zone on In2.Cu, net /Project Architecture/ProtectionCircuitry/out5V
- removed copper zone on B.Cu, net /Project Architecture/Sensors/outBatt
- removed copper zone on F.Cu, net /Project Architecture/Sensors/outBatt
- removed copper zone on In2.Cu, net /Project Architecture/Sensors/outBatt
- removed copper zone on B.Cu, net GND
- removed copper zone on F.Cu, net GND
Other:
- board size 98 x 77 mm -> 110 x 86 mm
- board text removed: "(max 10A)"
- board text removed: "12V"
- board text removed: "12V Buck Input"
- board text removed: "12V Buck Output"
- board text removed: "15V"
- board text removed: "15V Buck Input"
- board text removed: "15V Buck Output"
- board text removed: "24V"
- board text removed: "24V Buck Input"
- board text removed: "24V Buck Output"
- board text removed: "5V"
- board text removed: "5V Buck Input"
- board text removed: "5V Buck Output"
- board text removed: "ALAIN AZIZ"
- board text removed: "BUCKY++ REV A"
- board text removed: "Battery Input"
- board text removed: "DEBUG"
- board text removed: "DISPLAY"
- board text removed: "FAN"
- board text removed: "From Bucks"
- board text removed: "Input: 22V - 29.5V DC"
- board text removed: "Motor Output"
- board text removed: "Outputs"
- board text removed: "To Bucks"
- board text removed: "UART"
- board text removed: "USB"
