File: Icky/PowerConnectors.kicad_sch (KiCad schematic)
At the start: 36 parts, among them J1 XT60PW-M, J11 XT30AW-M, J12 XT30AW-M, J13 XT30AW-M, J14 XT30AW-M, J17 XT30UPB-F, J18 XT30UPB-F, J2 XT60PW-F, J3 XT30PW-F, J4 XT30PW-F, J5 XT30PW-F, J6 XT30PW-F, J7 XT30UPB-F, J8 XT30UPB-F

Commit message: ERC passed
Parts:
- removed C5, C6: 100u, Capacitor_SMD:C_1812_4532Metric_Pad1.57x3.40mm_HandSolder, symbol Device:C
- removed D18, D6: SMCJ12CA, Diode_SMD:D_SMA, symbol Diode:SMAJ12CA
- removed D9: SMCJ30CA, Diode_SMD:D_SMA, symbol Diode:SMAJ30CA
- removed J12: XT30AW-M, XT30AWM, symbol SamacSys_Parts:XT30AW-M
- removed J18: XT30UPB-F, XT30UPBF, symbol SamacSys_Parts:XT30UPB-F
- removed J4: XT30PW-F, XT30PWF, symbol SamacSys_Parts:XT30PW-F
Connections:
- net Batt_out renamed VBAT_OUT
- net VBatt_in renamed VBAT_IN
- no-connect marks 12 -> 10
Other:
- moved on the sheet: C10, C11, C14, C7, D19, D20, D21, D3, D4, D8, J13, J14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

Commit message: ERC passed v2
Parts:
- added D6: 5.0SMDJ30CA, DIONM7959X262N, symbol Device:D_TVS
- added J4: XT60PW-F, XT60PWF, symbol SamacSys_Parts:XT60PW-F
Connections:
- net GND: now also D6.1 (A1), J4.2
- new net VMOT_OUT: D6.2 (A2), J4.1
- no-connect marks 10 -> 12
Other:
- moved on the sheet: D5, J2

Commit message: routing
Parts:
- removed J3, J5, J6: XT30PW-F, XT30PWF, symbol SamacSys_Parts:XT30PW-F
- removed J4: XT60PW-F, XT60PWF, symbol SamacSys_Parts:XT60PW-F
- added J3, J4, J5: XT30UPB-F, XT30UPBF, symbol SamacSys_Parts:XT30UPB-F
- added J6: XT60PW-F, XT60PWF, symbol SamacSys_Parts:XT60PW-F
- C10, C11, C12, C13, C14, C7: footprint Capacitor_SMD:C_1812_4532Metric_Pad1.57x3.40mm_HandSolder -> Capacitor_SMD:C_0603_1608Metric
Connections:
- net 15V_VSAFE: now also J3.1
- net 24V_VSAFE: now also J4.1
- net 5V_VSAFE: now also J8.1
- net GND: now also J3.2, J4.2, J5.2, J6.2
- net VIN_SAFE: now also J5.1; no longer J8.1
- net VMOT_OUT: now also J6.1
- no-connect marks 12 -> 6
Other:
- moved on the sheet: J8
