File: Icky/Precharge.kicad_sch (KiCad schematic)
At the start: 22 parts, among them IC1 LM5069MM-2_NOPB, IC5 INA239AQDGSRQ1, Q1 SOT233 BSS123N, U17 SQJQ112E-T1_GE3, U7 SQJQ112E-T1_GE3, U8 SQJQ112E-T1_GE3

Commit message: routing
Parts:
- removed NT1: NetTieShuntH, 0_net_tie:NetTie-2_SMD_Pad0.2mm, symbol Device:NetTie_2
- removed NT2: NetTieShuntL, 0_net_tie:NetTie-2_SMD_Pad0.2mm, symbol Device:NetTie_2
- C20, C22, C29, C6: footprint 0_capacitor_smd:C_0402_1005_DensityHigh -> Capacitor_SMD:C_0603_1608Metric
- IC1: footprint SOP50P490X110-10N -> SamacSys_Parts:SOP50P490X110-10N
- IC5: footprint 0_diode_smd:SOP50P490X110-10N -> SamacSys_Parts:SOP50P490X110-10N
- Q1: footprint 0_package_SOT_TO_SMD:SOT-23-3 -> SamacSys_Parts:BSS123N
- R20: value 1m 1% 4W -> 1m 1% 8W; footprint (none) -> SamacSys_Parts:WSL39211L000JEA; Mfr BVS-M-R001-1.0 -> SEWF3920F1L00P9
- R21, R44, R45, R51, R56: footprint (none) -> Resistor_SMD:R_0603_1608Metric
- U17, U7, U8: footprint DPAK_2E-T1_GE3_VIS -> SamacSys_Parts:DPAK_2E-T1_GE3_VIS
Connections:
- net VBAT_IN: now also IC5.10 (IN+)
- net VMOT_SENS-: now also IC5.8 (VBUS), IC5.9 (IN-)
Other:
- moved on the sheet: C29, IC5
