File: Icky/Project Architecture.kicad_sch (KiCad schematic)
At the start: 8 parts

Commit message: ERC passed
Other:
- removed sheet Sensors
- sheet MCU & Local Power ports: added VIN_FLT, VIN_SAFE, VMOT_ALERT, {15V_PROT}, {24V_PROT}, {5V_PROT}; removed +VBAT, 12V, 12V alert, 15V alert, 24V alert, 5V alert, PG_12V, PG_15V, PG_24V, PG_5V, PG_Batt, input alert, {SHDN_CTRL}
- sheet PowerConnectors ports: added VBAT_IN, VBAT_OUT, VIN_SAFE, {VBUCK}, {VSAFE}; removed Batt_out, VBatt_in, {Buck_Outputs}, {Safe_Outputs}
- sheet Protection & Monitoring ports: added VBAT, VIN_FLT, VIN_SAFE, VMOT_ALERT, {15V_PROT}, {24V_PROT}, {5V_PROT}, {SPI_BAT}, {VBUCK}, {VSAFE}; removed 12V_fans, PG_12V, PG_15V, PG_24V, PG_5V, PG_Batt, VBatt_protection, VBatt_safe, {SHDN_CTRL}, {Safe_Outputs}, {Shunt_Outputs}
- note removed: "Page 4"
- note removed: "Page 5"
- moved on the sheet: C16, C17, C21, C9, H1, H2, H3, H501

Commit message: ERC passed v2
Other:
- sheet MCU & Local Power ports: added VIN_SAFE_LOCAL, {SPI_SENSORS}, {VIN_PROT}, {VMOT_PROT}; removed VIN_FLT, VIN_SAFE, VMOT_ALERT, {SPI_BAT}
- sheet PowerConnectors ports: added VMOT_OUT; removed none
- sheet Protection & Monitoring ports: added VIN_SAFE_LOCAL, VMOT, {SPI_SENSORS}, {VIN_PROT}, {VMOT_PROT}; removed VIN_FLT, VMOT_ALERT, {SPI_BAT}

Commit message: routing
Parts:
- C16, C17, C21, C9: footprint 0_capacitor_smd:C_0402_1005_DensityHigh -> Capacitor_SMD:C_0603_1608Metric
- H1, H2, H3: value M2 (3.2mm) -> M2 (2.2mm)
- H4: renamed from H501; value M2 (3.2mm) -> M2 (2.2mm)
Changed lines of the file:
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@@
 			)
 		)
-		(property "Value" "M2 (3.2mm)"
+		(property "Value" "M2 (2.2mm)"
 			(at 65.405 147.3199 0)
 			(effects
@@
 			)
 		)
-		(property "Footprint" "0_capacitor_smd:C_0402_1005_DensityHigh"
+		(property "Footprint" "Capacitor_SMD:C_0603_1608Metric"
 			(at 63.1952 157.48 0)
 			(effects
@@
 			)
 		)
-		(property "Footprint" "0_capacitor_smd:C_0402_1005_DensityHigh"
+		(property "Footprint" "Capacitor_SMD:C_0603_1608Metric"
 			(at 63.1952 184.15 0)
 			(effects
@@
 			)
 		)
-		(property "Footprint" "0_capacitor_smd:C_0402_1005_DensityHigh"
+		(property "Footprint" "Capacitor_SMD:C_0603_1608Metric"
 			(at 39.0652 157.48 0)
 			(effects
@@
 			)
 		)
-		(property "Value" "M2 (3.2mm)"
+		(property "Value" "M2 (2.2mm)"
 			(at 65.405 173.9899 0)
 			(effects
@@
 		(dnp no)
 		(fields_autoplaced yes)
-		(property "Reference" "H501"
+		(property "Reference" "H4"
 			(at 41.275 171.4499 0)
 			(effects
@@
 			)
 		)
-		(property "Value" "M2 (3.2mm)"
+		(property "Value" "M2 (2.2mm)"
 			(at 41.275 173.9899 0)
 			(effects
@@
 			(project "Bucky++"
 				(path "/0650c7a8-acba-429c-9f8e-eec0baf0bc1c/fede4c36-00cc-4d3d-b71c-5243ba232202"
-					(reference "H501")
+					(reference "H4")
 					(unit 1)
 				)
@@
 			)
 		)
-		(property "Footprint" "0_capacitor_smd:C_0402_1005_DensityHigh"
+		(property "Footprint" "Capacitor_SMD:C_0603_1608Metric"
 			(at 39.0652 184.15 0)
 			(effects
@@
 			)
 		)
-		(property "Value" "M2 (3.2mm)"
+		(property "Value" "M2 (2.2mm)"
 			(at 41.275 147.3199 0)
 			(effects
