File: Icky/ProtectionCircuitry.kicad_sch (KiCad schematic)
At the start: 15 parts, among them IC10 LTC4368IMS-2#PBF, IC6 INA239AQDGSRQ1

Commit message: ERC passed
Connections:
- net SPI1_NSS4 renamed SPI1_NSS3
Other:
- removed sheet 12V

Commit message: ERC passed v2
Parts:
- removed R39: 1m 1% 4W, symbol Device:R
Connections:
- net VMOT_SENS+ is gone; now on net VIN_D: NT7.2
- net VMOT_SENS- is gone; now on net VIN_SAFE: NT8.2
- net VMOT_ALERT renamed VIN_ALERT
Other:
- added sheet VMOT (Precharge.kicad_sch)
- sheet 15V ports: added {SPI_SENSORS}; removed {SPI_BAT}
- sheet 24V ports: added {SPI_SENSORS}; removed {SPI_BAT}
- sheet 5V ports: added {SPI_SENSORS}; removed {SPI_BAT}
- moved on the sheet: C27, C28, C8, IC10, IC6, NT7, NT8, R40, R41, R42, R43, R58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

Commit message: routing
Parts:
- removed NT7: NetTieShuntH, 0_net_tie:NetTie-2_SMD_Pad0.2mm, symbol Device:NetTie_2
- removed NT8: NetTieShuntL, 0_net_tie:NetTie-2_SMD_Pad0.2mm, symbol Device:NetTie_2
- C27, C28: footprint (none) -> Capacitor_SMD:C_0603_1608Metric
- C8: footprint 0_capacitor_smd:C_0402_1005_DensityHigh -> Capacitor_SMD:C_0603_1608Metric
- IC10: footprint SOP50P490X110-10N -> SamacSys_Parts:SOP50P490X110-10N
- IC6: footprint 0_diode_smd:SOP50P490X110-10N -> SamacSys_Parts:SOP50P490X110-10N
- R40, R41, R42, R43, R58, R62: footprint (none) -> Resistor_SMD:R_0603_1608Metric
- R8: value 1m 1% 4W -> 1m 1% 8W; footprint (none) -> SamacSys_Parts:WSL39211L000JEA
Connections:
- net VIN_D: now also IC6.10 (IN+)
- net VIN_SAFE: now also IC6.8 (VBUS), IC6.9 (IN-)
Changed lines of the file:
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@@
 	)
 	(bus_alias "VBUCK"
-		(members "5V_VSAFE" "15V_VSAFE" "24V_VSAFE")
+		(members "5V_VBUCK" "15V_VBUCK" "24V_VBUCK")
 	)
 	(bus_alias "VSAFE"
@@
 	(wire
 		(pts
-			(xy 87.63 125.73) (xy 92.71 125.73)
+			(xy 87.63 125.73) (xy 100.33 125.73)
 		)
 		(stroke
@@
 	(wire
 		(pts
-			(xy 97.79 128.27) (xy 111.76 128.27)
-		)
-		(stroke
-			(width 0)
-			(type default)
-		)
-	)
-	(wire
-		(pts
 			(xy 90.17 97.79) (xy 90.17 87.63)
 		)
@@
 	(wire
 		(pts
-			(xy 90.805 128.27) (xy 92.71 128.27)
+			(xy 90.805 128.27) (xy 100.33 128.27)
 		)
 		(stroke
@@
 	(wire
 		(pts
-			(xy 97.79 125.73) (xy 111.76 125.73)
-		)
-		(stroke
-			(width 0)
-			(type default)
-		)
-	)
-	(wire
-		(pts
 			(xy 167.64 48.26) (xy 156.21 48.26)
 		)
@@
 	)
 	(label "VIN_OUT"
-		(at 111.76 128.27 180)
+		(at 100.33 128.27 180)
 		(effects
 			(font
@@
 	)
 	(label "VIN_D"
-		(at 111.76 125.73 180)
+		(at 100.33 125.73 180)
 		(effects
 			(font
@@
 			)
 		)
-		(property "Footprint" ""
+		(property "Footprint" "Resistor_SMD:R_0603_1608Metric"
 			(at 107.442 58.42 90)
 			(effects
@@
 			)
 		)
-		(property "Footprint" ""
+		(property "Footprint" "Capacitor_SMD:C_0603_1608Metric"
 			(at 90.17 82.55 0)
 			(effects
@@
 			)
 		)
-		(property "Footprint" ""
+		(property "Footprint" "Resistor_SMD:R_0603_1608Metric"
 			(at 26.162 82.55 90)
 			(effects
@@
 			)
 		)
-		(property "Footprint" ""
+		(property "Footprint" "Resistor_SMD:R_0603_1608Metric"
 			(at 38.1 58.928 90)
 			(effects
@@
 	)
 	(symbol
-		(lib_id "Device:NetTie_2")
-		(at 95.25 125.73 0)
-		(unit 1)
-		(exclude_from_sim no)
-		(in_bom no)
-		(on_board yes)
-		(dnp no)
-		(property "Reference" "NT7"
-			(at 95.885 121.92 0)
-			(effects
-				(font
-					(size 1.27 1.27)
-				)
-			)
-		)
-		(property "Value" "NetTieShuntH"
-			(at 96.52 123.825 0)
-			(effects
-				(font
-					(size 1.27 1.27)
-				)
-			)
-		)
-		(property "Footprint" "0_net_tie:NetTie-2_SMD_Pad0.2mm"
-			(at 95.25 125.73 0)
-			(effects
-				(font
-					(size 1.27 1.27)
-				)
-				(hide yes)
-			)
-		)
-		(property "Datasheet" "~"
-			(at 95.25 125.73 0)
-			(effects
-				(font
-					(size 1.27 1.27)
-				)
-				(hide yes)
-			)
-		)
-		(property "Description" ""
-			(at 95.25 125.73 0)
-			(effects
-				(font
-					(size 1.27 1.27)
-				)
-				(hide yes)
-			)
-		)
-		(pin "1"
-		)
-		(pin "2"
-		)
-		(instances
-			(project "Icky"
-				(path "/0650c7a8-acba-429c-9f8e-eec0baf0bc1c/fede4c36-00cc-4d3d-b71c-5243ba232202/7d5a1283-086b-46b0-8df7-a9850521fb5e"
-					(reference "NT7")
-					(unit 1)
-				)
-			)
-		)
-	)
-	(symbol
 		(lib_id "power:+3V3")
 		(at 109.22 133.35 0)
@@
 			)
 		)
-		(property "Footprint" ""
+		(property "Footprint" "Resistor_SMD:R_0603_1608Metric"
 			(at 26.162 72.39 90)
 			(effects
@@
 	)
 	(symbol
-		(lib_id "Device:NetTie_2")
-		(at 95.25 128.27 0)
-		(unit 1)
-		(exclude_from_sim no)
-		(in_bom no)
-		(on_board yes)
-		(dnp no)
-		(property "Reference" "NT8"
-			(at 95.885 129.54 0)
-			(effects
-				(font
-					(size 1.27 1.27)
-				)
-			)
-		)
-		(property "Value" "NetTieShuntL"
-			(at 96.52 131.445 0)
-			(effects
-				(font
-					(size 1.27 1.27)
-				)
-			)
-		)
-		(property "Footprint" "0_net_tie:NetTie-2_SMD_Pad0.2mm"
-			(at 95.25 128.27 0)
-			(effects
-				(font
-					(size 1.27 1.27)
-				)
-				(hide yes)
-			)
-		)
-		(property "Datasheet" "~"
-			(at 95.25 128.27 0)
-			(effects
-				(font
-					(size 1.27 1.27)
-				)
-				(hide yes)
-			)
-		)
-		(property "Description" ""
-			(at 95.25 128.27 0)
-			(effects
-				(font
-					(size 1.27 1.27)
-				)
-				(hide yes)
-			)
-		)
-		(pin "1"
-		)
-		(pin "2"
-		)
-		(instances
-			(project "Icky"
-				(path "/0650c7a8-acba-429c-9f8e-eec0baf0bc1c/fede4c36-00cc-4d3d-b71c-5243ba232202/7d5a1283-086b-46b0-8df7-a9850521fb5e"
-					(reference "NT8")
-					(unit 1)
-				)
-			)
-		)
-	)
-	(symbol
 		(lib_id "Device:C_Small")
 		(at 97.79 137.16 0)
@@
 			)
 		)
-		(property "Footprint" "0_capacitor_smd:C_0402_1005_DensityHigh"
+		(property "Footprint" "Capacitor_SMD:C_0603_1608Metric"
 			(at 97.79 137.16 0)
 			(effects
@@
 			)
 		)
-		(property "Footprint" ""
+		(property "Footprint" "Resistor_SMD:R_0603_1608Metric"
 			(at 99.822 58.42 90)
 			(effects
@@
 			)
 		)
-		(property "Footprint" "SOP50P490X110-10N"
+		(property "Footprint" "SamacSys_Parts:SOP50P490X110-10N"
 			(at 73.66 162.23 0)
 			(effects
@@
 			)
 		)
-		(property "Value" "1m 1% 4W"
+		(property "Value" "1m 1% 8W"
 			(at 70.866 45.72 90)
 			(effects
@@
 			)
 		)
-		(property "Footprint" ""
+		(property "Footprint" "SamacSys_Parts:WSL39211L000JEA"
 			(at 71.12 46.482 90)
 			(effects
@@
 			)
 		)
-		(property "Description" "BVS-M-R001-1.0"
+		(property "Description" "SEWF3920F1L00P9"
 			(at 71.12 48.26 0)
 			(effects
@@
 			)
 		)
-		(property "Footprint" "0_diode_smd:SOP50P490X110-10N"
+		(property "Footprint" "SamacSys_Parts:SOP50P490X110-10N"
 			(at 83.82 220.65 0)
 			(effects
@@
 			)
 		)
-		(property "Footprint" ""
+		(property "Footprint" "Resistor_SMD:R_0603_1608Metric"
 			(at 26.162 92.71 90)
 			(effects
@@
 			)
 		)
-		(property "Footprint" ""
+		(property "Footprint" "Capacitor_SMD:C_0603_1608Metric"
 			(at 31.75 60.96 0)
 			(effects
