File: Castor/LT8705A.kicad_sch (KiCad schematic)
At the start: 45 parts, among them J1 IPS1-105-01-L-D, J6 IPS1-105-01-L-D, Q3 SQJ850EP, Q4 SQJ886EP, Q5 SQJ486EP, Q6 SQJ410EP, U8 TPS16851VMAR, U9 LT8705AxFE

Commit message: fixed en bug
Connections:
- net EN is gone; now on net Vin: U9.4 (~{SHDN})
Other:
- note added: "Mode Floating for Burst operation"
Changed lines of the file:
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@@
+		)
+	)
+	(text "Mode Floating for Burst operation"
+		(exclude_from_sim no)
+		(at 78.232 154.686 0)
+		(effects
+			(font
+				(size 1.27 1.27)
+			)
 		)
 	)
@@
 	(junction
 		(at 39.624 19.558)
+		(diameter 0)
+		(color 0 0 0 0)
+	)
+	(junction
+		(at 108.458 141.478)
 		(diameter 0)
 		(color 0 0 0 0)
@@
 	(wire
 		(pts
+			(xy 113.284 144.018) (xy 108.458 144.018)
+		)
+		(stroke
+			(width 0)
+			(type default)
+		)
+	)
+	(wire
+		(pts
 			(xy 165.354 171.958) (xy 180.594 171.958)
 		)
@@
 	(wire
 		(pts
-			(xy 102.87 141.478) (xy 113.284 141.478)
+			(xy 102.87 141.478) (xy 108.458 141.478)
 		)
 		(stroke
@@
 	(wire
 		(pts
-			(xy 110.744 149.098) (xy 113.284 149.098)
-		)
-		(stroke
-			(width 0)
-			(type default)
-		)
-	)
-	(wire
-		(pts
 			(xy 241.808 19.558) (xy 241.808 117.348)
 		)
@@
 	(wire
 		(pts
+			(xy 108.458 141.478) (xy 113.284 141.478)
+		)
+		(stroke
+			(width 0)
+			(type default)
+		)
+	)
+	(wire
+		(pts
 			(xy 146.304 113.538) (xy 146.304 99.568)
 		)
@@
 		(pts
 			(xy 102.87 141.478) (xy 102.87 141.986)
+		)
+		(stroke
+			(width 0)
+			(type default)
+		)
+	)
+	(wire
+		(pts
+			(xy 108.458 144.018) (xy 108.458 141.478)
 		)
 		(stroke
@@
 		)
 	)
-	(hierarchical_label "EN"
-		(shape input)
-		(at 110.744 149.098 180)
-		(effects
-			(font
-				(size 1.27 1.27)
-			)
-			(justify right)
-		)
-	)

Commit message: castor
Parts:
- added C? (x4): 1nF, Capacitor_SMD:C_1210_3225Metric, symbol Device:C
- added C?: 0.22uF, Capacitor_SMD:C_1210_3225Metric, symbol Device:C
- added C?: 0.01uF, Capacitor_SMD:C_1210_3225Metric, symbol Device:C
- added CDV/DT, Ctimer: ?, Capacitor_SMD:C_1210_3225Metric, symbol Device:C
- added R1OVLO, R1UVLO, R2OVLO, R2UVLO, R2UVLO? (x2), RILIM, RIMON, RIREF: ?, Resistor_SMD:R_0603_1608Metric, symbol Device:R
- added R2OVLO?: 150k, Resistor_SMD:R_0603_1608Metric, symbol Device:R
- added R?: 150, Resistor_SMD:R_0603_1608Metric, symbol Device:R
Connections:
- net GND: now also U8.5 (GND), C?.1, C?.1, C?.1, C?.1, C?.1, C?.1, CDV/DT.1, Ctimer.2, R2OVLO.2, R2OVLO?.2, R2UVLO.2, RILIM.2, RIMON.2, RIREF.2
- net IN: now also C?.2, R1OVLO.1, R1UVLO.1, R?.1
- net at U8.1 (ILIM): now also RILIM.1
- net at U8.13 (~{FLT}): now also R2UVLO?.2
- net at U8.14 (ITIMER): now also Ctimer.1
- net at U8.16 (EN/UVLO): now also C?.2, R1UVLO.2, R2UVLO.1
- net at U8.18 (OVP): now also C?.2, R1OVLO.2, R2OVLO.1
- net at U8.19 (PGOOD): now also R2UVLO?.2
- net at U8.2 (IMON): now also C?.2, RIMON.1
- net at U8.3 (IREF): now also C?.2, RIREF.1
- net at U8.4 (DVDT): now also CDV/DT.2
- net at U8.6 (SFT_SEL): now also R2OVLO?.1
- net at U8.9 (VDD): now also C?.2, R?.2
Other:
- moved on the sheet: U8
